File: 2020/Robot_Lancer/Aqualius_Sadalmeric/Main/Main.kicad_pcb (KiCad board)
At the start: 2 copper layers, 100 x 100 mm, 320 parts, among them J1 SERIAL0, J10 I/O_Vdd, J11 ENC0, J12 ENC1, J13 ENC2, J14 ENC3, J15 5Vin, J16 EMERGENCY, J17 MOTOR0, J18 MOTOR1, J19 MOTOR2, J2 ADC, J20 MOTOR3, J21 MOTOR4, J22 MOTOR5, J23 BATT_IN, J24 BATT_IN, J25 FUSE, J3 SWD, J4 CAN, J5 ADC_Vdd, J6 SERIAL1, J7 CAN, J8 I/O, J9 SERIAL2, Q1 NPN, Q10 NVMFD5C446NLT1G, Q11 FET_N, Q12 NVMFD5C446NLT1G, Q13 NVMFD5C446NLT1G, Q14 NVMFD5C446NLT1G, Q15 NVMFD5C446NLT1G, Q16 NVMFD5C446NLT1G, Q17 NVMFD5C446NLT1G, Q18 FET_P, Q2 NPN, Q3 FET_P, Q4 FET_P, Q5 NVMFD5C446NLT1G, Q6 NVMFD5C446NLT1G, Q7 NVMFD5C446NLT1G, Q8 NVMFD5C446NLT1G, Q9 NVMFD5C446NLT1G, SW1 RESET, SW2 DIP_SW, SW3 SW0, SW4 SW1, SW5 Control-Power_SW, SW6 SW2, SW7 SW3, SW8 EMERGENCY_SW, SW9 MAIN_SW, U1 MAX3051, U10 BD9G101G, U11 CCG30-24-12, U12 NCP5104, U13 NCP5104, U14 NCP5104, U15 NCP5104, U16 NCP5104, U17 NCP5104, U18 V23086-C1001, U19 NCP5104, U2 AP3211, U20 NCP5104, U21 NCP5104, U22 NCP5104, U23 NCP5104, U24 NCP5104, U25 LOGO, U26 7805, U3 MCP2221A, U4 AQM1602_BL, U5 AZ1086H, U6 STM32F407VG, U7 OSTBABS4C2B, U8 ADRESS, U9 25LC010A, Y1 8MHz

Commit message: いい感じじゃね
Parts:
- C13, C15, C41, C50, C59, D16, D39, D47, L2, Q18, R57, R71, R72, R73, R81, R82, U2: moved to B.Cu
- C52: value 470u -> 220u; footprint Capacitor_THT:CP_Radial_D10.0mm_P5.00mm -> Capacitor_THT:CP_Radial_D8.0mm_P3.50mm
- C60, C61: footprint Capacitor_THT:CP_Radial_D10.0mm_P5.00mm -> Mizz_lib:CAPAE1300X1400N
- R8: value R -> 50k
- R9: value R -> 10k
- moved L2 217.6 mm to (96.5, 62.5)
- moved C55 214.8 mm to (109.2, 78.5), turned to 270 degrees
- moved D39 197.0 mm to (91.5, 60.8), turned to 90 degrees
- moved D36 197.0 mm to (129.5, 64.5), turned to 180 degrees
- moved R73 192.8 mm to (111.5, 78.4), turned to 180 degrees
- moved D16 192.7 mm to (51.2, 53.2), turned to 90 degrees
- moved R71 182.8 mm to (111.5, 72.2), turned to 180 degrees
- moved C45 181.6 mm to (100.2, 71.8), turned to 270 degrees
- moved C39 177.9 mm to (94.5, 110.5)
- moved D48 173.1 mm to (77.5, 64.6)
- moved D47 169.2 mm to (102.8, 62.5), turned to 180 degrees
- moved C59 168.3 mm to (101.0, 60.0), turned to 90 degrees
- moved R65 163.3 mm to (126.5, 64.5), turned to 180 degrees
- moved C44 159.1 mm to (100.2, 65.6), turned to 270 degrees
- moved C41 159.0 mm to (86.8, 65.5)
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Routing:
- net +12P: track 0.00 -> 53.1 mm, vias 0 -> 9
- net +5P: track 10.2 -> 49.3 mm
- net Batt: track 0.00 -> 29.6 mm
- net /MOTOR0L_PWM: track 0.00 -> 23.7 mm, vias 0 -> 2
- net /MOTOR5R_PWM: track 0.00 -> 23.4 mm, vias 0 -> 2
- net /MOTOR2R_PWM: track 0.00 -> 22.7 mm, vias 0 -> 2
- net /FB_OUT: track 0.00 -> 19.3 mm, vias 0 -> 1
- net /MOTOR5L_PWM: track 0.00 -> 18.3 mm, vias 0 -> 2
- net /MOTOR2L_PWM: track 0.00 -> 17.8 mm, vias 0 -> 2
- net /MOTOR3L_PWM: track 0.00 -> 17.3 mm, vias 0 -> 2
- net /MOTOR0R_PWM: track 0.00 -> 13.2 mm, vias 0 -> 2
- net /MOTOR4R_PWM: track 0.00 -> 13.0 mm, vias 0 -> 2
- net /MOTOR1R_PWM: track 0.00 -> 12.8 mm, vias 0 -> 2
- net /MOTOR3R_PWM: track 0.00 -> 12.2 mm, vias 0 -> 2
- net /MOTOR4L_PWM: track 0.00 -> 11.1 mm, vias 0 -> 2
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Other:
- board text added: "Main + Power + MD*6"

Commit message: ブートストラップコンデンサ並べた,進捗git add -Agit add -A
Parts:
- removed R10, R26: 10, Resistor_SMD:R_0603_1608Metric
- added SW10: TOGGLESW1, Mizz_lib:2MS1-T1-B4-VS2-Q-E, F.Cu at (73.5, 131.5)
- added SW11: TOGGLESW2, Mizz_lib:2MS1-T1-B4-VS2-Q-E, F.Cu at (79.0, 131.5)
- added SW12: TOGGLESW3, Mizz_lib:2MS1-T1-B4-VS2-Q-E, F.Cu at (84.5, 131.5)
- C10, C2, C25, C26, C27, C28, C31, C6, D12, D20, D24, D35, JP1, Q2, R24, R25, R27, R74, R8, R9, U3, U5: moved to B.Cu
- C20: footprint Capacitor_SMD:C_0603_1608Metric -> Capacitor_SMD:C_0805_2012Metric
- J4, J7: footprint Mizz_lib:XA_4L -> Mizz_lib:XA_4P
- SW1: footprint Button_Switch_SMD:SW_SPST_PTS645 -> Button_Switch_SMD:SW_SPST_PTS810
- SW2: value DIP_SW -> TOGGLESW0; footprint Mizz_lib:KHS4 -> Mizz_lib:2MS1-T1-B4-VS2-Q-E
- SW3, SW4, SW6, SW7: footprint Button_Switch_SMD:SW_SPST_CK_RS282G05A3 -> Button_Switch_SMD:SW_SPST_PTS810
- U4: value AQM1602_BL -> AQM0802_BL; footprint Mizz_lib:AQM1602_BL_Fad -> Mizz_lib:AQM0802_LED
- moved C71 239.2 mm to (109.2, 121.5), turned to 270 degrees
- moved J3 236.5 mm to (51.0, 135.2), turned to 180 degrees
- moved J5 225.7 mm to (40.2, 82.8), turned to 180 degrees
- moved J8 222.7 mm to (42.9, 86.8)
- moved U9 222.2 mm to (75.5, 99.2)
- moved J11 217.7 mm to (39.2, 109.2), turned to 270 degrees
- moved J16 217.5 mm to (133.1, 70.7), turned to 90 degrees
- moved SW2 215.5 mm to (68.0, 131.5), turned to 270 degrees
- moved C56 215.3 mm to (109.2, 84.5), turned to 270 degrees
- moved J13 212.0 mm to (45.8, 129.2), turned to 90 degrees
- moved J6 211.0 mm to (75.1, 112.8), turned to 180 degrees
- moved JP1 208.5 mm to (54.8, 132.0), turned to 270 degrees
- moved J12 206.8 mm to (39.2, 121.8), turned to 270 degrees
- moved J1 206.1 mm to (67.6, 119.2)
- moved J10 202.8 mm to (40.3, 104.5), turned to 180 degrees
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Connections:
- Q1 pad 1: Net-(Q1-Pad1) -> /PB8_Buzzer_TIM10_CH1
- Q2 pad 1: Net-(Q2-Pad1) -> /PB9_LCD_BL_TIM11_CH1
- R39 pad 1: GND -> /PD3_DIPSW_1
- R39 pad 2: /PD6_DIPSW_3 -> +3V3
- R42 pad 1: GND -> /PD4_DIPSW_2
- R42 pad 2: /PD4_DIPSW_2 -> +3V3
- R45 pad 1: GND -> /PD6_DIPSW_3
- R45 pad 2: /PD3_DIPSW_1 -> +3V3
- R46 pad 1: GND -> /PD2_DIPSW_0
- R46 pad 2: /PD2_DIPSW_0 -> +3V3
- SW2 pad 1: +3V3 -> Net-(SW2-Pad1)
- SW2 pad 2: +3V3 -> /PD2_DIPSW_0
- SW2 pad 3: +3V3 -> GND
Routing:
- net +12P: track 53.1 -> 84.6 mm
- net +12V: track 0.00 -> 12.5 mm, vias 0 -> 2
- net Net-(C42-Pad1): track 0.00 -> 9.79 mm
- net /~RST: track 0.00 -> 9.00 mm, vias 0 -> 1
- net Net-(C15-Pad1): track 0.00 -> 5.50 mm
- net Net-(J3-Pad2): track 0.00 -> 3.41 mm
- net +3V3: track 0.00 -> 2.67 mm
- net Net-(D12-Pad2): track 0.00 -> 2.22 mm
- net Net-(C13-Pad2): track 0.00 -> 1.95 mm
- net Net-(C13-Pad1): track 0.00 -> 1.95 mm
- net Net-(D6-Pad2): vias 0 -> 1
Other:
- board text added: "."
- board text added: "0"
- board text added: "1"
- board text added: "2"
- board text added: "3"
- board text added: "7"
- board text added: "9"
- board text added: "EMG"
- board text added: "ENC"
- board text added: "Main+Power+MD*6="
- board text added: "SW"
- board text added: "TOGLE_SWITCH"
- board text removed: "Main + Power + MD*6"

Commit message: CAN通信の終端抵抗のジャンパー抵抗部分を忘れていた.追加,進捗git add -Agit add -A
Parts:
- C20, C4, C8, D23, D33, L1, Q3: moved to B.Cu
- D24: moved to F.Cu
- U1: footprint Package_SO:SOIC-8_3.9x4.9mm_P1.27mm -> Package_SO:TSSOP-8_3x3mm_P0.65mm; moved to B.Cu
- moved J15 176.2 mm to (78.8, 73.0), turned to 180 degrees
- moved Q4 167.4 mm to (67.4, 65.4), turned to 180 degrees
- moved D34 163.5 mm to (70.7, 66.2), turned to 270 degrees
- moved U1 161.8 mm to (48.9, 60.3), turned to 90 degrees
- moved SW5 150.6 mm to (52.6, 62.6), turned to 90 degrees
- moved Q3 150.4 mm to (57.2, 65.0), turned to 270 degrees
- moved C4 145.9 mm to (47.8, 64.0), turned to 180 degrees
- moved D33 145.3 mm to (66.3, 60.8), turned to 180 degrees
- moved JP2 144.4 mm to (106.3, 35.1), turned to 180 degrees
- moved R53 126.4 mm to (67.8, 68.0)
- moved D23 19.8 mm to (64.7, 57.0)
- moved L1 16.8 mm to (60.5, 50.7), turned to 270 degrees
- moved C20 16.7 mm to (62.5, 56.3), turned to 270 degrees
- moved D20 15.7 mm to (54.3, 50.0), turned to 90 degrees
- moved C8 13.1 mm to (60.8, 56.1), turned to 270 degrees
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Routing:
- net Net-(C15-Pad1): track 5.50 -> 0.17 mm
- net Net-(C13-Pad2): track 1.95 -> 0.00 mm
- net Net-(C13-Pad1): track 1.95 -> 0.00 mm

Commit message: バックアップ
Parts:
- added JP3: CAN_JP, Connector_PinHeader_2.54mm:PinHeader_1x02_P2.54mm_Vertical, F.Cu at (44.4, 42.6)
- added R10: 120, Resistor_SMD:R_0603_1608Metric, B.Cu at (41.5, 45.5)
- C11, C14, C16, C17, C18, C21, C24, C29, C30, D1, D10, R100, R101, R102, R103, R104, R105, R39, R42, R45, R46, R75, R76, R77, R78, R79, R80, R94, R95, R96, R97, R98, R99: moved to B.Cu
- moved D1 226.6 mm to (74.2, 116.0)
- moved R105 208.6 mm to (111.5, 136.3), turned to 180 degrees
- moved R79 197.5 mm to (111.5, 96.7), turned to 180 degrees
- moved R102 194.7 mm to (111.5, 127.7), turned to 180 degrees
- moved R98 192.1 mm to (111.5, 115.3), turned to 180 degrees
- moved R45 189.6 mm to (82.5, 132.3), turned to 90 degrees
- moved R99 188.2 mm to (111.5, 117.8), turned to 180 degrees
- moved R97 185.4 mm to (111.5, 111.7), turned to 180 degrees
- moved C62 183.4 mm to (100.2, 102.6), turned to 270 degrees
- moved R39 182.7 mm to (71.5, 132.3), turned to 90 degrees
- moved R101 180.8 mm to (111.5, 124.0), turned to 180 degrees
- moved C49 180.7 mm to (100.2, 96.4), turned to 270 degrees
- moved R76 180.1 mm to (111.5, 87.0), turned to 180 degrees
- moved R42 174.9 mm to (77.1, 132.3), turned to 90 degrees
- moved R104 174.9 mm to (111.5, 133.8), turned to 180 degrees
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Connections:
- C62 pad 1: MOTOR_Batt -> +12P
- C63 pad 1: MOTOR_Batt -> +12P
- C64 pad 1: MOTOR_Batt -> +12P
- C65 pad 1: MOTOR_Batt -> +12P
- C66 pad 1: MOTOR_Batt -> +12P
- C67 pad 1: MOTOR_Batt -> +12P
- D50 pad 2: MOTOR_Batt -> +12P
- D51 pad 2: MOTOR_Batt -> +12P
- D52 pad 2: MOTOR_Batt -> +12P
- D53 pad 2: MOTOR_Batt -> +12P
- D54 pad 2: MOTOR_Batt -> +12P
- D55 pad 2: MOTOR_Batt -> +12P
- R39 pad 1: /PD3_DIPSW_1 -> GND
- R39 pad 2: +3V3 -> /PD3_DIPSW_1
- R42 pad 1: /PD4_DIPSW_2 -> GND
- R42 pad 2: +3V3 -> /PD4_DIPSW_2
- R45 pad 1: /PD6_DIPSW_3 -> GND
- R45 pad 2: +3V3 -> /PD6_DIPSW_3
- R46 pad 1: /PD2_DIPSW_0 -> GND
- R46 pad 2: +3V3 -> /PD2_DIPSW_0
- R88 pad 1: MOTOR_Batt -> +12P
- R89 pad 1: MOTOR_Batt -> +12P
- R90 pad 1: MOTOR_Batt -> +12P
- R91 pad 1: MOTOR_Batt -> +12P
- R92 pad 1: MOTOR_Batt -> +12P
- R93 pad 1: MOTOR_Batt -> +12P
- SW10 pad 1: Net-(SW10-Pad1) -> +3V3
- SW10 pad 3: GND -> Net-(SW10-Pad3)
- SW11 pad 1: Net-(SW11-Pad1) -> +3V3
- SW11 pad 3: GND -> Net-(SW11-Pad3)
- SW12 pad 1: Net-(SW12-Pad1) -> +3V3
- SW12 pad 3: GND -> Net-(SW12-Pad3)
- SW2 pad 1: Net-(SW2-Pad1) -> +3V3
- SW2 pad 3: GND -> Net-(SW2-Pad3)
- SW9 pad 2: POWER_Batt -> Net-(D49-Pad2)
- U19 pad 1: MOTOR_Batt -> +12P
- U20 pad 1: MOTOR_Batt -> +12P
- U21 pad 1: MOTOR_Batt -> +12P
- U22 pad 1: MOTOR_Batt -> +12P
- U23 pad 1: MOTOR_Batt -> +12P
- U24 pad 1: MOTOR_Batt -> +12P
Routing:
- net Batt: track 29.6 -> 8.67 mm
- net Net-(D56-Pad2): track 0.00 -> 20.6 mm
- net /CAN_H: track 0.00 -> 11.2 mm
- net POWER_Batt: track 10.0 -> 0.00 mm
- net /Motor1R: track 0.00 -> 8.10 mm, vias 18 -> 20
- net Net-(JP3-Pad2): track 0.00 -> 6.49 mm
- net Net-(D49-Pad2): track 6.04 -> 11.0 mm
- net Net-(D56-Pad1): track 0.00 -> 4.88 mm
- net Net-(R75-Pad2): track 0.00 -> 3.39 mm, vias 0 -> 1
- net Net-(R74-Pad2): track 0.00 -> 3.36 mm, vias 0 -> 1
- net /CAN_L: track 0.00 -> 2.92 mm
- net /Motor2R: track 0.00 -> 2.02 mm
- net /Motor3R: track 0.00 -> 2.02 mm, vias 0 -> 18
- net /Motor3L: track 0.00 -> 2.02 mm, vias 0 -> 18
- net /Motor2L: track 0.00 -> 2.02 mm
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Other:
- board text added: "SPEAKER"

Commit message: Aloe
Parts:
- removed D21, D22, D25, D26: DIODE, Diode_SMD:D_SOD-123
- R17, R36, R37, R38, R5, R59, R60, R61, R62, R63, R64, R83, R88, R89, R90, R91, R92, R93: moved to B.Cu
- moved D30 241.3 mm to (83.5, 94.1), turned to 180 degrees
- moved R93 191.1 mm to (103.2, 129.0), turned to 180 degrees
- moved R90 181.8 mm to (103.3, 135.2), turned to 180 degrees
- moved D29 176.5 mm to (83.5, 91.3), turned to 180 degrees
- moved D27 168.5 mm to (83.5, 85.7), turned to 180 degrees
- moved R88 167.0 mm to (103.3, 110.5), turned to 180 degrees
- moved R17 165.9 mm to (64.0, 132.3), turned to 270 degrees
- moved R89 164.6 mm to (103.0, 122.8), turned to 180 degrees
- moved R59 163.3 mm to (103.5, 73.5), turned to 180 degrees
- moved R92 163.0 mm to (103.1, 116.7), turned to 180 degrees
- moved R64 162.1 mm to (103.3, 92.0), turned to 180 degrees
- moved R61 160.0 mm to (103.3, 98.2), turned to 180 degrees
- moved R91 157.1 mm to (103.3, 104.2), turned to 180 degrees
- moved D19 155.9 mm to (64.0, 133.9), turned to 270 degrees
- moved C32 151.9 mm to (69.5, 90.2)
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Connections:
- C22 pad 2: Net-(C22-Pad2) -> +5V
- C23 pad 2: Net-(C23-Pad2) -> +5V
- C33 pad 2: Net-(C33-Pad2) -> +5V
- C34 pad 2: Net-(C34-Pad2) -> +5V
- J11 pad 2: Net-(C22-Pad2) -> +5V
- J12 pad 2: Net-(C23-Pad2) -> +5V
- J13 pad 2: Net-(C33-Pad2) -> +5V
- J14 pad 2: Net-(C34-Pad2) -> +5V
Routing:
- net +12P: track 84.6 -> 156.6 mm, vias 9 -> 15
- net Net-(D56-Pad1): track 4.88 -> 40.6 mm
- net MOTOR_Batt: track 9.32 -> 29.9 mm
- net /Motor5L: track 0.00 -> 8.19 mm, vias 18 -> 20
- net /Motor4R: track 0.00 -> 8.12 mm, vias 18 -> 20
- net /Motor5R: track 0.00 -> 8.10 mm, vias 18 -> 20
- net /Motor4L: track 0.00 -> 7.96 mm, vias 18 -> 20
- net /Motor3R: track 2.02 -> 8.05 mm, vias 18 -> 20
- net /Motor3L: track 2.02 -> 8.05 mm, vias 18 -> 20
- net /Motor2R: track 2.02 -> 8.01 mm, vias 18 -> 20
- net /Motor2L: track 2.02 -> 8.00 mm, vias 18 -> 20
- net Net-(R104-Pad2): track 0.00 -> 3.44 mm, vias 0 -> 1
- net Net-(R100-Pad2): track 0.00 -> 3.44 mm, vias 0 -> 1
- net Net-(R101-Pad2): track 0.00 -> 3.43 mm, vias 0 -> 1
- net Net-(R105-Pad2): track 0.00 -> 3.43 mm, vias 0 -> 1
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- added copper zone on F.Cu, net /Motor3L
- added copper zone on F.Cu, net /Motor3R
- added copper zone on F.Cu, net /Motor4L
- added copper zone on F.Cu, net /Motor4R
- added copper zone on F.Cu, net /Motor5L
- added copper zone on F.Cu, net /Motor5R
Other:
- board text added: "ACT"
