File: 2020/Robot_Lancer/Aqualius_Sadalmeric/Main/Main.sch (KiCad schematic (older format))
At the start: 320 parts, among them J1 SERIAL0, J10 I/O_Vdd, J11 ENC0, J12 ENC1, J13 ENC2, J14 ENC3, J15 5Vin, J16 EMERGENCY, J17 MOTOR0, J18 MOTOR1, J19 MOTOR2, J2 ADC, J20 MOTOR3, J21 MOTOR4, J22 MOTOR5, J23 BATT_IN, J24 BATT_IN, J25 FUSE, J3 SWD, J4 CAN, J5 ADC_Vdd, J6 SERIAL1, J7 CAN, J8 I/O, J9 SERIAL2, Q1 NPN, Q10 NVMFD5C446NLT1G, Q11 FET_N, Q12 NVMFD5C446NLT1G, Q13 NVMFD5C446NLT1G, Q14 NVMFD5C446NLT1G, Q15 NVMFD5C446NLT1G, Q16 NVMFD5C446NLT1G, Q17 NVMFD5C446NLT1G, Q18 FET_P, Q2 NPN, Q3 FET_P, Q4 FET_P, Q5 NVMFD5C446NLT1G, Q6 NVMFD5C446NLT1G, Q7 NVMFD5C446NLT1G, Q8 NVMFD5C446NLT1G, Q9 NVMFD5C446NLT1G, SW1 RESET, SW2 DIP_SW, SW3 SW0, SW4 SW1, SW5 Control-Power_SW, SW6 SW2, SW7 SW3, SW8 EMERGENCY_SW, SW9 MAIN_SW, U1 MAX3051, U10 BD9G101G, U11 CCG30-24-12, U12 NCP5104, U13 NCP5104, U14 NCP5104, U15 NCP5104, U16 NCP5104, U17 NCP5104, U18 V23086-C1001, U19 NCP5104, U2 AP3211, U20 NCP5104, U21 NCP5104, U22 NCP5104, U23 NCP5104, U24 NCP5104, U25 LOGO, U26 7805, U3 MCP2221A, U4 AQM1602_BL, U5 AZ1086H, U6 STM32F407VG, U7 OSTBABS4C2B, U8 ADRESS, U9 25LC010A, Y1 8MHz

Commit message: いい感じじゃね
Parts:
- C52: value 470u -> 220u; footprint Capacitor_THT:CP_Radial_D10.0mm_P5.00mm -> Capacitor_THT:CP_Radial_D8.0mm_P3.50mm
- C60, C61: footprint Capacitor_THT:CP_Radial_D10.0mm_P5.00mm -> Mizz_lib:CAPAE1300X1400N
- R8: value R -> 50k
- R9: value R -> 10k
- gave numbers to parts that had none: 2
Changed lines of the file:
@@
 P 15400 1300
 F 0 "C52" H 15515 1346 50  0000 L CNN
-F 1 "470u" H 15515 1255 50  0000 L CNN
-F 2 "Capacitor_THT:CP_Radial_D10.0mm_P5.00mm" H 15400 1300 50  0001 C CNN
+F 1 "220u" H 15515 1255 50  0000 L CNN
+F 2 "Capacitor_THT:CP_Radial_D8.0mm_P3.50mm" H 15400 1300 50  0001 C CNN
 F 3 "~" H 15400 1300 50  0001 C CNN
 	1    15400 1300
@@
 F 0 "C61" H 20365 4196 50  0000 L CNN
 F 1 "470u" H 20365 4105 50  0000 L CNN
-F 2 "Capacitor_THT:CP_Radial_D10.0mm_P5.00mm" H 20250 4150 50  0001 C CNN
+F 2 "Mizz_lib:CAPAE1300X1400N" H 20250 4150 50  0001 C CNN
 F 3 "~" H 20250 4150 50  0001 C CNN
 	1    20250 4150
@@
 F 0 "C60" H 19965 4196 50  0000 L CNN
 F 1 "470u" H 19965 4105 50  0000 L CNN
-F 2 "Capacitor_THT:CP_Radial_D10.0mm_P5.00mm" H 19850 4150 50  0001 C CNN
+F 2 "Mizz_lib:CAPAE1300X1400N" H 19850 4150 50  0001 C CNN
 F 3 "~" H 19850 4150 50  0001 C CNN
 	1    19850 4150
@@
 P 3300 975
 F 0 "R8" H 3370 1021 50  0000 L CNN
-F 1 "R" H 3370 930 50  0000 L CNN
+F 1 "50k" H 3370 930 50  0000 L CNN
 F 2 "Resistor_SMD:R_0603_1608Metric" V 3230 975 50  0001 C CNN
 F 3 "~" H 3300 975 50  0001 C CNN
@@
 P 3300 1275
 F 0 "R9" H 3370 1321 50  0000 L CNN
-F 1 "R" H 3370 1230 50  0000 L CNN
+F 1 "10k" H 3370 1230 50  0000 L CNN
 F 2 "Resistor_SMD:R_0603_1608Metric" V 3230 1275 50  0001 C CNN
 F 3 "~" H 3300 1275 50  0001 C CNN
@@
 $EndComp
 $Comp
-L power:+12V #PWR?
+L power:+12V #PWR0243
 U 1 1 5E15667F
 P 1275 1900
-F 0 "#PWR?" H 1275 1750 50  0001 C CNN
+F 0 "#PWR0243" H 1275 1750 50  0001 C CNN
 F 1 "+12V" H 1290 2073 50  0000 C CNN
 F 2 "" H 1275 1900 50  0001 C CNN
@@
 $EndComp
 $Comp
-L Device:C C?
+L Device:C C76
 U 1 1 5DEFD7AA
 P 20650 4150
-F 0 "C?" H 20765 4196 50  0000 L CNN
+F 0 "C76" H 20765 4196 50  0000 L CNN
 F 1 "4.7u" H 20765 4105 50  0000 L CNN
 F 2 "Capacitor_SMD:C_0805_2012Metric" H 20688 4000 50  0001 C CNN
@@
 $EndComp
 $Comp
-L Device:C C?
+L Device:C C77
 U 1 1 5DEFE212
 P 21025 4150
-F 0 "C?" H 21140 4196 50  0000 L CNN
+F 0 "C77" H 21140 4196 50  0000 L CNN
 F 1 "4.7u" H 21140 4105 50  0000 L CNN
 F 2 "Capacitor_SMD:C_0805_2012Metric" H 21063 4000 50  0001 C CNN

Commit message: ブートストラップコンデンサ並べた,進捗git add -Agit add -A
Parts:
- removed R10, R26: 10, Resistor_SMD:R_0603_1608Metric, symbol Device:R
- removed SW2: DIP_SW, Mizz_lib:KHS4, symbol Switch:SW_DIP_x04
- added SW10: TOGGLESW1, Mizz_lib:2MS1-T1-B4-VS2-Q-E, symbol Switch:SW_DPDT_x2
- added SW11: TOGGLESW2, Mizz_lib:2MS1-T1-B4-VS2-Q-E, symbol Switch:SW_DPDT_x2
- added SW12: TOGGLESW3, Mizz_lib:2MS1-T1-B4-VS2-Q-E, symbol Switch:SW_DPDT_x2
- added SW2: TOGGLESW0, Mizz_lib:2MS1-T1-B4-VS2-Q-E, symbol Switch:SW_DPDT_x2
- C20: footprint Capacitor_SMD:C_0603_1608Metric -> Capacitor_SMD:C_0805_2012Metric
- J4, J7: footprint Mizz_lib:XA_4L -> Mizz_lib:XA_4P
- SW1: footprint Button_Switch_SMD:SW_SPST_PTS645 -> Button_Switch_SMD:SW_SPST_PTS810
- SW3, SW4, SW6, SW7: footprint Button_Switch_SMD:SW_SPST_CK_RS282G05A3 -> Button_Switch_SMD:SW_SPST_PTS810
- U4: value AQM1602_BL -> AQM0802_BL; footprint Mizz_lib:AQM1602_BL_Fad -> Mizz_lib:AQM0802_LED
Connections:
- net +3V3: now also R39.2, R42.2, R45.2, R46.2
- net GND: now also SW10.3 (C), SW11.3 (C), SW12.3 (C), SW2.3 (C); no longer R39.1, R42.1, R45.1, R46.1
- net PB8_Buzzer_TIM10_CH1: now also Q1.1 (B)
- net PB9_LCD_BL_TIM11_CH1: now also Q2.1 (B)
- net PD2_DIPSW_0: now also R46.1, SW2.2 (B); no longer R46.2
- net PD3_DIPSW_1: now also R39.1, SW10.2 (B); no longer R45.2
- net PD4_DIPSW_2: now also R42.1, SW11.2 (B); no longer R42.2
- net PD6_DIPSW_3: now also R45.1, SW12.2 (B); no longer R39.2
- no-connect marks 10 -> 14
Other:
- moved on the sheet: R46, U8

Commit message: CAN通信の終端抵抗のジャンパー抵抗部分を忘れていた.追加,進捗git add -Agit add -A
Parts:
- added JP3: CAN_JP, Connector_PinHeader_2.54mm:PinHeader_1x02_P2.54mm_Vertical, symbol Device:Jumper
- added R10: 120, Resistor_SMD:R_0603_1608Metric, symbol Device:R
- U1: footprint Package_SO:SOIC-8_3.9x4.9mm_P1.27mm -> Package_SO:TSSOP-8_3x3mm_P0.65mm
Connections:
- net CAN_H: now also JP3.1
- net CAN_L: now also R10.2
- new net: JP3.2, R10.1
Changed lines of the file:
@@
 F 0 "U1" H 1975 11931 50  0000 C CNN
 F 1 "MAX3051" H 1975 11840 50  0000 C CNN
-F 2 "Package_SO:SOIC-8_3.9x4.9mm_P1.27mm" H 1975 11350 50  0001 C CIN
+F 2 "Package_SO:TSSOP-8_3x3mm_P0.65mm" H 1975 11350 50  0001 C CIN
 F 3 "http://datasheets.maximintegrated.com/en/ds/MAX3051.pdf" H 1975 11350 50  0001 C CNN
 	1    1975 11350
@@
 Wire Wire Line
 	10700 13225 10725 13225
+$Comp
+L Device:Jumper JP3
+U 1 1 5E02D870
+P 2900 12000
+F 0 "JP3" H 2900 12225 50  0000 C CNN
+F 1 "CAN_JP" H 2900 12150 50  0000 C CNN
+F 2 "Connector_PinHeader_2.54mm:PinHeader_1x02_P2.54mm_Vertical" H 2900 12000 50  0001 C CNN
+F 3 "~" H 2900 12000 50  0001 C CNN
+	1    2900 12000
+	1    0    0    -1
+$EndComp
+Text Label 2600 12000 2    50   ~ 0
+CAN_H
+$Comp
+L Device:R R10
+U 1 1 5E0337D1
+P 3350 12000
+F 0 "R10" V 3557 12000 50  0000 C CNN
+F 1 "120" V 3466 12000 50  0000 C CNN
+F 2 "Resistor_SMD:R_0603_1608Metric" V 3280 12000 50  0001 C CNN
+F 3 "~" H 3350 12000 50  0001 C CNN
+	1    3350 12000
+	0    -1   -1   0
+$EndComp
+Text Label 3500 12000 0    50   ~ 0
+CAN_L
 $EndSCHEMATC

Commit message: バックアップ
Connections:
- net +12P: now also C62.1, C63.1, C64.1, C65.1, C66.1, C67.1, D50.2 (A), D51.2 (A), D52.2 (A), D53.2 (A), D54.2 (A), D55.2 (A), R88.1, R89.1, R90.1, R91.1, R92.1, R93.1, U19.1 (Vcc), U20.1 (Vcc), U21.1 (Vcc), U22.1 (Vcc), U23.1 (Vcc), U24.1 (Vcc)
- net +3V3: now also SW10.1 (A), SW11.1 (A), SW12.1 (A), SW2.1 (A); no longer R39.2, R42.2, R45.2, R46.2
- net GND: now also R39.1, R42.1, R45.1, R46.1; no longer SW10.3 (C), SW11.3 (C), SW12.3 (C), SW2.3 (C)
- net MOTOR_Batt: no longer C62.1, C63.1, C64.1, C65.1, C66.1, C67.1, D50.2 (A), D51.2 (A), D52.2 (A), D53.2 (A), D54.2 (A), D55.2 (A), R88.1, R89.1, R90.1, R91.1, R92.1, R93.1, U19.1 (Vcc), U20.1 (Vcc), U21.1 (Vcc), U22.1 (Vcc), U23.1 (Vcc), U24.1 (Vcc)
- net PD2_DIPSW_0: now also R46.2; no longer R46.1
- net PD3_DIPSW_1: now also R39.2; no longer R39.1
- net PD4_DIPSW_2: now also R42.2; no longer R42.1
- net PD6_DIPSW_3: now also R45.2; no longer R45.1
- net POWER_Batt: no longer SW9.2 (B)
- net at D49.2 (K), Q18.3 (S): now also SW9.2 (B)
- no-connect marks 14 -> 13
Other:
- moved on the sheet: D49, R39, R42, R45, R46

Commit message: Aloe
Parts:
- removed D1, D10, D13, D21, D22, D25, D26, D7: DIODE, Diode_SMD:D_SOD-123, symbol Miz:DIODE_rev
- added D1: LED0, LED_SMD:LED_0603_1608Metric, symbol Device:LED
- added D10: LED3, LED_SMD:LED_0603_1608Metric, symbol Device:LED
- added D11: LED4, LED_SMD:LED_0603_1608Metric, symbol Device:LED
- added D13: LED5, LED_SMD:LED_0603_1608Metric, symbol Device:LED
- added D2: LED1, LED_SMD:LED_0603_1608Metric, symbol Device:LED
- added D21: LED6, LED_SMD:LED_0603_1608Metric, symbol Device:LED
- added D22: LED7, LED_SMD:LED_0603_1608Metric, symbol Device:LED
- added D7: LED2, LED_SMD:LED_0603_1608Metric, symbol Device:LED
- added JP4: VALVE_JP, Jumper:SolderJumper-3_P1.3mm_Open_RoundedPad1.0x1.5mm, symbol Device:Jumper_NC_Dual
- added R106, R107, R108, R109, R26, R84, R85, R86: 330, Resistor_SMD:R_0603_1608Metric, symbol Device:R
- added U27: TBD62083A, Package_SO:SOIC-18W_7.5x11.6mm_P1.27mm, symbol Miz:TBD62083A
Connections:
- net +12V: now also JP4.1
- net +3V3: now also C7.2, J5.1 (Pin_1), J5.11 (Pin_11), J5.13 (Pin_13), J5.15 (Pin_15), J5.17 (Pin_17), J5.19 (Pin_19), J5.3 (Pin_3), J5.5 (Pin_5), J5.7 (Pin_7), J5.9 (Pin_9)
- net +5V: now also C22.2, C23.2, C33.2, C34.2, C5.1, C9.1, J1.2 (Pin_2), J11.2 (Pin_2), J12.2 (Pin_2), J13.2 (Pin_2), J14.2 (Pin_2), J6.2 (Pin_2), JP4.3
- net GND: now also D1.1 (K), D10.1 (K), D11.1 (K), D13.1 (K), D2.1 (K), D21.1 (K), D22.1 (K), D7.1 (K), U27.9 (GND)
- net PA11_IO: now also R108.2, U27.7 (IN7); no longer J8.7 (Pin_7)
- net PA12_IO: now also R109.2, U27.8 (IN8); no longer J8.8 (Pin_8)
- net PA4_IO: now also R106.2, U27.5 (IN5); no longer J8.5 (Pin_5)
- net PA8_IO: now also R107.2, U27.6 (IN6); no longer J8.6 (Pin_6)
- net PE0_IO: now also R26.2, U27.1 (IN1); no longer J8.1 (Pin_1)
- net PE12_IO: now also R85.2, U27.3 (IN3); no longer J8.3 (Pin_3)
- net PE15_IO: now also R86.2, U27.4 (IN4); no longer J8.4 (Pin_4)
- net PE1_IO: now also R84.2, U27.2 (IN2); no longer J8.2 (Pin_2)
- net Valve_Vdd: now reaches C12.2, J10.1 (Pin_1), J10.11 (Pin_11), J10.13 (Pin_13), J10.15 (Pin_15), J10.3 (Pin_3), J10.5 (Pin_5), J10.7 (Pin_7), J10.9 (Pin_9)
- net Valve_Vdd: now also JP4.2, U27.10 (COM)
- new net: J8.8 (Pin_8), U27.11 (OUT8)
- new net: J8.7 (Pin_7), U27.12 (OUT7)
- new net: J8.6 (Pin_6), U27.13 (OUT6)
- new net: J8.5 (Pin_5), U27.14 (OUT5)
- new net: J8.4 (Pin_4), U27.15 (OUT4)
- new net: J8.3 (Pin_3), U27.16 (OUT3)
- new net: J8.2 (Pin_2), U27.17 (OUT2)
- new net: J8.1 (Pin_1), U27.18 (OUT1)
- new net: D1.2 (A), R26.1
- new net: D2.2 (A), R84.1
- new net: D7.2 (A), R85.1
- new net: D10.2 (A), R86.1
- new net: D11.2 (A), R106.1
- new net: D13.2 (A), R107.1
- new net: D21.2 (A), R108.1
- new net: D22.2 (A), R109.1
Other:
- moved on the sheet: C12, C19, C5, C7, C9, D15, D17, D18, D19, J1, J10, J2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
