File: 2020/Robot_Lancer/Aqualius_Sadalmeric/Main.sch (KiCad schematic (older format))
At the start: 333 parts, among them J1 SERIAL0, J10 I/O_Vdd, J11 ENC0, J12 ENC1, J13 ENC2, J14 ENC3, J15 5Vin, J16 EMERGENCY, J17 MOTOR0, J18 MOTOR1, J19 MOTOR2, J2 ADC, J20 MOTOR3, J21 MOTOR4, J22 MOTOR5, J23 BATT_IN, J24 BATT_IN, J25 FUSE, J3 SWD, J4 CAN, J5 ADC_Vdd, J6 SERIAL1, J7 CAN, J8 I/O, J9 SERIAL2, Q1 NPN, Q10 NVMFD5C446NLT1G, Q11 FET_N, Q12 NVMFD5C446NLT1G, Q13 NVMFD5C446NLT1G, Q14 NVMFD5C446NLT1G, Q15 NVMFD5C446NLT1G, Q16 NVMFD5C446NLT1G, Q17 NVMFD5C446NLT1G, Q18 FET_P, Q2 NPN, Q3 FET_P, Q4 FET_P, Q5 NVMFD5C446NLT1G, Q6 NVMFD5C446NLT1G, Q7 NVMFD5C446NLT1G, Q8 NVMFD5C446NLT1G, Q9 NVMFD5C446NLT1G, SW1 RESET, SW10 TOGGLESW1, SW11 TOGGLESW2, SW12 TOGGLESW3, SW2 TOGGLESW0, SW3 SW0, SW4 SW1, SW5 Control-Power_SW, SW6 SW2, SW7 SW3, SW8 EMERGENCY_SW, SW9 MAIN_SW, U1 MAX3051, U10 BD9G101G, U11 CCG30-24-12, U12 NCP5104, U13 NCP5104, U14 NCP5104, U15 NCP5104, U16 NCP5104, U17 NCP5104, U18 V23086-C1001, U19 NCP5104, U2 AP3211, U20 NCP5104, U21 NCP5104, U22 NCP5104, U23 NCP5104, U24 NCP5104, U25 LOGO, U26 7805, U27 TBD62083A, U3 MCP2221A, U4 AQM0802_BL, U5 AZ1086H, U6 STM32F407VG, U7 OSTBABS4C2B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

Commit message: ランサー基板,配置のみ完
Parts:
- removed D37: LED, LED_SMD:LED_0603_1608Metric, symbol Device:LED
- removed Q2: NPN, Package_TO_SOT_SMD:SOT-23W, symbol Device:Q_NPN_BEC
- removed R39, R41, R42, R44, R45, R46, R48, R50: 10k, Resistor_SMD:R_0603_1608Metric, symbol Device:R
- removed R66: 2.2k, Resistor_SMD:R_0603_1608Metric, symbol Device:R
- removed U4: AQM0802_BL, Mizz_lib:AQM0802_LED, symbol Main-rescue:AQM0802_BL-Miz
- added D25: RESET, LED_SMD:LED_0603_1608Metric, symbol Device:LED
- added U4: AQM0802, Mizz_lib:AQM0802, symbol Miz:AQM1602
- J8: value I/O -> VALVE
- R27: value 120 -> 240
- U27: footprint Package_SO:SOIC-18W_7.5x11.6mm_P1.27mm -> Package_SO:SSOP-18_4.4x6.5mm_P0.65mm
Connections:
- net +3V3: now also U4.5 (VDD), U4.9 (/RST); no longer SW10.1 (A), SW11.1 (A), SW12.1 (A), SW2.1 (A)
- net Control_5V: no longer R1.2
- net External_5V: now also R1.2
- net GND: now also SW10.3 (C), SW11.3 (C), SW12.3 (C), SW2.3 (C), D25.1 (K), U4.6 (VSS)
- net PB6_I2C1_SCL: now also U4.8 (SCL)
- net PB7_I2C1_SDA: now also U4.7 (SDA)
- net PB9_LCD_BL_TIM11_CH1: now also R27.2
- net at R27.1: now also D25.2 (A)
- net at C26.1: now also U4.2 (VOUT)
- net at C27.1: now also U4.3 (CAP1N)
- net at C27.2: now also U4.4 (CAP1P)
- no-connect marks 13 -> 14
