File: 2020/Robot_Lancer/Aqualius_Sadalmeric/Main.sch (KiCad schematic (older format))
At the start: 323 parts, among them J1 SERIAL0, J10 I/O_Vdd, J11 ENC0, J12 ENC1, J13 ENC2, J14 ENC3, J15 5Vin, J16 EMERGENCY, J17 MOTOR0, J18 MOTOR1, J19 MOTOR2, J2 ADC, J20 MOTOR3, J21 MOTOR4, J22 MOTOR5, J23 BATT_IN, J24 BATT_IN, J25 FUSE, J3 SWD, J4 CAN, J5 ADC_Vdd, J6 SERIAL1, J7 CAN, J8 VALVE, J9 SERIAL2, Q1 NPN, Q10 NVMFD5C446NLT1G, Q11 FET_N, Q12 NVMFD5C446NLT1G, Q13 NVMFD5C446NLT1G, Q14 NVMFD5C446NLT1G, Q15 NVMFD5C446NLT1G, Q16 NVMFD5C446NLT1G, Q17 NVMFD5C446NLT1G, Q18 FET_P, Q3 FET_P, Q4 FET_P, Q5 NVMFD5C446NLT1G, Q6 NVMFD5C446NLT1G, Q7 NVMFD5C446NLT1G, Q8 NVMFD5C446NLT1G, Q9 NVMFD5C446NLT1G, SW1 RESET, SW10 TOGGLESW1, SW11 TOGGLESW2, SW12 TOGGLESW3, SW2 TOGGLESW0, SW3 SW0, SW4 SW1, SW5 Control-Power_SW, SW6 SW2, SW7 SW3, SW8 EMERGENCY_SW, SW9 MAIN_SW, U1 MAX3051, U10 BD9G101G, U11 CCG30-24-12, U12 NCP5104, U13 NCP5104, U14 NCP5104, U15 NCP5104, U16 NCP5104, U17 NCP5104, U18 V23086-C1001, U19 NCP5104, U2 AP3211, U20 NCP5104, U21 NCP5104, U22 NCP5104, U23 NCP5104, U24 NCP5104, U25 LOGO, U26 7805, U27 TBD62083A, U3 MCP2221A, U4 AQM0802, U5 AZ1086H, U6 STM32F407VG, U7 OSTBABS4C2B, U8 ADRESS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

Commit message: ALoe
Parts:
- removed D49: SBR_DIODE, Diode_SMD:D_SMB_Modified, symbol Device:D_Schottky_AKA
- added D26: DIODE, Diode_SMD:D_SMA, symbol pspice:DIODE
Connections:
- net +BATT: now also D26.1 (K)
- net at Q18.3 (S), SW9.2 (B): now also D26.2 (A)
Changed lines of the file:
@@
 	1    0    0    -1
 $EndComp
-Text GLabel 17225 825  0    50   Input ~ 0
-POWER_Batt
 $Comp
 L Device:Q_NMOS_GDS Q11
@@
 	18425 1425 18300 1425
 Wire Wire Line
-	17225 825  17275 825
-Wire Wire Line
-	17275 725  17275 825
-Connection ~ 17275 825
-Wire Wire Line
 	17575 2650 17575 2975
 Wire Wire Line
@@
 	16300 775  16500 775
 Connection ~ 16500 775
-$Comp
-L Device:D_Schottky_AKA D49
-U 1 1 5E4A3FBF
-P 17475 825
-F 0 "D49" H 17500 1106 50  0000 C CNN
-F 1 "SBR_DIODE" H 17500 1015 50  0000 C CNN
-F 2 "Diode_SMD:D_SMB_Modified" H 17475 825 50  0001 C CNN
-F 3 "~" H 17475 825 50  0001 C CNN
-	1    17475 825
-	-1   0    0    -1
-$EndComp
 Wire Wire Line
 	15350 1000 15800 1000
@@
 Wire Wire Line
 	17625 825  18425 825
-Connection ~ 17625 825
 Connection ~ 5975 14300
 Connection ~ 5975 15300
@@
 Text Label 12100 4275 0    50   ~ 0
 PE12_IO
+$Comp
+L power:+BATT #PWR0223
+U 1 1 5DEF531D
+P 17150 825
+F 0 "#PWR0223" H 17150 675 50  0001 C CNN
+F 1 "+BATT" H 17165 998 50  0000 C CNN
+F 2 "" H 17150 825 50  0001 C CNN
+F 3 "" H 17150 825 50  0001 C CNN
+	1    17150 825
+	1    0    0    -1
+$EndComp
+$Comp
+L pspice:DIODE D26
+U 1 1 5DF6A377
+P 17425 825
+F 0 "D26" H 17425 1090 50  0000 C CNN
+F 1 "DIODE" H 17425 999 50  0000 C CNN
+F 2 "Diode_SMD:D_SMA" H 17425 825 50  0001 C CNN
+F 3 "~" H 17425 825 50  0001 C CNN
+	1    17425 825
+	1    0    0    -1
+$EndComp
+Connection ~ 17625 825
+Wire Wire Line
+	17150 825  17225 825
 $EndSCHEMATC

Commit message: 2019/12/09
Parts:
- removed C5: 0.1u, Capacitor_SMD:C_0603_1608Metric, symbol Device:C
- removed J1: SERIAL0, Mizz_lib:XA_4P, symbol Connector_Generic:Conn_01x04
- removed R54, R55, R56: 10, Resistor_SMD:R_0603_1608Metric, symbol Device:R
- removed U9: 25LC010A, Package_DIP:DIP-8_W7.62mm_Socket, symbol Miz:25LC010A
- added C78: 1u, Capacitor_SMD:C_0603_1608Metric, symbol Device:C
- added C79, C80: 0.1u, Capacitor_SMD:C_0603_1608Metric, symbol Device:C
- added D37: DATA, symbol Device:LED
- added D49: COMM, symbol Device:LED
- added D58: DIODE, Diode_SMD:D_SOD-123, symbol Miz:DIODE_rev
- added J26: Micro_SD_Card, symbol Connector:Micro_SD_Card
- added J27: USB_A, Mizz_lib:USB_A_Vertical, symbol Connector:USB_A
- added J28: PICkit3, Mizz_lib:ZH_6P, symbol Connector_Generic:Conn_01x06
- added JP5: PIKkit_Vdd, Mizz_lib:GS2, symbol Device:Jumper
- added R39: 10, Resistor_SMD:R_0603_1608Metric, symbol Device:R
- added R41: 10k, Resistor_SMD:R_0603_1608Metric, symbol Device:R
- added R42, R44: 330, Resistor_SMD:R_0603_1608Metric, symbol Device:R
- added U9: PIC24FJ32GB004, Package_QFP:LQFP-44_10x10mm_P0.8mm, symbol Miz:PIC24FJ32GB004-pic24fjxxgb
- J6: value SERIAL1 -> SERIAL0
Connections:
- net +3V3: now also C79.1, C80.1, J26.4 (VDD), R41.2, R42.1, R44.1, U9.10 (Vusb), U9.17 (AVdd), U9.28 (Vdd), U9.40 (Vdd)
- net +5V: now also J27.1 (VBUS), U9.42 (Vbus)
- net GND: now also C78.2, C79.2, C80.2, J26.6 (VSS), J27.4 (GND), J28.3 (Pin_3), U9.16 (AVss), U9.29 (Vss), U9.39 (Vss), U9.6 (DISVREG)
- net PA10_USART1_RX: now also U9.2 (RP22_CN18_RC6)
- net PA4_IO: no longer R106.2, U6.29 (PA4/SPI1_NSS/SPI3_NSS/USART2_CK/DCMI_HSYNC/OTG_HS_SOF/I2S3_WS/EVENTOUT)
- net PA5_SPI1_SCK: now also J26.5 (CLK)
- net PA6_SPI1_MISO: now also J26.7 (DAT0)
- net PA7_SPI1_MOSI: now also J26.3 (CMD)
- net PA9_USART1_TX: now also U9.3 (RP23_CN17_RC7)
- new net: D37.1 (K), U9.14 (AN10_C3INB_CVref_VBUSON_RP14_CN12_RB14)
- new net: D49.1 (K), U9.15 (AN9_C3INA_VBUSCHG_RP15_CN11_RB15)
- new net: C78.1, U9.7 (Vcap_VddCore)
- new net: D49.2 (A), R44.2
- new net: D37.2 (A), R42.2
- new net: D58.2 (A), J28.2 (Pin_2)
- new net: D58.1 (K), JP5.1
- new net MCLR: J28.1 (Pin_1), R41.1, U9.18 (MCLR)
- new net PA4_SPI1_NSS: J26.2 (DAT3/CD), U6.29 (PA4/SPI1_NSS/SPI3_NSS/USART2_CK/DCMI_HSYNC/OTG_HS_SOF/I2S3_WS/EVENTOUT)
- new net PGEC1: J28.5 (Pin_5), U9.22 (PGEDC1_AN3_C2INA_RP1_CN5_RB1)
- new net PGED1: J28.4 (Pin_4), U9.21 (PGED1_AN2_C2INB_RP0_CN4_RB0)
- new net USB_A_D+: J27.3 (D+), U9.8 (PGED2_D+_RP10_CN16_RB10)
- new net USB_A_D-: J27.2 (D-), U9.9 (PGEC2_D-_RP11_CN15_RB11)
- no-connect marks 14 -> 40
Other:
- moved on the sheet: C10, C12, C19, C25, C26, C27, C36, C37, C38, C39, C4, C6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

Commit message: back up
Parts:
- removed J26: Micro_SD_Card, symbol Connector:Micro_SD_Card
- added J1: microSD, Connector_Card:microSD_HC_Hirose_DM3AT-SF-PEJM5, symbol Connector:Micro_SD_Card_Det_Hirose_DM3AT
- added R45, R54, R55, R56, R66: 10k, Resistor_SMD:R_0603_1608Metric, symbol Device:R
- added R46, R48, R50: FILTER, Resistor_SMD:R_0603_1608Metric, symbol Device:R
- added U28: LOGO, Mizz_lib:Aqualius_Sadalmeric_silk_40x9.4, symbol Miz:LOGO
- D37, D49: footprint (none) -> LED_SMD:LED_0603_1608Metric
- J11: value ENC0 -> ENC1
- J12: value ENC1 -> ENC0
- J13: value ENC2 -> ENC3
- J14: value ENC3 -> ENC2
- J27: value USB_A -> Advanced_SBDBT
- R100, R101, R102, R103, R104, R105, R69, R70, R71, R72, R73, R74, R75, R76, R77, R78, R79, R80, R94, R95, R96, R97, R98, R99: value 3 -> FILTER
- R39: value 10 -> FILTER
Connections:
- net +3V3: now also JP5.2, J1.4 (VDD), R45.2, R54.2, R55.2, R56.2, R66.2
- net GND: now also J1.10 (DET_A), J1.6 (VSS)
- net PA2_ADC12_IN2: now also J2.5 (Pin_5); no longer J2.9 (Pin_9)
- net PA3_ADC12_IN3: now also J2.6 (Pin_6); no longer J2.10 (Pin_10)
- net PA4_SPI1_NSS: now also R46.2
- net PA5_SPI1_SCK: now also R50.2
- net PA6_SPI1_MISO: now also R39.2
- net PA7_SPI1_MOSI: now also R48.2
- net PB0_ADC12_IN8: now also J2.9 (Pin_9); no longer J2.7 (Pin_7)
- net PB1_ADC12_IN9: now also J2.10 (Pin_10); no longer J2.8 (Pin_8)
- net PB2_ROM_~WP: no longer U6.37 (PB2/BOOT1/EVENTOUT)
- net PC4_ADC12_IN14: now also J2.7 (Pin_7); no longer J2.5 (Pin_5)
- net PC5_ADC12_IN15: now also J2.8 (Pin_8); no longer J2.6 (Pin_6)
- net SW0: now also R54.1
- net SW1: now also R55.1
- net SW2: now also R56.1
- net SW3: now also R66.1
- net at R39.1: now also J1.7 (DAT0)
- net PE7_ROM_~CS renamed PE7_SD_Connection
- net PE8_ROM_~HOLD renamed PE8
- new net: J1.2 (DAT3/CD), R46.1
- new net: J1.3 (CMD), R48.1
- new net: J1.5 (CLK), R50.1
- new net PB2_SD_Connection: J1.9 (DET_B), R45.1, U6.37 (PB2/BOOT1/EVENTOUT)
- no-connect marks 40 -> 43
Other:
- moved on the sheet: R39
