File: 2020/Robot_Lancer/Aqualius_Sadalmeric/Main.kicad_pcb (KiCad board)
At the start: 2 copper layers, 100 x 100 mm, 319 parts, among them J1 SERIAL0, J10 I/O_Vdd, J11 ENC0, J12 ENC1, J13 ENC2, J14 ENC3, J15 5Vin, J16 EMERGENCY, J17 MOTOR0, J18 MOTOR1, J19 MOTOR2, J2 ADC, J20 MOTOR3, J21 MOTOR4, J22 MOTOR5, J23 BATT_IN, J24 BATT_IN, J25 FUSE, J3 SWD, J4 CAN, J5 ADC_Vdd, J6 SERIAL1, J7 CAN, J8 I/O, J9 SERIAL2, Q1 NPN, Q10 NVMFD5C446NLT1G, Q11 FET_N, Q12 NVMFD5C446NLT1G, Q13 NVMFD5C446NLT1G, Q14 NVMFD5C446NLT1G, Q15 NVMFD5C446NLT1G, Q16 NVMFD5C446NLT1G, Q17 NVMFD5C446NLT1G, Q18 FET_P, Q2 NPN, Q3 FET_P, Q4 FET_P, Q5 NVMFD5C446NLT1G, Q6 NVMFD5C446NLT1G, Q7 NVMFD5C446NLT1G, Q8 NVMFD5C446NLT1G, Q9 NVMFD5C446NLT1G, SW1 RESET, SW10 TOGGLESW1, SW11 TOGGLESW2, SW12 TOGGLESW3, SW2 TOGGLESW0, SW3 SW0, SW4 SW1, SW5 Control-Power_SW, SW6 SW2, SW7 SW3, SW8 EMERGENCY_SW, SW9 MAIN_SW, U1 MAX3051, U10 BD9G101G, U11 CCG30-24-12, U12 NCP5104, U13 NCP5104, U14 NCP5104, U15 NCP5104, U16 NCP5104, U17 NCP5104, U18 V23086-C1001, U19 NCP5104, U2 AP3211, U20 NCP5104, U21 NCP5104, U22 NCP5104, U23 NCP5104, U24 NCP5104, U25 LOGO, U26 7805, U3 MCP2221A, U4 AQM0802_BL, U5 AZ1086H, U6 STM32F407VG, U7 OSTBABS4C2B, U8 ADRESS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

Commit message: ランサー基板,配置のみ完
Parts:
- removed D37: LED, LED_SMD:LED_0603_1608Metric
- removed Q2: NPN, Package_TO_SOT_SMD:SOT-23W
- removed R39, R41, R42, R44, R45, R46, R48, R50: 10k, Resistor_SMD:R_0603_1608Metric
- removed R66: 2.2k, Resistor_SMD:R_0603_1608Metric
- added D11: LED4, LED_SMD:LED_0603_1608Metric, F.Cu at (46.0, 70.2)
- added D2: LED1, LED_SMD:LED_0603_1608Metric, F.Cu at (46.0, 62.5)
- added D21: LED6, LED_SMD:LED_0603_1608Metric, F.Cu at (46.0, 75.3)
- added D22: LED7, LED_SMD:LED_0603_1608Metric, F.Cu at (46.0, 77.8)
- added D25: RESET, LED_SMD:LED_0603_1608Metric, F.Cu at (48.0, 136.0)
- added JP4: VALVE_JP, Jumper:SolderJumper-3_P1.3mm_Open_RoundedPad1.0x1.5mm, B.Cu at (40.2, 57.8)
- added R106: 330, Resistor_SMD:R_0603_1608Metric, F.Cu at (48.5, 70.2)
- added R107: 330, Resistor_SMD:R_0603_1608Metric, F.Cu at (48.5, 72.8)
- added R108: 330, Resistor_SMD:R_0603_1608Metric, F.Cu at (48.5, 75.3)
- added R109: 330, Resistor_SMD:R_0603_1608Metric, F.Cu at (48.5, 77.8)
- added R26: 330, Resistor_SMD:R_0603_1608Metric, F.Cu at (48.6, 60.0)
- added R84: 330, Resistor_SMD:R_0603_1608Metric, F.Cu at (48.6, 62.5)
- added R85: 330, Resistor_SMD:R_0603_1608Metric, F.Cu at (48.5, 65.0)
- added R86: 330, Resistor_SMD:R_0603_1608Metric, F.Cu at (48.5, 67.7)
- added U27: TBD62083A, Package_SO:SSOP-18_4.4x6.5mm_P0.65mm, B.Cu at (48.2, 69.5)
- C12, C22, C23, C33, C34, C35, C37, C40, C5, C7, C9, LS1, Q11, R1, R12, R13, R14, R15, R16, R18, R19, R2, R20, R21, R22, R23, R28, R29, R3, R30, R31, R32, R33, R34, R35, R54, R55, R56, R6, R67, R68, R7, R87: moved to B.Cu
- D1: value DIODE -> LED0; footprint Diode_SMD:D_SOD-123 -> LED_SMD:LED_0603_1608Metric; moved to F.Cu
- D10: value DIODE -> LED3; footprint Diode_SMD:D_SOD-123 -> LED_SMD:LED_0603_1608Metric; moved to F.Cu
- D13: value DIODE -> LED5; footprint Diode_SMD:D_SOD-123 -> LED_SMD:LED_0603_1608Metric
- D7: value DIODE -> LED2; footprint Diode_SMD:D_SOD-123 -> LED_SMD:LED_0603_1608Metric
- J8: value I/O -> VALVE
- R27: value 120 -> 240
- R36, R37, R38: moved to F.Cu
- U4: value AQM0802_BL -> AQM0802; footprint Mizz_lib:AQM0802_LED -> Mizz_lib:AQM0802
- moved D46 252.8 mm to (91.3, 72.5)
- moved D31 250.0 mm to (84.2, 92.8), turned to 180 degrees
- moved Q11 226.3 mm to (92.7, 48.9), turned to 180 degrees
- moved D38 195.7 mm to (101.7, 44.0)
- moved D15 194.1 mm to (65.8, 128.2), turned to 270 degrees
- moved D3 169.8 mm to (73.4, 71.3), turned to 90 degrees
- moved D14 168.7 mm to (78.2, 92.7), turned to 270 degrees
- moved R55 168.0 mm to (80.5, 104.7)
- moved R87 165.6 mm to (93.1, 45.4), turned to 180 degrees
- moved R43 162.9 mm to (82.0, 87.5), turned to 180 degrees
- moved R14 162.6 mm to (65.8, 132.3), turned to 270 degrees
- moved R51 160.2 mm to (82.0, 92.8), turned to 180 degrees
- moved D17 157.8 mm to (65.8, 133.9), turned to 270 degrees
- moved R49 156.8 mm to (82.0, 91.0), turned to 180 degrees
- moved C5 156.2 mm to (73.4, 121.2)
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Connections:
- C12 pad 2: Net-(C12-Pad2) -> Valve_Vdd
- C5 pad 1: Net-(C5-Pad1) -> +5V
- C7 pad 2: Net-(C7-Pad2) -> +3V3
- C9 pad 1: Net-(C9-Pad1) -> +5V
- D1 pad 1: Net-(C5-Pad1) -> GND
- D1 pad 2: +5V -> Net-(D1-Pad2)
- D10 pad 1: Net-(C9-Pad1) -> GND
- D10 pad 2: +5V -> Net-(D10-Pad2)
- D13 pad 1: Net-(C12-Pad2) -> GND
- D13 pad 2: +5V -> Net-(D13-Pad2)
- D7 pad 1: Net-(C7-Pad2) -> GND
- D7 pad 2: +3V3 -> Net-(D7-Pad2)
- J1 pad 2: Net-(C5-Pad1) -> +5V
- J10 pad 1: Net-(C12-Pad2) -> Valve_Vdd
- J10 pad 11: Net-(C12-Pad2) -> Valve_Vdd
- J10 pad 13: Net-(C12-Pad2) -> Valve_Vdd
- J10 pad 15: Net-(C12-Pad2) -> Valve_Vdd
- J10 pad 3: Net-(C12-Pad2) -> Valve_Vdd
- J10 pad 5: Net-(C12-Pad2) -> Valve_Vdd
- J10 pad 7: Net-(C12-Pad2) -> Valve_Vdd
- J10 pad 9: Net-(C12-Pad2) -> Valve_Vdd
- J5 pad 1: Net-(C7-Pad2) -> +3V3
- J5 pad 11: Net-(C7-Pad2) -> +3V3
- J5 pad 13: Net-(C7-Pad2) -> +3V3
- J5 pad 15: Net-(C7-Pad2) -> +3V3
- J5 pad 17: Net-(C7-Pad2) -> +3V3
- J5 pad 19: Net-(C7-Pad2) -> +3V3
- J5 pad 3: Net-(C7-Pad2) -> +3V3
- J5 pad 5: Net-(C7-Pad2) -> +3V3
- J5 pad 7: Net-(C7-Pad2) -> +3V3
- J5 pad 9: Net-(C7-Pad2) -> +3V3
- J6 pad 2: Net-(C9-Pad1) -> +5V
- J8 pad 1: /PE0_IO -> Net-(J8-Pad1)
- J8 pad 2: /PE1_IO -> Net-(J8-Pad2)
- J8 pad 3: /PE12_IO -> Net-(J8-Pad3)
- J8 pad 4: /PE15_IO -> Net-(J8-Pad4)
- J8 pad 5: /PA4_IO -> Net-(J8-Pad5)
- J8 pad 6: /PA8_IO -> Net-(J8-Pad6)
- J8 pad 7: /PA11_IO -> Net-(J8-Pad7)
- J8 pad 8: /PA12_IO -> Net-(J8-Pad8)
- R1 pad 2: Control_5V -> External_5V
- R27 pad 2: Net-(R27-Pad2) -> /PB9_LCD_BL_TIM11_CH1
- SW10 pad 1: +3V3 -> Net-(SW10-Pad1)
- SW10 pad 3: Net-(SW10-Pad3) -> GND
- SW11 pad 1: +3V3 -> Net-(SW11-Pad1)
- SW11 pad 3: Net-(SW11-Pad3) -> GND
- SW12 pad 1: +3V3 -> Net-(SW12-Pad1)
- SW12 pad 3: Net-(SW12-Pad3) -> GND
- SW2 pad 1: +3V3 -> Net-(SW2-Pad1)
- SW2 pad 3: Net-(SW2-Pad3) -> GND
Routing:
- net Valve_Vdd: track 0.00 -> 33.8 mm, vias 0 -> 1
- net +5V: track 0.00 -> 24.4 mm, vias 0 -> 2
- net Control_5V: track 0.00 -> 20.3 mm, vias 0 -> 1
- net Net-(D56-Pad1): track 40.6 -> 59.7 mm, vias 0 -> 2
- net /PC0_ADC12_IN10: track 0.00 -> 18.9 mm
- net /PC1_ADC12_IN11: track 0.00 -> 16.7 mm
- net /PC3_ADC12_IN13: track 0.00 -> 16.2 mm
- net Net-(D56-Pad2): track 20.6 -> 36.3 mm
- net /PC2_ADC12_IN12: track 0.00 -> 15.6 mm
- net Net-(C13-Pad1): track 0.00 -> 11.7 mm
- net Net-(C31-Pad1): track 0.00 -> 8.91 mm, vias 0 -> 1
- net Net-(J8-Pad1): track 0.00 -> 8.62 mm
- net +12V: track 12.5 -> 20.8 mm
- net Net-(D33-Pad1): track 0.00 -> 8.28 mm, vias 0 -> 1
- net /FB_Control_OUT: track 0.00 -> 7.91 mm, vias 0 -> 1
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Other:
- board text added: "12V"
- board text added: "5V"
- board text added: "MAIN"
- board text added: "POWER_SW"
- board text removed: "7"

Commit message: アロエ
Parts:
- moved U9 24.6 mm to (50.8, 99.8)
- moved C40 24.5 mm to (56.7, 98.9), turned to 90 degrees
- moved R56 24.5 mm to (56.0, 107.4)
- moved R55 24.3 mm to (56.1, 103.8), turned to 270 degrees
- moved R37 22.6 mm to (77.0, 98.7)
- moved U7 22.6 mm to (77.0, 103.8)
- moved R36 22.6 mm to (78.5, 98.7)
- moved R38 22.6 mm to (75.3, 98.7)
- moved R54 20.0 mm to (53.5, 102.3), turned to 0 degrees
- moved U8 0.65 mm to (58.2, 114.2), turned to 270 degrees
Routing:
- net /PB1_ADC12_IN9: track 0.00 -> 27.5 mm
- net /PB0_ADC12_IN8: track 0.00 -> 24.8 mm
- net /PC5_ADC12_IN15: track 0.00 -> 22.2 mm
- net /PC4_ADC12_IN14: track 0.00 -> 20.5 mm
- net /PA12_IO: track 0.00 -> 9.26 mm, vias 0 -> 1
- net /PE0_IO: track 0.00 -> 8.05 mm, vias 0 -> 1
- net /PE1_IO: track 0.00 -> 6.09 mm, vias 0 -> 1
- net /PA11_IO: track 0.00 -> 5.58 mm, vias 0 -> 1
- net /PE12_IO: track 0.00 -> 4.28 mm, vias 0 -> 1
- net /PA8_IO: track 0.00 -> 3.67 mm, vias 0 -> 1
- net /PE15_IO: track 0.00 -> 2.47 mm, vias 0 -> 1
- net /PA4_IO: track 0.00 -> 1.95 mm, vias 0 -> 1
- net Net-(D22-Pad2): track 0.00 -> 0.88 mm
- net Net-(D21-Pad2): track 0.00 -> 0.88 mm
- net Net-(D13-Pad2): track 0.00 -> 0.88 mm
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