File: 2020/Robot_Lancer/Aqualius_Sadalmeric/Main.kicad_pcb (KiCad board)
At the start: 2 copper layers, 100 x 100 mm, 323 parts, among them J1 SERIAL0, J10 I/O_Vdd, J11 ENC0, J12 ENC1, J13 ENC2, J14 ENC3, J15 5Vin, J16 EMERGENCY, J17 MOTOR0, J18 MOTOR1, J19 MOTOR2, J2 ADC, J20 MOTOR3, J21 MOTOR4, J22 MOTOR5, J23 BATT_IN, J24 BATT_IN, J25 FUSE, J3 SWD, J4 CAN, J5 ADC_Vdd, J6 SERIAL1, J7 CAN, J8 VALVE, J9 SERIAL2, Q1 NPN, Q10 NVMFD5C446NLT1G, Q11 FET_N, Q12 NVMFD5C446NLT1G, Q13 NVMFD5C446NLT1G, Q14 NVMFD5C446NLT1G, Q15 NVMFD5C446NLT1G, Q16 NVMFD5C446NLT1G, Q17 NVMFD5C446NLT1G, Q18 FET_P, Q3 FET_P, Q4 FET_P, Q5 NVMFD5C446NLT1G, Q6 NVMFD5C446NLT1G, Q7 NVMFD5C446NLT1G, Q8 NVMFD5C446NLT1G, Q9 NVMFD5C446NLT1G, SW1 RESET, SW10 TOGGLESW1, SW11 TOGGLESW2, SW12 TOGGLESW3, SW2 TOGGLESW0, SW3 SW0, SW4 SW1, SW5 Control-Power_SW, SW6 SW2, SW7 SW3, SW8 EMERGENCY_SW, SW9 MAIN_SW, U1 MAX3051, U10 BD9G101G, U11 CCG30-24-12, U12 NCP5104, U13 NCP5104, U14 NCP5104, U15 NCP5104, U16 NCP5104, U17 NCP5104, U18 V23086-C1001, U19 NCP5104, U2 AP3211, U20 NCP5104, U21 NCP5104, U22 NCP5104, U23 NCP5104, U24 NCP5104, U25 LOGO, U26 7805, U27 TBD62083A, U3 MCP2221A, U4 AQM0802, U5 AZ1086H, U6 STM32F407VG, U7 OSTBABS4C2B, U8 ADRESS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

Commit message: アロエ
Changed lines of the file:
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@@
   )
   (gr_text Main+Power+MD*6= (at 133.25 131.75 90) (layer F.SilkS)
-    (effects (font (size 1.5 1.5) (thickness 0.375) italic) (justify left))
+    (effects (font (size 1.5 1.5) (thickness 0.3) italic) (justify left))
   )
   (dimension 3 (width 0.15) (layer Margin)
@@
   )
   (gr_text "Aquarius Sadalmelik" (at 133.25 108.5 90) (layer F.SilkS)
-    (effects (font (size 2 2) (thickness 0.5) italic) (justify left))
+    (effects (font (size 2 2) (thickness 0.4) italic) (justify left))
   )
   (gr_arc (start 133 135) (end 133 138) (angle -90) (layer Edge.Cuts) (width 0.05))

Commit message: ALoe
Parts:
- removed D49: SBR_DIODE, Diode_SMD:D_SMB_Modified
- added D26: DIODE, Diode_SMD:D_SMA, B.Cu at (109.0, 45.5)
- moved C1 15.0 mm to (58.4, 70.1), turned to 135 degrees
- moved C3 11.0 mm to (52.2, 73.8), turned to 225 degrees
- moved Y1 10.3 mm to (55.9, 73.8), turned to 225 degrees
- moved C32 7.83 mm to (62.6, 94.0), turned to 315 degrees
- moved U6 2.76 mm to (64.5, 82.7), turned to 315 degrees
- moved U25 2.72 mm to (64.5, 82.6)
Routing:
- net Batt: track 14.3 -> 42.4 mm
- net /PB1_ADC12_IN9: track 27.5 -> 0.00 mm
- net /PB0_ADC12_IN8: track 24.8 -> 0.00 mm
- net /PC5_ADC12_IN15: track 22.2 -> 0.00 mm
- net /PC4_ADC12_IN14: track 20.5 -> 0.00 mm
- net /PC0_ADC12_IN10: track 18.9 -> 0.00 mm
- net /PC1_ADC12_IN11: track 16.7 -> 0.00 mm
- net /PC3_ADC12_IN13: track 16.2 -> 0.00 mm
- net External_5V: track 3.62 -> 19.7 mm, vias 0 -> 1
- net +BATT: track 7.75 -> 23.4 mm
- net /PC2_ADC12_IN12: track 15.6 -> 0.00 mm
- net /CAN_L: track 7.66 -> 20.0 mm
- net +12V: track 20.8 -> 28.5 mm
- net /CAN_H: track 18.7 -> 24.4 mm, vias 0 -> 1
- net /FB_Control: track 0.00 -> 4.50 mm
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
Commit message: 2019/12/09
Parts:
- removed C5: 0.1u, Capacitor_SMD:C_0603_1608Metric
- removed J1: SERIAL0, Mizz_lib:XA_4P
- removed R54, R55, R56: 10, Resistor_SMD:R_0603_1608Metric
- added C78: 1u, Capacitor_SMD:C_0603_1608Metric, F.Cu at (81.0, 126.0)
- added C79: 0.1u, Capacitor_SMD:C_0603_1608Metric, B.Cu at (72.3, 118.7)
- added C80: 0.1u, Capacitor_SMD:C_0603_1608Metric, B.Cu at (74.6, 133.5)
- added D58: DIODE, Diode_SMD:D_SOD-123, F.Cu at (85.8, 159.9)
- added J27: USB_A, Mizz_lib:USB_A_Vertical, F.Cu at (84.9, 128.1)
- added J28: PICkit3, Mizz_lib:ZH_6P, F.Cu at (64.3, 129.3)
- added JP5: PIKkit_Vdd, Mizz_lib:GS2, F.Cu at (84.4, 168.4)
- added R39: 10, Resistor_SMD:R_0603_1608Metric, F.Cu at (90.7, 159.5)
- added R41: 10k, Resistor_SMD:R_0603_1608Metric, B.Cu at (73.0, 135.0)
- added R42: 330, Resistor_SMD:R_0603_1608Metric, F.Cu at (94.7, 159.5)
- added R44: 330, Resistor_SMD:R_0603_1608Metric, F.Cu at (88.9, 165.3)
- J6: value SERIAL1 -> SERIAL0
- U9: value 25LC010A -> PIC24FJ32GB004; footprint Package_DIP:DIP-8_W7.62mm_Socket -> Package_QFP:LQFP-44_10x10mm_P0.8mm; moved to B.Cu
- moved U9 34.9 mm to (73.8, 126.0), turned to 180 degrees
- moved C40 28.1 mm to (66.3, 125.3)
- moved SW7 22.1 mm to (52.8, 105.8)
- moved SW3 22.1 mm to (58.5, 102.2)
- moved SW4 22.1 mm to (58.5, 105.9)
- moved SW6 22.1 mm to (52.8, 102.2)
- moved SW11 19.7 mm to (74.8, 112.3)
- moved SW10 19.7 mm to (69.8, 112.3)
- moved SW12 19.7 mm to (80.0, 112.3)
- moved SW2 19.7 mm to (64.8, 112.3)
- moved D15 11.0 mm to (54.9, 126.8)
- moved J6 10.3 mm to (72.4, 102.8)
- moved U7 6.43 mm to (82.1, 100.0), turned to 270 degrees
- moved C9 6.26 mm to (66.6, 105.0)
- moved U8 4.34 mm to (57.1, 118.4)
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Connections:
- R106 pad 2: /PA4_IO -> Net-(R106-Pad2)
- U6 pad 29: /PA4_IO -> /PA4_SPI1_NSS
- U9 pad 1: /PE7_ROM_~CS -> Net-(U9-Pad1)
- U9 pad 2: Net-(R54-Pad1) -> /PA10_USART1_RX
- U9 pad 3: /PB2_ROM_~WP -> /PA9_USART1_TX
- U9 pad 4: GND -> Net-(U9-Pad4)
- U9 pad 6: Net-(R55-Pad2) -> GND
- U9 pad 7: /ROM_PE8_~HOLD -> Net-(C78-Pad1)
- U9 pad 8: +3V3 -> /USB_A_D+
Routing:
- net +3V3: track 2.67 -> 34.7 mm
- net /MCLR: track 0.00 -> 14.3 mm, vias 0 -> 1
- net /PGEC1: track 0.00 -> 13.9 mm, vias 0 -> 1
- net +5V: track 24.4 -> 37.6 mm, vias 2 -> 3
- net /PGED1: track 0.00 -> 12.0 mm, vias 0 -> 1
- net /USB_A_D+: track 0.00 -> 8.01 mm
- net /USB_A_D-: track 0.00 -> 6.78 mm
- net Net-(C78-Pad1): track 0.00 -> 3.95 mm, vias 0 -> 1
- net Net-(D46-Pad2): track 0.00 -> 1.77 mm, vias 0 -> 1

Commit message: back up
Parts:
- added D37: DATA, LED_SMD:LED_0603_1608Metric, F.Cu at (92.2, 134.2)
- added D49: COMM, LED_SMD:LED_0603_1608Metric, F.Cu at (92.2, 137.0)
- added J1: microSD, Connector_Card:microSD_HC_Hirose_DM3AT-SF-PEJM5, F.Cu at (74.2, 129.3)
- added R45: 10k, Resistor_SMD:R_0603_1608Metric, B.Cu at (80.0, 119.9)
- added R46: FILTER, Resistor_SMD:R_0603_1608Metric, F.Cu at (61.4, 111.3)
- added R48: FILTER, Resistor_SMD:R_0603_1608Metric, F.Cu at (59.0, 111.3)
- added R50: FILTER, Resistor_SMD:R_0603_1608Metric, F.Cu at (56.6, 111.3)
- added R54: 10k, Resistor_SMD:R_0603_1608Metric, B.Cu at (50.8, 104.1)
- added R55: 10k, Resistor_SMD:R_0603_1608Metric, B.Cu at (56.5, 104.1)
- added R56: 10k, Resistor_SMD:R_0603_1608Metric, B.Cu at (56.5, 107.7)
- added R66: 10k, Resistor_SMD:R_0603_1608Metric, B.Cu at (50.7, 107.8)
- added U28: LOGO, Mizz_lib:Aqualius_Sadalmeric_silk_40x9.4, F.Cu at (133.5, 92.0)
- C35: moved to F.Cu
- C78, R42, R44: moved to B.Cu
- J11: value ENC0 -> ENC1
- J12: value ENC1 -> ENC0
- J13: value ENC2 -> ENC3
- J14: value ENC3 -> ENC2
- J27: value USB_A -> Advanced_SBDBT
- R100, R101, R102, R103, R104, R105, R69, R70, R71, R72, R73, R74, R75, R76, R77, R78, R79, R80, R94, R95, R96, R97, R98, R99: value 3 -> FILTER
- R39: value 10 -> FILTER
- moved R39 60.3 mm to (54.2, 111.3), turned to 90 degrees
- moved JP5 48.2 mm to (59.8, 127.0), turned to 90 degrees
- moved D58 40.0 mm to (60.3, 129.0)
- moved R44 32.9 mm to (84.5, 132.8)
- moved R42 30.0 mm to (84.5, 131.2)
- moved C35 10.9 mm to (75.5, 85.0), turned to 45 degrees
- moved C24 9.29 mm to (74.0, 82.8)
- moved C29 8.55 mm to (65.2, 73.7), turned to 45 degrees
- moved R5 7.61 mm to (67.2, 75.8), turned to 45 degrees
- moved C30 6.99 mm to (62.2, 75.3), turned to 135 degrees
- moved SW6 6.79 mm to (58.5, 105.8)
- moved C21 6.48 mm to (63.9, 91.8), turned to 225 degrees
- moved SW3 5.73 mm to (52.8, 102.2)
- moved C16 5.46 mm to (60.8, 77.2), turned to 135 degrees
- moved C18 5.44 mm to (55.5, 82.5), turned to 135 degrees
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Connections:
- net /PE7_ROM_~CS renamed /PE7_SD_Connection
- net /PE8_ROM_~HOLD renamed /PE8
- J2 pad 10: /PA3_ADC12_IN3 -> /PB1_ADC12_IN9
- J2 pad 5: /PC4_ADC12_IN14 -> /PA2_ADC12_IN2
- J2 pad 6: /PC5_ADC12_IN15 -> /PA3_ADC12_IN3
- J2 pad 7: /PB0_ADC12_IN8 -> /PC4_ADC12_IN14
- J2 pad 8: /PB1_ADC12_IN9 -> /PC5_ADC12_IN15
- J2 pad 9: /PA2_ADC12_IN2 -> /PB0_ADC12_IN8
- JP5 pad 2: Net-(JP5-Pad2) -> +3V3
- R39 pad 2: Net-(R39-Pad2) -> /PA6_SPI1_MISO
- U6 pad 37: /PB2_ROM_~WP -> /PB2_SD_Connection
Routing:
- net +3V3: track 34.7 -> 291.0 mm, vias 0 -> 25
- net +5V: track 37.6 -> 110.6 mm, vias 3 -> 9
- net /PB1_ADC12_IN9: track 0.00 -> 23.9 mm
- net Net-(J1-Pad7): track 0.00 -> 23.7 mm
- net Net-(J1-Pad5): track 0.00 -> 23.3 mm
- net Net-(J1-Pad3): track 0.00 -> 23.2 mm
- net Net-(R14-Pad1): track 0.00 -> 23.2 mm, vias 0 -> 2
- net Net-(J1-Pad2): track 0.00 -> 21.8 mm
- net /PB0_ADC12_IN8: track 0.00 -> 21.6 mm
- net /PC5_ADC12_IN15: track 0.00 -> 20.2 mm
- net /PC3_ADC12_IN13: track 0.00 -> 19.6 mm
- net /PC2_ADC12_IN12: track 0.00 -> 19.2 mm
- net /PC4_ADC12_IN14: track 0.00 -> 19.0 mm
- net /PC1_ADC12_IN11: track 0.00 -> 18.9 mm
- net Net-(D49-Pad1): track 0.00 -> 18.6 mm, vias 0 -> 1
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Other:
- board text removed: "Aquarius Sadalmelik"
