File: 2020/Robot_Lancer/Aqualius_Sadalsuud/Main.sch (KiCad schematic (older format))
At the start: 341 parts, among them J1 microSD, J10 I/O_Vdd, J11 ENC1, J12 ENC0, J13 ENC3, J14 ENC2, J15 5Vin, J16 EMERGENCY, J17 MOTOR0, J18 MOTOR1, J19 MOTOR2, J2 ADC, J20 MOTOR3, J21 MOTOR4, J22 MOTOR5, J23 BATT_IN, J24 BATT_IN, J25 FUSE, J27 Advanced_SBDBT, J28 PICkit3, J3 SWD, J4 CAN, J5 ADC_Vdd, J6 SERIAL0, J7 CAN, J8 VALVE, J9 SERIAL2, Q1 NPN, Q10 NVMFD5C446NLT1G, Q11 FET_N, Q12 NVMFD5C446NLT1G, Q13 NVMFD5C446NLT1G, Q14 NVMFD5C446NLT1G, Q15 NVMFD5C446NLT1G, Q16 NVMFD5C446NLT1G, Q17 NVMFD5C446NLT1G, Q18 FET_P, Q3 FET_P, Q4 FET_P, Q5 NVMFD5C446NLT1G, Q6 NVMFD5C446NLT1G, Q7 NVMFD5C446NLT1G, Q8 NVMFD5C446NLT1G, Q9 NVMFD5C446NLT1G, SW1 RESET, SW10 TOGGLESW1, SW11 TOGGLESW2, SW12 TOGGLESW3, SW2 TOGGLESW0, SW3 SW0, SW4 SW1, SW5 Control-Power_SW, SW6 SW2, SW7 SW3, SW8 EMERGENCY_SW, SW9 MAIN_SW, U1 MAX3051, U10 BD9G101G, U11 CCG30-24-12, U12 NCP5104, U13 NCP5104, U14 NCP5104, U15 NCP5104, U16 NCP5104, U17 NCP5104, U18 V23086-C1001, U19 NCP5104, U2 AP3211, U20 NCP5104, U21 NCP5104, U22 NCP5104, U23 NCP5104, U24 NCP5104, U25 LOGO, U26 7805, U27 TBD62083A, U28 LOGO, U3 MCP2221A, U4 AQM0802, U5 AZ1086H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

Commit message: 2019/12/13_AM2:35
Parts:
- C42: footprint Capacitor_THT:CP_Radial_D8.0mm_P3.50mm -> Capacitor_THT:CP_Radial_D6.3mm_P2.50mm
- D3: value LED -> XA_5V
- D36: value LED -> BATT
- D38: value LED -> MAIN
- D4: value LED -> 12V-5V
- D46: value LED -> 5Vp
- D48: value LED -> MOTOR_BATT
- D5: value LED -> 5Vc
- D57: value LED -> 12Vp
- D6: value LED -> 12V
- D8: value LED -> 5V
- D9: value LED -> 3V3
- U28: footprint Mizz_lib:Aqualius_Sadalmeric_silk_40x9.4 -> Mizz_lib:Aqualius_Sadalsuud_silk_40x9.4
Connections:
- net PA4_IO is gone; now on net PE4_IO: U27.5 (IN5)
- net PE8 is gone; now on net PE8_ADRESS0: U6.39 (PE8/FSMC_D5/TIM1_CH1N/EVENTOUT)
- net ADRESS2_PD14: no longer U8.4
- net ADRESS3_PD15: no longer U8.6 (8)
- net LED0: no longer U6.1 (PE2/TRACECLK/FSMC_A23/ETH_MII_TXD3/EVENTOUT)
- net LED1: no longer U6.2 (PE3/TRACED0/FSMC_A19/EVENTOUT)
- net LED2: no longer U6.3 (PE4/TRACED1/FSMC_A20/DCMI_D4/EVENTOUT)
- net LED3: no longer U6.7 (PC13/EVENTOUT)
- net LED4: no longer U6.8 (PC14/OSC32_IN/EVENTOUT)
- net LED5: now also U6.57 (PD10/FSMC_D15/USART3_CK/EVENTOUT); no longer U6.9 (PC15/OSC32_OUT/EVENTOUT)
- net PD6_DIPSW_3: no longer U6.88 (PD7/USART2_CK/FSMC_NE1/FSMC_NCE2/EVENTOUT)
- net motor2_L_signal: now also U6.65 (PC8/TIM8_CH3/SDIO_D0/TIM3_CH3/USART6_CK/DCMI_D2/EVENTOUT); no longer U6.40 (PE9/FSMC_D6/TIM1_CH1/EVENTOUT)
- net motor2_R_signal: now also U6.66 (PC9/I2S_CKIN/MCO2/TIM8_CH4/SDIO_D1/I2C3_SDA/DCMI_D3/TIM3_CH4/EVENTOUT); no longer U6.42 (PE11/FSMC_D8/TIM1_CH2/EVENTOUT)
- net motor3_L_signal: now also U6.54 (PB15/SPI2_MOSI/I2S2_SD/TIM1_CH3N/TIM8_CH3N/TIM12_CH2/OTG_HS_DP/EVENTOUT); no longer U6.44 (PE13/FSMC_D10/TIM1_CH3/EVENTOUT)
- net motor3_R_signal: now also U6.53 (PB14/SPI2_MISO/TIM1_CH2N/TIM12_CH1/OTG_HS_DM/USART3_RTS/TIM8_CH2N/I2S2ext_SD/EVENTOUT); no longer U6.45 (PE14/FSMC_D11/TIM1_CH4/EVENTOUT)
- net motor4_L_signal: now also U6.45 (PE14/FSMC_D11/TIM1_CH4/EVENTOUT); no longer U6.53 (PB14/SPI2_MISO/TIM1_CH2N/TIM12_CH1/OTG_HS_DM/USART3_RTS/TIM8_CH2N/I2S2ext_SD/EVENTOUT)
- net motor4_R_signal: now also U6.44 (PE13/FSMC_D10/TIM1_CH3/EVENTOUT); no longer U6.54 (PB15/SPI2_MOSI/I2S2_SD/TIM1_CH3N/TIM8_CH3N/TIM12_CH2/OTG_HS_DP/EVENTOUT)
- net motor5_L_signal: now also U6.42 (PE11/FSMC_D8/TIM1_CH2/EVENTOUT); no longer U6.65 (PC8/TIM8_CH3/SDIO_D0/TIM3_CH3/USART6_CK/DCMI_D2/EVENTOUT)
- net motor5_R_signal: now also U6.40 (PE9/FSMC_D6/TIM1_CH1/EVENTOUT); no longer U6.66 (PC9/I2S_CKIN/MCO2/TIM8_CH4/SDIO_D1/I2C3_SDA/DCMI_D3/TIM3_CH4/EVENTOUT)
- net PE4_IO: now reaches R106.2
- net PE4_IO: now also U6.3 (PE4/TRACED1/FSMC_A20/DCMI_D4/EVENTOUT)
- net ADRESS0_PD10 renamed PE8_ADRESS0
- net PE8_ADRESS0: no longer U6.57 (PD10/FSMC_D15/USART3_CK/EVENTOUT)
- net ADRESS1_PD11: no longer names the net of U6.58 (PD11/FSMC_CLE/FSMC_A16/USART3_CTS/EVENTOUT)
- net ADRESS1_PD11: no longer U8.1 (2)
- net BLUE: no longer names the net of U6.80 (PC12/UART5_TX/SDIO_CK/DCMI_D9/SPI3_MOSI/I2S3_SD/USART3_CK/EVENTOUT)
- net BLUE: no longer R36.1
- net GREEN: no longer names the net of U6.79 (PC11/UART4_RX/SPI3_MISO/SDIO_D3/DCMI_D4/USART3_RX/I2S3ext_SD/EVENTOUT)
- net GREEN: no longer R37.1
- net PA11_IO renamed PC14_IO
- net PC14_IO: now also U6.8 (PC14/OSC32_IN/EVENTOUT); no longer U6.70 (PA11/USART1_CTS/CAN1_RX/TIM1_CH4_/OTG_FS_DM/EVENTOUT)
- net PA12_IO renamed PC13_IO
- net PC13_IO: now also U6.7 (PC13/EVENTOUT); no longer U6.71 (PA12/USART1_RTS/CAN1_TX/TIM1_ETR/OTG_FS_DP/EVENTOUT)
- net PA8_IO renamed PC15_IO
- net PC15_IO: now also U6.9 (PC15/OSC32_OUT/EVENTOUT); no longer U6.67 (PA8/MCO1/USART1_CK/TIM1_CH1/I2C3_SCL/OTG_FS_SOF/EVENTOUT)
- net PB2_SD_Connection renamed _SD_Connection
- net _SD_Connection: no longer U6.37 (PB2/BOOT1/EVENTOUT)
- net PE10 renamed PE10_ADRESS1
- net PE10_ADRESS1: now also U8.1 (2)
- net PE12_IO renamed PE2_IO
- net PE2_IO: now also U6.1 (PE2/TRACECLK/FSMC_A23/ETH_MII_TXD3/EVENTOUT); no longer U6.43 (PE12/FSMC_D9/TIM1_CH3N/EVENTOUT)
- net PE15_IO renamed PE3_IO
- net PE3_IO: now also U6.2 (PE3/TRACED0/FSMC_A19/EVENTOUT); no longer U6.46 (PE15/FSMC_D12/TIM1_BKIN/EVENTOUT)
- net PE7_SD_Connection renamed PE7_SW3
- net PE7_SW3: now also R66.1, SW7.2
- net RED: no longer names the net of U6.78 (PC10/SPI3_SCK/I2S3_CK/UART4_TX/SDIO_D2/DCMI_D8/USART3_TX/EVENTOUT)
- net RED: no longer R38.1
- net SW0 renamed PB2_SW0
- net PB2_SW0: now also U6.37 (PB2/BOOT1/EVENTOUT); no longer U6.47 (PB10/SPI2_SCK/I2S2_CK/I2C2_SCL/USART3_TX/OTG_HS_ULPI_D3/ETH_MII_RX_ER/TIM2_CH3/EVENTOUT)
- net SW1 renamed PE15_SW1
- net PE15_SW1: now also U6.46 (PE15/FSMC_D12/TIM1_BKIN/EVENTOUT); no longer U6.48 (PB11/I2C2_SDA/USART3_RX/OTG_HS_ULPI_D4/ETH_RMII_TX_EN/ETH_MII_TX_EN/TIM2_CH4/EVENTOUT)
- net SW2 renamed PE12_SW2
- net PE12_SW2: now also U6.43 (PE12/FSMC_D9/TIM1_CH3N/EVENTOUT); no longer U6.51 (PB12/SPI2_NSS/I2S2_WS/I2C2_SMBA/USART3_CK/TIM1_BKIN/CAN2_RX/OTG_HS_ULPI_D5/ETH_RMII_TXD0/ETH_MII_TXD0/OTG_HS_ID/EVENTOUT)
- removed net SW3: R66.1, SW7.2, U6.52 (PB13/SPI2_SCK/I2S2_CK/USART3_CTS/TIM1_CH1N/CAN2_TX/OTG_HS_ULPI_D6/ETH_RMII_TXD1/ETH_MII_TXD1/EVENTOUT)
- new net PB10_RED: R38.1, U6.47 (PB10/SPI2_SCK/I2S2_CK/I2C2_SCL/USART3_TX/OTG_HS_ULPI_D3/ETH_MII_RX_ER/TIM2_CH3/EVENTOUT)
- new net PB11_GREEN: R37.1, U6.48 (PB11/I2C2_SDA/USART3_RX/OTG_HS_ULPI_D4/ETH_RMII_TX_EN/ETH_MII_TX_EN/TIM2_CH4/EVENTOUT)
- new net PB12_ADRESS2: U6.51 (PB12/SPI2_NSS/I2S2_WS/I2C2_SMBA/USART3_CK/TIM1_BKIN/CAN2_RX/OTG_HS_ULPI_D5/ETH_RMII_TXD0/ETH_MII_TXD0/OTG_HS_ID/EVENTOUT), U8.4
- new net PB12_BLUE: R36.1
- new net PB13_ADRESS3: U6.52 (PB13/SPI2_SCK/I2S2_CK/USART3_CTS/TIM1_CH1N/CAN2_TX/OTG_HS_ULPI_D6/ETH_RMII_TXD1/ETH_MII_TXD1/EVENTOUT), U8.6 (8)
- new net PD7_DIPSW_3: U6.88 (PD7/USART2_CK/FSMC_NE1/FSMC_NCE2/EVENTOUT)
Other:
- moved on the sheet: C11, C14, C16, C17, C18, C21, C24, C29, C30, C36, C37, C38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

Commit message: 2013/12/13 Aqua
Parts:
- removed D25: RESET, LED_SMD:LED_0603_1608Metric, symbol Device:LED
- removed R27: 240, Resistor_SMD:R_0603_1608Metric, symbol Device:R
Connections:
- net LED0 is gone; now on net PC12_LED0: R40.2
- net LED1 is gone; now on net PC11_LED1: R43.2
- net LED2 is gone; now on net PC10_LED2: R47.2
- net LED3 is gone; now on net PA12_LED3: R49.2
- net LED4 is gone; now on net PA11_LED4: R51.2
- net PD6_DIPSW_3 is gone; now on net PD15_TOGGLESW_3: SW12.2 (B)
- net _SD_Connection is gone; now on net PB9_SD_Connection: J1.9 (DET_B), R45.1
- net PB4_TIM3_CH1: now also R21.1; no longer R33.1
- net PB5_TIM3_CH2: now also R23.1; no longer R35.1
- net PD12_TIM4_CH1: now also R33.1; no longer R21.1
- net PD13_TIM4_CH2: now also R35.1; no longer R23.1
- net PD2_DIPSW_0: no longer SW2.2 (B)
- net PD3_DIPSW_1: no longer SW10.2 (B)
- net PD4_DIPSW_2: no longer SW11.2 (B)
- net motor1_L_signal: now also U6.66 (PC9/I2S_CKIN/MCO2/TIM8_CH4/SDIO_D1/I2C3_SDA/DCMI_D3/TIM3_CH4/EVENTOUT); no longer U6.63 (PC6/I2S2_MCK/TIM8_CH1/SDIO_D6/USART6_TX/DCMI_D0/TIM3_CH1/EVENTOUT)
- net motor1_R_signal: now also U6.65 (PC8/TIM8_CH3/SDIO_D0/TIM3_CH3/USART6_CK/DCMI_D2/EVENTOUT); no longer U6.64 (PC7/I2S3_MCK/TIM8_CH2/SDIO_D7/USART6_RX/DCMI_D1/TIM3_CH2/EVENTOUT)
- net motor2_L_signal: now also U6.64 (PC7/I2S3_MCK/TIM8_CH2/SDIO_D7/USART6_RX/DCMI_D1/TIM3_CH2/EVENTOUT); no longer U6.65 (PC8/TIM8_CH3/SDIO_D0/TIM3_CH3/USART6_CK/DCMI_D2/EVENTOUT)
- net motor2_R_signal: now also U6.63 (PC6/I2S2_MCK/TIM8_CH1/SDIO_D6/USART6_TX/DCMI_D0/TIM3_CH1/EVENTOUT); no longer U6.66 (PC9/I2S_CKIN/MCO2/TIM8_CH4/SDIO_D1/I2C3_SDA/DCMI_D3/TIM3_CH4/EVENTOUT)
- net PD11_TOGGLESW_1: now reaches U6.58 (PD11/FSMC_CLE/FSMC_A16/USART3_CTS/EVENTOUT)
- net PD11_TOGGLESW_1: now also SW10.2 (B)
- net PA8_LED5: now reaches U6.67 (PA8/MCO1/USART1_CK/TIM1_CH1/I2C3_SCL/OTG_FS_SOF/EVENTOUT)
- net PA8_LED5: now also R52.2
- net PA11_LED4: now reaches U6.70 (PA11/USART1_CTS/CAN1_RX/TIM1_CH4_/OTG_FS_DM/EVENTOUT)
- net PA12_LED3: now reaches U6.71 (PA12/USART1_RTS/CAN1_TX/TIM1_ETR/OTG_FS_DP/EVENTOUT)
- net PC10_LED2: now reaches U6.78 (PC10/SPI3_SCK/I2S3_CK/UART4_TX/SDIO_D2/DCMI_D8/USART3_TX/EVENTOUT)
- net PC11_LED1: now reaches U6.79 (PC11/UART4_RX/SPI3_MISO/SDIO_D3/DCMI_D4/USART3_RX/I2S3ext_SD/EVENTOUT)
- net PC12_LED0: now reaches U6.80 (PC12/UART5_TX/SDIO_CK/DCMI_D9/SPI3_MOSI/I2S3_SD/USART3_CK/EVENTOUT)
- net ADRESS2_PD14 renamed PD14_TOGGLESW_2
- net PD14_TOGGLESW_2: now also SW11.2 (B)
- net ADRESS3_PD15 renamed PD15_TOGGLESW_3
- net LED5 renamed PD10_TOGGLESW_0
- net PD10_TOGGLESW_0: now also SW2.2 (B); no longer R52.2
- net PB9_LCD_BL_TIM11_CH1 renamed PB9_SD_Connection
Other:
- moved on the sheet: D27, D28, D29, D30, D31, D32, R40, R43, R47, R49, R51, R52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

Commit message: ランサー1機体目回路完成
Parts:
- removed D32: LED5, LED_SMD:LED_0603_1608Metric, symbol Device:LED
- removed Q11: FET_N, Package_TO_SOT_SMD:SOT-23W, symbol Device:Q_NMOS_GDS
- removed Q18: FET_P, Package_TO_SOT_SMD:SOT-23W, symbol Device:Q_PMOS_GDS
- removed Q3, Q4: FET_P, Package_TO_SOT_SMD:SOT-23W, symbol Device:Q_NMOS_GDS
- removed R52: 330, Resistor_SMD:R_0603_1608Metric, symbol Device:R
- added C5, C81, C82, C83, C84, C85: 0.1u, Capacitor_SMD:C_0603_1608Metric, symbol Device:C
- added Q11: FET_N, Package_TO_SOT_SMD:SOT-23W, symbol Device:Q_NMOS_GSD
- added Q2, Q3, Q4: FET_P, Package_TO_SOT_SMD:SOT-23W, symbol Device:Q_NMOS_GSD
- added U29: LOGO, Mizz_lib:Aqualius_silk_20.3x15.2_onlyStar, symbol Miz:LOGO
- R8: value 50k -> 3.9k
- R9: value 10k -> 680
- U2: value AP3211 -> BD9G101G
Connections:
- net PB12_BLUE is gone; now on net PA8_BLUE: R36.1
- net +3V3: now also D14.1 (K); no longer D14.2 (A)
- net +5V: now also Q3.3 (D)
- net Batt: now also C50.1, C51.1, U10.4 (EN), U10.5 (VCC), Q2.3 (D)
- net Control_5V: now also Q3.2 (S), Q4.3 (D)
- net External_5V: now also Q4.1 (G)
- net GNDPWR: now also Q11.2 (S)
- net MOTOR_Batt: no longer C50.1, C51.1, U10.4 (EN), U10.5 (VCC)
- net Motor0L: now also C5.1
- net Motor0R: now also C5.2
- net Motor1L: now also C81.1
- net Motor1R: now also C81.2
- net Motor2L: now also C82.1
- net Motor2R: now also C82.2
- net Motor3L: now also C83.1
- net Motor3R: now also C83.2
- net Motor4L: now also C84.1
- net Motor4R: now also C84.2
- net Motor5L: now also C85.1
- net Motor5R: now also C85.2
- net at D26.2 (A), SW9.2 (B): now also Q2.2 (S)
- net at D56.2 (A), JP2.2, U18.2: now also Q11.3 (D)
- net at SW5.2 (B): now also Q3.1 (G)
- net at R87.1, SW8.2 (B): now also Q11.1 (G)
- net at D33.1 (K): now also Q4.2 (S)
- net at R82.1, SW9.1 (A): now also Q2.1 (G)
- net at LS1.2, R11.2: now also D14.2 (A); no longer D14.1 (K)
- net PA8_LED5 renamed PA8_BLUE
Other:
- moved on the sheet: J17, J18, J19, J20, J21, J22, J23, J24, R45, U8
