File: 2020/Robot_Lancer/Aqualius_Sadalsuud/Main.kicad_pcb (KiCad board)
At the start: 2 copper layers, 100 x 100 mm, 341 parts, among them J1 microSD, J10 I/O_Vdd, J11 ENC1, J12 ENC0, J13 ENC3, J14 ENC2, J15 5Vin, J16 EMERGENCY, J17 MOTOR0, J18 MOTOR1, J19 MOTOR2, J2 ADC, J20 MOTOR3, J21 MOTOR4, J22 MOTOR5, J23 BATT_IN, J24 BATT_IN, J25 FUSE, J27 Advanced_SBDBT, J28 PICkit3, J3 SWD, J4 CAN, J5 ADC_Vdd, J6 SERIAL0, J7 CAN, J8 VALVE, J9 SERIAL2, Q1 NPN, Q10 NVMFD5C446NLT1G, Q11 FET_N, Q12 NVMFD5C446NLT1G, Q13 NVMFD5C446NLT1G, Q14 NVMFD5C446NLT1G, Q15 NVMFD5C446NLT1G, Q16 NVMFD5C446NLT1G, Q17 NVMFD5C446NLT1G, Q18 FET_P, Q3 FET_P, Q4 FET_P, Q5 NVMFD5C446NLT1G, Q6 NVMFD5C446NLT1G, Q7 NVMFD5C446NLT1G, Q8 NVMFD5C446NLT1G, Q9 NVMFD5C446NLT1G, SW1 RESET, SW10 TOGGLESW1, SW11 TOGGLESW2, SW12 TOGGLESW3, SW2 TOGGLESW0, SW3 SW0, SW4 SW1, SW5 Control-Power_SW, SW6 SW2, SW7 SW3, SW8 EMERGENCY_SW, SW9 MAIN_SW, U1 MAX3051, U10 BD9G101G, U11 CCG30-24-12, U12 NCP5104, U13 NCP5104, U14 NCP5104, U15 NCP5104, U16 NCP5104, U17 NCP5104, U18 V23086-C1001, U19 NCP5104, U2 AP3211, U20 NCP5104, U21 NCP5104, U22 NCP5104, U23 NCP5104, U24 NCP5104, U25 LOGO, U26 7805, U27 TBD62083A, U28 LOGO, U3 MCP2221A, U4 AQM0802, U5 AZ1086H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

Commit message: 2013/12/13 Aqua
Parts:
- removed D25: RESET, LED_SMD:LED_0603_1608Metric
- removed R27: 240, Resistor_SMD:R_0603_1608Metric
- moved U4 0.06 mm to (49.6, 77.2)
Connections:
- J1 pad 9: /_SD_Connection -> /PB9_SD_Connection
- R21 pad 1: /PD12_TIM4_CH1 -> /PB4_TIM3_CH1
- R23 pad 1: /PD13_TIM4_CH2 -> /PB5_TIM3_CH2
- R33 pad 1: /PB4_TIM3_CH1 -> /PD12_TIM4_CH1
- R35 pad 1: /PB5_TIM3_CH2 -> /PD13_TIM4_CH2
- R40 pad 2: /LED0 -> /PC12_LED0
- R43 pad 2: /LED1 -> /PC11_LED1
- R45 pad 1: /_SD_Connection -> /PB9_SD_Connection
- R47 pad 2: /LED2 -> /PC10_LED2
- R49 pad 2: /LED3 -> /PA12_LED3
- R51 pad 2: /LED4 -> /PA11_LED4
- R52 pad 2: /LED5 -> /PA8_LED5
- SW10 pad 2: /PD3_DIPSW_1 -> /PD11_TOGGLESW_1
- SW11 pad 2: /PD4_DIPSW_2 -> /PD14_TOGGLESW_2
- SW12 pad 2: /PD6_DIPSW_3 -> /PD15_TOGGLESW_3
- SW2 pad 2: /PD2_DIPSW_0 -> /PD10_TOGGLESW_0
- U6 pad 57: Net-(U6-Pad57) -> /PD10_TOGGLESW_0
- U6 pad 58: Net-(U6-Pad58) -> /PD11_TOGGLESW_1
- U6 pad 61: /ADRESS2_PD14 -> /PD14_TOGGLESW_2
- U6 pad 62: /ADRESS3_PD15 -> /PD15_TOGGLESW_3
- U6 pad 63: /motor1_L_signal -> /motor2_R_signal
- U6 pad 64: /motor1_R_signal -> /motor2_L_signal
- U6 pad 65: /motor2_L_signal -> /motor1_R_signal
- U6 pad 66: /motor2_R_signal -> /motor1_L_signal
- U6 pad 67: Net-(U6-Pad67) -> /PA8_LED5
- U6 pad 70: Net-(U6-Pad70) -> /PA11_LED4
- U6 pad 71: Net-(U6-Pad71) -> /PA12_LED3
- U6 pad 78: Net-(U6-Pad78) -> /PC10_LED2
- U6 pad 79: Net-(U6-Pad79) -> /PC11_LED1
- U6 pad 80: Net-(U6-Pad80) -> /PC12_LED0
- U6 pad 96: /PB9_LCD_BL_TIM11_CH1 -> /PB9_SD_Connection
Routing:
- net /PB9_SD_Connection: track 0.00 -> 96.8 mm, vias 0 -> 6
- net /PA15_TIM2_CH1: track 0.00 -> 58.0 mm, vias 0 -> 2
- net /PD10_TOGGLESW_0: track 0.00 -> 47.8 mm, vias 0 -> 3
- net /PD11_TOGGLESW_1: track 0.00 -> 47.5 mm, vias 0 -> 3
- net /PD15_TOGGLESW_3: track 0.00 -> 39.1 mm, vias 0 -> 3
- net /SWDIO: track 0.00 -> 38.6 mm, vias 0 -> 1
- net /PD14_TOGGLESW_2: track 0.00 -> 38.3 mm, vias 0 -> 3
- net /PD2_DIPSW_0: track 30.1 -> 0.00 mm, vias 1 -> 0
- net /PD3_DIPSW_1: track 29.2 -> 0.00 mm, vias 1 -> 0
- net /PA10_USART1_RX: track 28.4 -> 50.3 mm, vias 1 -> 3
- net /PD4_DIPSW_2: track 21.0 -> 0.00 mm, vias 1 -> 0
- net /motor1_R_signal: track 0.00 -> 20.9 mm
- net /motor1_L_signal: track 0.00 -> 20.8 mm
- net /PD6_DIPSW_3: track 20.7 -> 0.00 mm, vias 1 -> 0
- net /PA9_USART1_TX: track 34.4 -> 55.0 mm, vias 1 -> 3
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
Commit message: 配線
Parts:
- moved C35 0.22 mm to (75.4, 85.2)
Routing:
- net /PB5_TIM3_CH2: track 19.0 -> 72.1 mm, vias 1 -> 3
- net /PB4_TIM3_CH1: track 15.6 -> 67.4 mm, vias 1 -> 3
- net /SWDIO: track 38.6 -> 35.5 mm
- net /PA15_TIM2_CH1: track 58.0 -> 55.4 mm
- net GND: track 21.7 -> 24.1 mm, vias 67 -> 64
- net +5V: track 270.1 -> 271.3 mm

Commit message: 強引に完成させた
Parts:
- moved C79 0.89 mm to (73.0, 118.0), turned to 90 degrees
- moved U7 0.15 mm to (82.2, 100.0)
Routing:
- net /PD6_USART2_RX: track 0.00 -> 89.2 mm, vias 0 -> 11
- net /SWCLK: track 0.00 -> 88.1 mm, vias 0 -> 7
- net /PD5_USART2_TX: track 0.00 -> 85.4 mm, vias 0 -> 12
- net /PB3_TIM2_CH2: track 17.4 -> 88.7 mm, vias 1 -> 7
- net /~RST: track 18.2 -> 73.3 mm, vias 1 -> 6
- net /SWDIO: track 35.5 -> 82.4 mm, vias 1 -> 6
- net /PD12_TIM4_CH1: track 0.00 -> 45.2 mm, vias 0 -> 5
- net /PD13_TIM4_CH2: track 0.00 -> 43.8 mm, vias 0 -> 3
- net /PB12_ADRESS2: track 6.47 -> 44.3 mm, vias 1 -> 3
- net /PB13_ADRESS3: track 6.97 -> 43.2 mm, vias 1 -> 3
- net /PA15_TIM2_CH1: track 55.4 -> 71.4 mm, vias 2 -> 5
- net /PB9_SD_Connection: track 96.8 -> 86.2 mm, vias 6 -> 5
- net +3V3: track 395.9 -> 402.0 mm
- net /PE15_SW1: track 16.7 -> 21.9 mm
- net /PE10_ADRESS1: track 36.9 -> 31.8 mm, vias 3 -> 2
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
Commit message: 圧縮した
Routing:
- net GND: track 28.7 -> 32.2 mm, vias 82 -> 85
- net Net-(D3-Pad2): vias 0 -> 1
- net Net-(D19-Pad1): vias 0 -> 1
- net Net-(D17-Pad1): vias 0 -> 1
- net /Motor5R: vias 20 -> 23
- net /Motor5L: vias 20 -> 23
- net /Motor4R: vias 20 -> 23
- net /Motor3R: vias 20 -> 23
- net /Motor1R: vias 20 -> 23
- net /Motor1L: vias 20 -> 23
- net /Motor0R: vias 20 -> 23
- net /Motor0L: vias 20 -> 22

Commit message: ランサー1機体目回路完成
Parts:
- removed D32: LED5, LED_SMD:LED_0603_1608Metric
- removed Q18: FET_P, Package_TO_SOT_SMD:SOT-23W
- removed R52: 330, Resistor_SMD:R_0603_1608Metric
- added C5: 0.1u, Capacitor_SMD:C_0603_1608Metric, B.Cu at (123.8, 70.5)
- added C81: 0.1u, Capacitor_SMD:C_0603_1608Metric, B.Cu at (123.8, 82.5)
- added C82: 0.1u, Capacitor_SMD:C_0603_1608Metric, B.Cu at (123.8, 95.5)
- added C83: 0.1u, Capacitor_SMD:C_0603_1608Metric, B.Cu at (124.2, 107.8)
- added C84: 0.1u, Capacitor_SMD:C_0603_1608Metric, B.Cu at (124.2, 120.0)
- added C85: 0.1u, Capacitor_SMD:C_0603_1608Metric, B.Cu at (124.2, 132.0)
- added Q2: FET_P, Package_TO_SOT_SMD:SOT-23W, B.Cu at (103.0, 48.7)
- added U29: LOGO, Mizz_lib:Aqualius_silk_20.3x15.2_onlyStar, B.Cu at (53.9, 91.4)
- R8: value 50k -> 3.9k
- R9: value 10k -> 680
- U2: value AP3211 -> BD9G101G
- moved Q11 2.16 mm to (94.8, 49.1), turned to 270 degrees
- moved Q3 1.33 mm to (56.8, 63.8), turned to 0 degrees
- moved Q4 0.96 mm to (62.6, 65.2)
- turned D14 to 90 degrees
Connections:
- C50 pad 1: MOTOR_Batt -> Batt
- C51 pad 1: MOTOR_Batt -> Batt
- D14 pad 1: Net-(D14-Pad1) -> +3V3
- D14 pad 2: +3V3 -> Net-(D14-Pad2)
- LS1 pad 2: Net-(D14-Pad1) -> Net-(D14-Pad2)
- Q11 pad 2: Net-(D56-Pad2) -> GNDPWR
- Q11 pad 3: GNDPWR -> Net-(D56-Pad2)
- Q3 pad 2: +5V -> Control_5V
- Q3 pad 3: Control_5V -> +5V
- Q4 pad 2: Control_5V -> Net-(D33-Pad1)
- Q4 pad 3: Net-(D33-Pad1) -> Control_5V
- R11 pad 2: Net-(D14-Pad1) -> Net-(D14-Pad2)
- R36 pad 1: /PB12_BLUE -> /PA8_BLUE
- U10 pad 4: MOTOR_Batt -> Batt
- U10 pad 5: MOTOR_Batt -> Batt
- U6 pad 67: /PA8_LED5 -> /PA8_BLUE
Routing:
- net Batt: track 42.4 -> 68.8 mm, vias 2 -> 0
- net /PA8_BLUE: track 0.00 -> 24.6 mm, vias 0 -> 2
- net /PA8_LED5: track 19.2 -> 0.00 mm, vias 2 -> 0
- net /PB12_BLUE: track 7.21 -> 0.00 mm, vias 1 -> 0
- net Net-(D14-Pad2): track 0.00 -> 4.66 mm, vias 0 -> 2
- net Net-(D14-Pad1): track 4.66 -> 0.00 mm, vias 2 -> 0
- net Net-(Q2-Pad1): track 12.4 -> 8.95 mm
- net GND: track 32.2 -> 34.0 mm, vias 85 -> 193
- net Net-(D33-Pad1): track 8.28 -> 6.76 mm
- net MOTOR_Batt: track 29.9 -> 31.2 mm
- net /PD10_TOGGLESW_0: track 46.6 -> 47.8 mm
- net Net-(D56-Pad2): track 36.8 -> 35.7 mm
- net +5V: track 271.3 -> 272.4 mm
- net Control_5V: track 25.6 -> 24.6 mm
- net Net-(D32-Pad2): track 0.73 -> 0.00 mm
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Other:
- board text added: "Designed by A.Mizuta(twitter:@wrf_lab) in 2019/12/19."

Commit message: K-Kodani作ラインセンサ
Other:
- board text added: "4"
- board text added: "FULLCOLOR"
- board text added: "LED"
Changed lines of the file:
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@@
   (general
     (thickness 1.6)
-    (drawings 45)
+    (drawings 49)
     (tracks 4100)
     (zones 0)
@@
       (effects (font (size 1 1) (thickness 0.15)))
     )
-    (fp_text value Si8660 (at 0 6.2) (layer F.SilkS)
+    (fp_text value Si8660 (at 0 6) (layer F.SilkS)
       (effects (font (size 0.8 0.8) (thickness 0.15)))
     )
@@
       (effects (font (size 1 1) (thickness 0.15)) (justify mirror))
     )
-    (fp_text value FET_P (at 0 -2.5) (layer B.SilkS)
+    (fp_text value FET_P (at -2.45 0 90) (layer B.SilkS)
       (effects (font (size 0.8 0.8) (thickness 0.15)) (justify mirror))
     )
@@
       (xy 1.74625 7.611422) (xy 1.798252 7.614777) (xy 1.80975 7.611422)) (layer B.SilkS) (width 0.01))
   )
+  (gr_text FULLCOLOR (at 82.3 103.3) (layer F.SilkS)
+    (effects (font (size 1 1) (thickness 0.25)))
+  )
+  (gr_text 4 (at 86.75 92.75 90) (layer F.SilkS)
+    (effects (font (size 0.8 0.8) (thickness 0.15)))
+  )
+  (gr_text 0 (at 86.75 85.75 90) (layer F.SilkS)
+    (effects (font (size 0.8 0.8) (thickness 0.15)))
+  )
+  (gr_text LED (at 86.75 89.25 90) (layer F.SilkS)
+    (effects (font (size 1 1) (thickness 0.15)))
+  )
   (gr_text "Designed by A.Mizuta(twitter:@wrf_lab)\nin 2019/12/19." (at 46.95 108.35 270) (layer B.SilkS)
