File: 2020/Robot_Lancer/Aqualius_Sadalsuud/Main.kicad_pcb (KiCad board)
At the start: 2 copper layers, 100 x 100 mm, 344 parts, among them J1 microSD, J10 I/O_Vdd, J11 ENC1, J12 ENC0, J13 ENC3, J14 ENC2, J15 5Vin, J16 EMERGENCY, J17 MOTOR0, J18 MOTOR1, J19 MOTOR2, J2 ADC, J20 MOTOR3, J21 MOTOR4, J22 MOTOR5, J23 BATT_IN, J24 BATT_IN, J25 FUSE, J27 Advanced_SBDBT, J28 PICkit3, J3 SWD, J4 CAN, J5 ADC_Vdd, J6 SERIAL0, J7 CAN, J8 VALVE, J9 SERIAL2, Q1 NPN, Q10 NVMFD5C446NLT1G, Q11 FET_N, Q12 NVMFD5C446NLT1G, Q13 NVMFD5C446NLT1G, Q14 NVMFD5C446NLT1G, Q15 NVMFD5C446NLT1G, Q16 NVMFD5C446NLT1G, Q17 NVMFD5C446NLT1G, Q2 FET_P, Q3 FET_P, Q4 FET_P, Q5 NVMFD5C446NLT1G, Q6 NVMFD5C446NLT1G, Q7 NVMFD5C446NLT1G, Q8 NVMFD5C446NLT1G, Q9 NVMFD5C446NLT1G, SW1 RESET, SW10 TOGGLESW1, SW11 TOGGLESW2, SW12 TOGGLESW3, SW2 TOGGLESW0, SW3 SW0, SW4 SW1, SW5 Control-Power_SW, SW6 SW2, SW7 SW3, SW8 EMERGENCY_SW, SW9 MAIN_SW, U1 MAX3051, U10 BD9G101G, U11 CCG30-24-12, U12 NCP5104, U13 NCP5104, U14 NCP5104, U15 NCP5104, U16 NCP5104, U17 NCP5104, U18 V23086-C1001, U19 NCP5104, U2 BD9G101G, U20 NCP5104, U21 NCP5104, U22 NCP5104, U23 NCP5104, U24 NCP5104, U25 LOGO, U26 7805, U27 TBD62083A, U28 LOGO, U29 LOGO, U3 MCP2221A, U4 AQM0802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

Commit message: 信号線の配線終わり
Routing:
- net +5V: track 272.4 -> 274.1 mm
- net GND: vias 193 -> 188
Changed lines of the file:
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@@
     (thickness 1.6)
     (drawings 49)
-    (tracks 4100)
+    (tracks 4097)
     (zones 0)
     (modules 344)
@@
   )
   (setup
-    (last_trace_width 0.25)
+    (last_trace_width 0.5)
     (user_trace_width 0.2)
     (user_trace_width 0.3)
@@
   (via (at 75 130.25) (size 0.8) (drill 0.4) (layers F.Cu B.Cu) (net 2))
   (via (at 72.75 130.25) (size 0.8) (drill 0.4) (layers F.Cu B.Cu) (net 2))
-  (via (at 72.75 127.25) (size 0.8) (drill 0.4) (layers F.Cu B.Cu) (net 2))
-  (via (at 74.75 127.25) (size 0.8) (drill 0.4) (layers F.Cu B.Cu) (net 2))
-  (via (at 78 125.5) (size 0.8) (drill 0.4) (layers F.Cu B.Cu) (net 2))
   (via (at 77.75 130.25) (size 0.8) (drill 0.4) (layers F.Cu B.Cu) (net 2))
   (via (at 70.75 125) (size 0.8) (drill 0.4) (layers F.Cu B.Cu) (net 2))
-  (via (at 69.75 127) (size 0.8) (drill 0.4) (layers F.Cu B.Cu) (net 2))
   (via (at 68.5 132.75) (size 0.8) (drill 0.4) (layers F.Cu B.Cu) (net 2))
   (via (at 67 134) (size 0.8) (drill 0.4) (layers F.Cu B.Cu) (net 2))
@@
   (via (at 72.5 137) (size 0.8) (drill 0.4) (layers F.Cu B.Cu) (net 2))
   (via (at 76.25 137) (size 0.8) (drill 0.4) (layers F.Cu B.Cu) (net 2))
-  (via (at 79.5 137) (size 0.8) (drill 0.4) (layers F.Cu B.Cu) (net 2))
   (via (at 82.5 137) (size 0.8) (drill 0.4) (layers F.Cu B.Cu) (net 2))
   (via (at 85.5 137) (size 0.8) (drill 0.4) (layers F.Cu B.Cu) (net 2))
@@
   (segment (start 43.68 114.25) (end 39.25 114.25) (width 0.5) (layer B.Cu) (net 14))
   (segment (start 44 113.93) (end 43.68 114.25) (width 0.5) (layer B.Cu) (net 14))
-  (segment (start 76.2 133.2) (end 76.2 123.4) (width 0.5) (layer F.Cu) (net 14))
-  (segment (start 75.215 135.325) (end 76.2 134.34) (width 0.5) (layer F.Cu) (net 14))
-  (segment (start 62.850001 132.950001) (end 62.850001 131.949999) (width 0.5) (layer F.Cu) (net 14))
-  (segment (start 62.450002 133.35) (end 62.850001 132.950001) (width 0.5) (layer F.Cu) (net 14))
-  (segment (start 62.850001 131.949999) (end 64.05 130.75) (width 0.5) (layer F.Cu) (net 14))
-  (segment (start 76.2 134.34) (end 76.2 133.2) (width 0.5) (layer F.Cu) (net 14))
-  (segment (start 64.05 130.75) (end 68 130.75) (width 0.5) (layer F.Cu) (net 14))
-  (segment (start 68 130.75) (end 72.575 135.325) (width 0.5) (layer F.Cu) (net 14))
-  (segment (start 72.575 135.325) (end 75.215 135.325) (width 0.5) (layer F.Cu) (net 14))
   (segment (start 78.13 106.3) (end 78.13 117.6) (width 0.5) (layer F.Cu) (net 14))
   (segment (start 77.01 105.18) (end 78.13 106.3) (width 0.5) (layer F.Cu) (net 14))
@@
   (segment (start 54.449998 65.362498) (end 55.9875 66.9) (width 0.5) (layer B.Cu) (net 14))
   (segment (start 54.449998 65.03) (end 54.449998 65.362498) (width 0.5) (layer B.Cu) (net 14))
+  (segment (start 62.850001 132.950001) (end 62.450002 133.35) (width 0.5) (layer F.Cu) (net 14))
+  (segment (start 62.850001 131.949999) (end 62.850001 132.950001) (width 0.5) (layer F.Cu) (net 14))
+  (segment (start 64.05 130.75) (end 62.850001 131.949999) (width 0.5) (layer F.Cu) (net 14))
+  (segment (start 76.2 123.4) (end 78.3 125.5) (width 0.5) (layer F.Cu) (net 14))
+  (segment (start 78.3 125.5) (end 78.3 128.35) (width 0.5) (layer F.Cu) (net 14))
+  (segment (start 76.2 130.45) (end 76.2 134.34) (width 0.5) (layer F.Cu) (net 14))
+  (segment (start 68 130.75) (end 64.05 130.75) (width 0.5) (layer F.Cu) (net 14))
+  (segment (start 76.2 134.34) (end 75.215 135.325) (width 0.5) (layer F.Cu) (net 14))
+  (segment (start 72.575 135.325) (end 68 130.75) (width 0.5) (layer F.Cu) (net 14))
+  (segment (start 78.3 128.35) (end 76.2 130.45) (width 0.5) (layer F.Cu) (net 14))
+  (segment (start 75.215 135.325) (end 72.575 135.325) (width 0.5) (layer F.Cu) (net 14))
   (via (at 60 65.8125) (size 0.8) (drill 0.4) (layers F.Cu B.Cu) (net 15))
   (segment (start 61.9375 65.8125) (end 62 65.75) (width 0.5) (layer B.Cu) (net 15))
@@
       )
     )
+  )
+  (zone (net 0) (net_name "") (layer F.Cu) (hatch edge 0.508)
+    (connect_pads (clearance 0.508))
+    (min_thickness 0.254)
+    (keepout (tracks allowed) (vias allowed) (copperpour not_allowed))
+    (fill (arc_segments 32) (thermal_gap 0.508) (thermal_bridge_width 0.508))
+    (polygon
+      (pts
+        (xy 77.55 126.5) (xy 77.55 128.3) (xy 68.95 128.3) (xy 68.95 135.55) (xy 68.05 135.55)
+        (xy 68.05 130.15) (xy 66.85 130.15) (xy 66.85 121.95) (xy 67.8 121.95) (xy 67.8 127.75)
+        (xy 68.65 127.75) (xy 68.65 126.45) (xy 77.55 126.45) (xy 77.55 126.55)
+      )
+    )
+  )
+  (zone (net 0) (net_name "") (layer F.Cu) (hatch edge 0.508)
+    (connect_pads (clearance 0.508))
+    (min_thickness 0.254)
+    (keepout (tracks allowed) (vias allowed) (copperpour not_allowed))
+    (fill (arc_segments 32) (thermal_gap 0.508) (thermal_bridge_width 0.508))
+    (polygon
+      (pts
+        (xy 79.75 137.65) (xy 77.05 137.65) (xy 77.05 136.2) (xy 79.75 136.2)
+      )
+    )
