File: 2020/Robot_Lancer/新型ラインセンサ/新型ラインセンサ/LineSensor/rancer_sensor.kicad_pcb (KiCad board)
At the start: 2 copper layers, 170 x 44 mm, 31 parts, among them P1 CONN_01X08, P2 VR-5k, P3 VR-5k, P4 VR-5k, U1 S7136, U2 QRE1113, U3 QRE1113, U4 S7136, U5 S7136

Commit message: 小谷ランサー基板
Parts:
- removed P2, P3, P4: VR-5k, _local_TMD:myVR
- added R13: 4.7k, Mizz_lib:1608_WP, F.Cu at (168.8, 157.2)
- added R14: 10k, Mizz_lib:1608_WP, F.Cu at (168.8, 159.2)
- added R15: 4.7k, Mizz_lib:1608_WP, F.Cu at (172.3, 157.2)
- added R16: 10k, Mizz_lib:1608_WP, F.Cu at (172.3, 159.2)
- C1, C2: value C -> 0.1u
- P1: value CONN_01X08 -> XH_08
- U2, U3: value QRE1113 -> TPR-105F
Connections:
- D2 pad 1: /AN_1 -> Net-(D2-Pad1)
- D3 pad 1: /AN_2 -> Net-(D3-Pad1)
- P1 pad 2: /DB_L -> GND
- P1 pad 3: /AN_1 -> /DB_L
- P1 pad 4: /DB_CENTER -> /AN_1
- P1 pad 5: /DB_R -> /DB_CENTER
- P1 pad 6: /AN_2 -> /DB_R
- P1 pad 7: Net-(P1-Pad7) -> /AN_2
- P1 pad 8: GND -> Net-(P1-Pad8)
- R10 pad 2: /AN_2 -> Net-(D3-Pad1)
- R7 pad 2: /AN_1 -> Net-(D2-Pad1)
- U2 pad 3: /AN_1 -> Net-(D2-Pad1)
- U3 pad 3: /AN_2 -> Net-(D3-Pad1)
