File: 2020/Robot_Lancer/アロエ定食/Aloe_Set_Meal.sch (KiCad schematic (older format))
At the start: 9 parts

Commit message: アロエ
Parts:
- added C? (x3): 4.7u, symbol Device:C
- added C?: 15000p, symbol Device:C
- added C?: 10u, symbol Device:C
- added C?: 22u, symbol Device:C
- added D? (x2): DIODE, symbol Miz:DIODE_rev
- added J?: BATT_IN, symbol Connector_Generic:Conn_01x02
- added L?: 22uH, symbol Device:L_Small
- added R? (x2): R, symbol Device:R
- added U?: BD9G101G, symbol Miz:BD9G101G
- added U?: AZ1086H, symbol Miz:AZ1086H
Connections:
- net +3V3: now also C?.1, U?.2 (V_OUT)
- net GND: now also C?.2, C?.2, C?.2, C?.2, J?.1 (Pin_1), R?.2, U?.1 (GND), U?.2 (GND)
- new net: C?.2, U?.1 (BST)
- new net: C?.1, R?.1, R?.1, U?.3 (FB)
- new net: C?.1, L?.1, U?.6 (Lx)
- new net +5V: C?.1, C?.1, D?.1 (K), U?.3 (V_IN)
- new net +BATT: D?.2 (A), J?.2 (Pin_2)
- new net Batt: C?.1, D?.1 (K), U?.4 (EN), U?.5 (VCC)
- new net FB: C?.2, D?.2 (A), L?.2, R?.2

Commit message: アロエ
Parts:
- added C? (x14): 4.7u, symbol Device:C
- added C? (x19): 0.1u, symbol Device:C
- added C? (x2): 470u, symbol Device:CP1
- added C? (x2): 22p, symbol Device:C
- added D? (x14): DIODE, symbol Miz:DIODE_rev
- added D?: BATT, symbol Device:LED
- added D?: MAIN_BATT, symbol Device:LED
- added D?: MOTOR_BATT, symbol Device:LED
- added D?: 5V, symbol Device:LED
- added D?: 3.3V, symbol Device:LED
- added D? (x2): LED, symbol Device:LED
- added J?: 3522-2, 3522-2, symbol SamacSys_Parts:3522-2
- added J?: MOTOR0, symbol Connector_Generic:Conn_01x02
- added J?: MOTOR1, symbol Connector_Generic:Conn_01x02
- added J?: MOTOR2, symbol Connector_Generic:Conn_01x02
- added J?: MOTOR3, symbol Connector_Generic:Conn_01x02
- added J?: MOTOR4, symbol Connector_Generic:Conn_01x02
- added J?: MOTOR5, symbol Connector_Generic:Conn_01x02
- added J?: SWD, symbol Connector_Generic:Conn_01x06
- added J?: ADC, symbol Connector_Generic:Conn_01x10
- added J?: ADC_Vdd, symbol Connector_Generic:Conn_02x10_Odd_Even
- added J?: ENC, symbol Connector_Generic:Conn_01x04
- added JP?: Jumper, symbol Device:Jumper
- added Q? (x12): NVMFD5C446NLT1G, NVMFD5C446NLWFT1G, symbol Miz:NVMFD5C446NLT1G
- added Q?: FET_N, symbol Device:Q_NMOS_GDS
- added Q?: FET_P, symbol Device:Q_PMOS_GDS
- added R? (x24): 10, symbol Device:R
- added R? (x16): 10k, symbol Device:R
- added R? (x3): 2.2k, symbol Device:R
- added R?: 510, symbol Device:R
- added R? (x3): 330, symbol Device:R
- added SW?: EMG, symbol Switch:SW_Push_SPDT
- added SW?: SW0, symbol Switch:SW_Push
- added SW?: SW1, symbol Switch:SW_Push
- added U? (x12): NCP5104, symbol Miz:NCP5104
- added U?: V23086-C1001-A403, symbol Miz:V23086-C1001-A403-myDevice
- added U?: AQM0802, symbol Miz:AQM1602
- added Y?: 8MHz, symbol Device:Crystal
Connections:
- net +3V3: now also D?.1 (K), J?.1 (Pin_1), J?.11 (Pin_11), J?.13 (Pin_13), J?.15 (Pin_15), J?.17 (Pin_17), J?.19 (Pin_19), J?.3 (Pin_3), J?.5 (Pin_5), J?.7 (Pin_7), J?.9 (Pin_9), R?.1, R?.1, R?.2
- net +5V: now also C?.2, J?.2 (Pin_2), R?.2
- net +BATT: now also C?.1, C?.1, J?.2, J?.4, R?.2
- net Batt: now also C?.1, C?.1, C?.1, C?.1, C?.1, C?.1, C?.1, C?.1, C?.1, C?.1, C?.1, C?.1, D?.2 (A), D?.2 (A), D?.2 (A), D?.2 (A), D?.2 (A), D?.2 (A), D?.2 (A), D?.2 (A), D?.2 (A), D?.2 (A), D?.2 (A), D?.2 (A), Q?.3 (S), R?.1, R?.2, R?.2, R?.2, R?.2, R?.2, R?.2, R?.2, R?.2, R?.2, R?.2, R?.2, R?.2, R?.2, SW?.1 (A), U?.1 (Vcc), U?.1 (Vcc), U?.1 (Vcc), U?.1 (Vcc), U?.1 (Vcc), U?.1 (Vcc), U?.1 (Vcc), U?.1 (Vcc), U?.1 (Vcc), U?.1 (Vcc), U?.1 (Vcc), U?.1 (Vcc)
- net GND: now also C?.1, C?.2, C?.2, C?.2, C?.2, C?.2, C?.2, C?.2, C?.2, C?.2, C?.2, C?.2, C?.2, C?.2, C?.2, C?.2, C?.2, C?.2, C?.2, D?.1 (K), D?.1 (K), D?.1 (K), D?.1 (K), D?.1 (K), D?.1 (K), D?.1 (K), J?.1 (Pin_1), J?.1 (Pin_1), J?.10 (Pin_10), J?.12 (Pin_12), J?.14 (Pin_14), J?.16 (Pin_16), J?.18 (Pin_18), J?.2 (Pin_2), J?.20 (Pin_20), J?.4 (Pin_4), J?.6 (Pin_6), J?.8 (Pin_8), Q?.3 (S), Q?.3 (S2), Q?.3 (S2), Q?.3 (S2), Q?.3 (S2), Q?.3 (S2), Q?.3 (S2), Q?.3 (S2), Q?.3 (S2), Q?.3 (S2), Q?.3 (S2), Q?.3 (S2), Q?.3 (S2), R?.2, SW?.1, SW?.1, SW?.3 (C), U?.4 (GND), U?.4 (GND), U?.4 (GND), U?.4 (GND), U?.4 (GND), U?.4 (GND), U?.4 (GND), U?.4 (GND), U?.4 (GND), U?.4 (GND), U?.4 (GND), U?.4 (GND)
- net ~RST: now also J?.5 (Pin_5)
- net OSC_IN: now reaches U?.5 (PH0)
- net OSC_IN: now also C?.1, Y?.1
- net OSC_OUT: now reaches U?.6 (PH1)
- net OSC_OUT: now also C?.1, Y?.2
- new net: R?.1, U?.3 (~SD) (x12)
- new net: R?.2, U?.5 (DRV_LO) (x12)
- new net: C?.2, U?.6 (BRIDGE) (x12)
- new net: R?.2, U?.7 (DRV_HO) (x12)
- new net: C?.1, D?.1 (K), U?.8 (VBOOT) (x12)
- new net: Q?.2 (G1), R?.1 (x12)
- new net: Q?.4 (G2), R?.1 (x12)
- new net: D?.2 (A), Q?.2 (D), U?.1
- new net: D?.1 (K), Q?.2 (D), U?.2
- new net: J?.1, J?.3, U?.4
- new net: Q?.1 (G), R?.2, SW?.2 (B)
- new net: D?.2 (A), R?.1 (x5)
- new net: C?.1, J?.1 (Pin_1) (x3)
- new net: C?.2, J?.2 (Pin_2) (x3)
- new net: J?.2 (Pin_2), JP?.1
- new net: D?.2 (A), JP?.2
- new net: D?.2 (A), R?.2 (x2)
- new net EMG_IO: Q?.1 (G), R?.1
- new net MOTOR_BATT: C?.1, C?.1, Q?.10 (D1_4), Q?.10 (D1_4), Q?.10 (D1_4), Q?.10 (D1_4), Q?.10 (D1_4), Q?.10 (D1_4), Q?.10 (D1_4), Q?.10 (D1_4), Q?.10 (D1_4), Q?.10 (D1_4), Q?.10 (D1_4), Q?.10 (D1_4), Q?.14 (D1_5), Q?.14 (D1_5), Q?.14 (D1_5), Q?.14 (D1_5), Q?.14 (D1_5), Q?.14 (D1_5), Q?.14 (D1_5), Q?.14 (D1_5), Q?.14 (D1_5), Q?.14 (D1_5), Q?.14 (D1_5), Q?.14 (D1_5), Q?.7 (D1_1), Q?.7 (D1_1), Q?.7 (D1_1), Q?.7 (D1_1), Q?.7 (D1_1), Q?.7 (D1_1), Q?.7 (D1_1), Q?.7 (D1_1), Q?.7 (D1_1), Q?.7 (D1_1), Q?.7 (D1_1), Q?.7 (D1_1), Q?.8 (D1_2), Q?.8 (D1_2), Q?.8 (D1_2), Q?.8 (D1_2), Q?.8 (D1_2), Q?.8 (D1_2), Q?.8 (D1_2), Q?.8 (D1_2), Q?.8 (D1_2), Q?.8 (D1_2), Q?.8 (D1_2), Q?.8 (D1_2), Q?.9 (D1_3), Q?.9 (D1_3), Q?.9 (D1_3), Q?.9 (D1_3), Q?.9 (D1_3), Q?.9 (D1_3), Q?.9 (D1_3), Q?.9 (D1_3), Q?.9 (D1_3), Q?.9 (D1_3), Q?.9 (D1_3), Q?.9 (D1_3), R?.2, U?.5 (N.O)
- new net Motor0_L: C?.1, J?.1 (Pin_1), Q?.1 (S1), Q?.1 (S1), Q?.1 (S1), Q?.1 (S1), Q?.1 (S1), Q?.1 (S1), Q?.11 (D2_3), Q?.11 (D2_3), Q?.11 (D2_3), Q?.11 (D2_3), Q?.11 (D2_3), Q?.11 (D2_3), Q?.12 (D2_4), Q?.12 (D2_4), Q?.12 (D2_4), Q?.12 (D2_4), Q?.12 (D2_4), Q?.12 (D2_4), Q?.13 (D2_5), Q?.13 (D2_5), Q?.13 (D2_5), Q?.13 (D2_5), Q?.13 (D2_5), Q?.13 (D2_5), Q?.5 (D2_1), Q?.5 (D2_1), Q?.5 (D2_1), Q?.5 (D2_1), Q?.5 (D2_1), Q?.5 (D2_1), Q?.6 (D2_2), Q?.6 (D2_2), Q?.6 (D2_2), Q?.6 (D2_2), Q?.6 (D2_2), Q?.6 (D2_2)
- new net Motor0_L_PWM: U?.2 (IN), U?.2 (IN), U?.2 (IN), U?.2 (IN), U?.2 (IN), U?.2 (IN)
- new net Motor0_R: C?.2, J?.2 (Pin_2), Q?.1 (S1), Q?.1 (S1), Q?.1 (S1), Q?.1 (S1), Q?.1 (S1), Q?.1 (S1), Q?.11 (D2_3), Q?.11 (D2_3), Q?.11 (D2_3), Q?.11 (D2_3), Q?.11 (D2_3), Q?.11 (D2_3), Q?.12 (D2_4), Q?.12 (D2_4), Q?.12 (D2_4), Q?.12 (D2_4), Q?.12 (D2_4), Q?.12 (D2_4), Q?.13 (D2_5), Q?.13 (D2_5), Q?.13 (D2_5), Q?.13 (D2_5), Q?.13 (D2_5), Q?.13 (D2_5), Q?.5 (D2_1), Q?.5 (D2_1), Q?.5 (D2_1), Q?.5 (D2_1), Q?.5 (D2_1), Q?.5 (D2_1), Q?.6 (D2_2), Q?.6 (D2_2), Q?.6 (D2_2), Q?.6 (D2_2), Q?.6 (D2_2), Q?.6 (D2_2)
- new net Motor0_R_PWM: U?.2 (IN), U?.2 (IN), U?.2 (IN), U?.2 (IN), U?.2 (IN), U?.2 (IN)
- new net Motor1_L: C?.1, J?.1 (Pin_1)
- new net Motor1_R: C?.2, J?.2 (Pin_2)
- new net SW0: R?.2, SW?.2
- new net SW1: R?.2, SW?.2
- new net SWCLK: J?.3 (Pin_3)
- new net SWDIO: J?.4 (Pin_4)
- new net TIMx_CH1: J?.4 (Pin_4)
- new net TIMx_CH2: J?.3 (Pin_3)
- no-connect marks 0 -> 2
Other:
- moved on the sheet: C?, D?, J?, L?, R?, U?

Commit message: ALoe
Parts:
- removed U?: AQM0802, symbol Miz:AQM1602
- added C? (x2): 0.1u, symbol Device:C
- added D? (x3): LED, symbol Device:LED
- added D?: DIODE, symbol Miz:DIODE_rev
- added J?: BATT_IN, symbol Connector_Generic:Conn_01x02
- added J?: USB_B_Micro, symbol Connector:USB_B_Micro
- added JP?: Relay_JP, symbol Device:Jumper
- added R? (x3): 10k, symbol Device:R
- added R? (x3): 330, symbol Device:R
- added R? (x2): 100, symbol Device:R
- added SW?: RST, symbol Switch:SW_Push
- added U?: ROTARY, symbol Miz:SW_ROTARY_16
- added U?: MCP2221A, symbol Miz:MCP2221A
- D?: value LED -> LED0
- D?: value LED -> LED1
Connections:
- net +3V3: now also C?.1, R?.1, R?.1, R?.2, R?.2, R?.2, R?.2, U?.11 (Vusb)
- net +5V: now also D?.1 (K)
- net +BATT: now also J?.2 (Pin_2)
- net GND: now also C?.1, C?.2, J?.1 (Pin_1), J?.5 (GND), JP?.1, SW?.2, U?.14 (Vss), U?.2 (C), U?.5 (C)
- net Motor0_L: no longer Q?.1 (S1), Q?.1 (S1), Q?.1 (S1), Q?.1 (S1), Q?.1 (S1), Q?.11 (D2_3), Q?.11 (D2_3), Q?.11 (D2_3), Q?.11 (D2_3), Q?.11 (D2_3), Q?.12 (D2_4), Q?.12 (D2_4), Q?.12 (D2_4), Q?.12 (D2_4), Q?.12 (D2_4), Q?.13 (D2_5), Q?.13 (D2_5), Q?.13 (D2_5), Q?.13 (D2_5), Q?.13 (D2_5), Q?.5 (D2_1), Q?.5 (D2_1), Q?.5 (D2_1), Q?.5 (D2_1), Q?.5 (D2_1), Q?.6 (D2_2), Q?.6 (D2_2), Q?.6 (D2_2), Q?.6 (D2_2), Q?.6 (D2_2)
- net Motor0_L_PWM: no longer U?.2 (IN), U?.2 (IN), U?.2 (IN), U?.2 (IN), U?.2 (IN)
- net Motor0_R: no longer Q?.1 (S1), Q?.1 (S1), Q?.1 (S1), Q?.1 (S1), Q?.1 (S1), Q?.11 (D2_3), Q?.11 (D2_3), Q?.11 (D2_3), Q?.11 (D2_3), Q?.11 (D2_3), Q?.12 (D2_4), Q?.12 (D2_4), Q?.12 (D2_4), Q?.12 (D2_4), Q?.12 (D2_4), Q?.13 (D2_5), Q?.13 (D2_5), Q?.13 (D2_5), Q?.13 (D2_5), Q?.13 (D2_5), Q?.5 (D2_1), Q?.5 (D2_1), Q?.5 (D2_1), Q?.5 (D2_1), Q?.5 (D2_1), Q?.6 (D2_2), Q?.6 (D2_2), Q?.6 (D2_2), Q?.6 (D2_2), Q?.6 (D2_2)
- net Motor0_R_PWM: no longer U?.2 (IN), U?.2 (IN), U?.2 (IN), U?.2 (IN), U?.2 (IN)
- net Motor1_L: now also Q?.1 (S1), Q?.11 (D2_3), Q?.12 (D2_4), Q?.13 (D2_5), Q?.5 (D2_1), Q?.6 (D2_2)
- net Motor1_R: now also Q?.1 (S1), Q?.11 (D2_3), Q?.12 (D2_4), Q?.13 (D2_5), Q?.5 (D2_1), Q?.6 (D2_2)
- net ~RST: now also C?.2, SW?.1
- net at D?.2 (A), Q?.2 (D), U?.1: now also JP?.2
- net Motor2_L: now reaches C?.1, J?.1 (Pin_1)
- net Motor2_L: now also Q?.1 (S1), Q?.11 (D2_3), Q?.12 (D2_4), Q?.13 (D2_5), Q?.5 (D2_1), Q?.6 (D2_2)
- net Motor2_R: now reaches C?.2, J?.2 (Pin_2)
- net Motor2_R: now also Q?.1 (S1), Q?.11 (D2_3), Q?.12 (D2_4), Q?.13 (D2_5), Q?.5 (D2_1), Q?.6 (D2_2)
- net Motor3_L: now reaches J?.1 (Pin_1)
- net Motor3_L: now also C?.1, Q?.1 (S1), Q?.11 (D2_3), Q?.12 (D2_4), Q?.13 (D2_5), Q?.5 (D2_1), Q?.6 (D2_2)
- net Motor3_R: now reaches J?.2 (Pin_2)
- net Motor3_R: now also C?.2, Q?.1 (S1), Q?.11 (D2_3), Q?.12 (D2_4), Q?.13 (D2_5), Q?.5 (D2_1), Q?.6 (D2_2)
- net Motor4_L: now reaches C?.1, J?.1 (Pin_1)
- net Motor4_L: now also Q?.1 (S1), Q?.11 (D2_3), Q?.12 (D2_4), Q?.13 (D2_5), Q?.5 (D2_1), Q?.6 (D2_2)
- net Motor4_R: now reaches C?.2, J?.2 (Pin_2)
- net Motor4_R: now also Q?.1 (S1), Q?.11 (D2_3), Q?.12 (D2_4), Q?.13 (D2_5), Q?.5 (D2_1), Q?.6 (D2_2)
- net Motor5_L: now reaches C?.1, J?.1 (Pin_1)
- net Motor5_L: now also Q?.1 (S1), Q?.11 (D2_3), Q?.12 (D2_4), Q?.13 (D2_5), Q?.5 (D2_1), Q?.6 (D2_2)
- net Motor5_R: now reaches C?.2, J?.2 (Pin_2)
- net Motor5_R: now also Q?.1 (S1), Q?.11 (D2_3), Q?.12 (D2_4), Q?.13 (D2_5), Q?.5 (D2_1), Q?.6 (D2_2)
- net ADC0: now reaches J?.1 (Pin_1)
- net ADC9: now reaches J?.10 (Pin_10)
- net ADC1: now reaches J?.2 (Pin_2)
- net ADC2: now reaches J?.3 (Pin_3)
- net ADC3: now reaches J?.4 (Pin_4)
- net ADC4: now reaches J?.5 (Pin_5)
- net ADC5: now reaches J?.6 (Pin_6)
- net ADC6: now reaches J?.7 (Pin_7)
- net ADC7: now reaches J?.8 (Pin_8)
- net ADC8: now reaches J?.9 (Pin_9)
- net LED0: now reaches R?.1
- net LED1: now reaches R?.1
- net TIMx_CH1: no longer names the net of J?.4 (Pin_4)
- net TIMx_CH1: now also R?.1, R?.2
- net TIMx_CH2: no longer names the net of J?.3 (Pin_3)
- net TIMx_CH2: now also R?.1, R?.2
- new net: D?.1 (K), U?.2 (GP0)
- new net: D?.1 (K), U?.3 (GP1)
- new net: R?.1, U?.4 (nRST)
- new net: D?.1 (K), U?.7 (GP2)
- new net: D?.2 (A), R?.1 (x3)
- new net: D?.2 (A), J?.1 (VBUS)
- new net ADRESS0: U?.3 (1)
- new net ADRESS1: U?.1 (2)
- new net ADRESS2: U?.4
- new net ADRESS3: U?.6 (8)
- new net D+: J?.3 (D+), U?.13 (D+)
- new net D-: J?.2 (D-), U?.12 (D-)
- new net ENC_CH1: R?.2
- new net ENC_CH2: R?.2
- new net Motor1_L_PWM: U?.2 (IN)
- new net Motor1_R_PWM: U?.2 (IN)
- new net Motor2_L_PWM: U?.2 (IN)
- new net Motor2_R_PWM: U?.2 (IN)
- new net Motor3_L_PWM: U?.2 (IN)
- new net Motor3_R_PWM: U?.2 (IN)
- new net Motor4_L_PWM: U?.2 (IN)
- new net Motor4_R_PWM: U?.2 (IN)
- new net Motor5_L_PWM: U?.2 (IN)
- new net Motor5_R_PWM: U?.2 (IN)
- new net SERIALx_RX: U?.6 (UTx)
- new net SERIALx_TX: U?.5 (URx)
- no-connect marks 2 -> 7
Other:
- note added: "EMG is HIGH -> EMG OFF"
- moved on the sheet: C?, D?, J?, L?, Q?, R?, SW?, U?

Commit message: back up
Parts:
- added J?: microSD, symbol Connector:Micro_SD_Card_Det_Hirose_DM3AT
- added U19: LOGO, Mizz_lib:Mini_Monster, symbol Miz:LOGO
- C1, C10, C12, C14, C15, C16, C17, C18, C19, C2, C20, C21, C22, C23, C24, C3, C31, C32, C33, C34, C35, C36, C4, C44, C45, C46, C5, C50, C51, C52, C6, C7: renamed from C?; footprint (none) -> Capacitor_SMD:C_0603_1608Metric
- D2, D22, D23, D24, D25, D26, D3, D4, D5, D6: renamed from D?; footprint (none) -> LED_SMD:LED_0603_1608Metric
- J10, J11, J12, J6, J7, J8: renamed from J?; footprint (none) -> Mizz_lib:XT30_F
- J13, J9: renamed from J?; footprint (none) -> Mizz_lib:XT60_F
- J14: renamed from J?; footprint 3522-2 -> SamacSys_Parts:3522-2
- L1: renamed from L?; footprint (none) -> Mizz_lib:Inductor_Taiyo-Yuden_NR-60xx
- Q1, Q10, Q11, Q12, Q2, Q3, Q4, Q5, Q6, Q7, Q8, Q9: renamed from Q?; footprint NVMFD5C446NLWFT1G -> Mizz_lib:NVMFD5C446NLWFT1G
- Q13, Q14: renamed from Q?; footprint (none) -> Package_TO_SOT_SMD:SOT-23W
- R1, R10, R11, R12, R13, R14, R15, R16, R17, R18, R19, R2, R20, R21, R22, R23, R24, R25, R26, R27, R28, R29, R3, R30, R31, R32, R33, R34, R35, R36, R37, R38, R39, R4, R40, R41, R42, R43, R44, R45, R46, R47, R48, R49, R5, R50, R51, R52, R53, R54, R55, R56, R57, R58, R6, R7, R8, R9: renamed from R?; footprint (none) -> Resistor_SMD:R_0603_1608Metric
- SW1, SW2, SW3: renamed from SW?; footprint (none) -> Button_Switch_SMD:SW_SPST_CK_RS282G05A3
- SW4: renamed from SW?; footprint (none) -> Mizz_lib:2MS1-T1-B4-VS2-Q-E
- U1: renamed from U?; footprint (none) -> Package_SO:TSOP-6_1.65x3.05mm_P0.95mm
- U10, U11, U12, U13, U14, U15, U16, U17, U6, U7, U8, U9: renamed from U?; footprint (none) -> Package_SO:SOIC-8_3.9x4.9mm_P1.27mm
- U18: renamed from U?; footprint (none) -> Mizz_lib:V23086-C1001-A403
- U2: renamed from U?; footprint (none) -> Package_SO:SOIC-14_3.9x8.7mm_P1.27mm
- U4: renamed from U?; footprint (none) -> Mizz_lib:rotary_0F
- U5: renamed from U?; footprint (none) -> Package_TO_SOT_SMD:SOT-223-3_TabPin2
- Y1: renamed from Y?; footprint (none) -> Mizz_lib:Crystal_SMD_5032_2Pads
- gave numbers to parts that had none: 45
Connections:
- net ADC0: now also U3.8 (PC0)
- net ADC1: now also U3.9 (PC1)
- net ADC2: now also U3.10 (PC2)
- net ADC3: now also U3.11 (PC3)
- net Batt: no longer SW4.1 (A)
- no-connect marks 7 -> 8
Other:
- moved on the sheet: C3, D2, D3, D4, D5, D6, D8, J4, R10, R11, R2, R3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
