File: 2020/Robot_Lancer/アロエ定食/Aloe_Set_Meal.sch (KiCad schematic (older format))
At the start: 229 parts, among them J1 SWD, J10 MOTOR1, J11 MOTOR3, J12 MOTOR5, J13 BATT_IN, J14 3522-2, J15 microSD, J16 SERIAL1, J17 VOLTMETER, J18 TO_VOLTMETER, J2 ADC, J3 ADC_Vdd, J4 SERIAL0, J5 ENC, J6 MOTOR0, J7 MOTOR2, J8 MOTOR4, J9 SERVO, Q1 NVMFD5C446NLT1G, Q10 NVMFD5C446NLT1G, Q11 NVMFD5C446NLT1G, Q12 NVMFD5C446NLT1G, Q13 FET_P, Q14 FET_N, Q15 FET_P, Q16 NPN, Q2 NVMFD5C446NLT1G, Q3 NVMFD5C446NLT1G, Q4 NVMFD5C446NLT1G, Q5 NVMFD5C446NLT1G, Q6 NVMFD5C446NLT1G, Q7 NVMFD5C446NLT1G, Q8 NVMFD5C446NLT1G, Q9 NVMFD5C446NLT1G, SW1 RST, SW2 SW0, SW3 SW1, SW4 EMG, SW5 MAIN_SW, U1 BD9G101G, U10 NCP5104, U11 NCP5104, U12 NCP5104, U13 NCP5104, U14 NCP5104, U15 NCP5104, U16 NCP5104, U17 NCP5104, U18 V23086-C1001, U19 LOGO, U2 MCP2221A, U20 LOGO, U21 LOGO, U22 AQM0802, U23 74HCT04, U24 74HC02, U25 74HC02, U26 74HC02, U3 STM32F446RETx, U4 ROTARY, U5 AZ1086H, U6 NCP5104, U7 NCP5104, U8 NCP5104, U9 NCP5104, Y1 8MHz

Commit message: つかれた
Parts:
- added D30: DIODE, Diode_SMD:D_SOD-123, symbol Miz:DIODE_rev
- added U27: LOGO, Mizz_lib:AloeSetMeal_Mask_50x5.8, symbol Miz:LOGO
- C19, C20, C21, C22, C23, C24, C31, C32, C33, C34, C35, C36: footprint Capacitor_SMD:C_0603_1608Metric -> Mizz_lib:1608_WP
- C6: value 15000p -> 0.1u
- R16, R17, R18, R19, R20, R21, R34, R35, R36, R37, R38, R39: footprint Resistor_SMD:R_0603_1608Metric -> Mizz_lib:1608_WP
- U21: footprint Mizz_lib:Goukazal_10.0x7.5_S.Itoh_silk -> Mizz_lib:Goukazal_15.0x11.3_S.Itoh_silk
Connections:
- net +3V3: now also U2.1 (Vdd)
- net ADC7: now also U3.24 (PC4); no longer U3.26 (PB0)
- net ADC8: now also U3.25 (PC5); no longer U3.24 (PC4)
- net ADC9: now also U3.26 (PB0); no longer U3.25 (PC5)
- net GND: now also D30.2 (A)
- net at C6.1, L1.1, U1.6 (Lx): now also D30.1 (K)
Other:
- moved on the sheet: C43, C47, C48, C49, D21
