File: 2020/Robot_Lancer/アロエ定食/Aloe_Set_Meal.sch (KiCad schematic (older format))
At the start: 231 parts, among them J1 SWD, J10 MOTOR1, J11 MOTOR3, J12 MOTOR5, J13 BATT_IN, J14 3522-2, J15 microSD, J16 SERIAL1, J17 VOLTMETER, J18 TO_VOLTMETER, J2 ADC, J3 ADC_Vdd, J4 SERIAL0, J5 ENC, J6 MOTOR0, J7 MOTOR2, J8 MOTOR4, J9 SERVO, Q1 NVMFD5C446NLT1G, Q10 NVMFD5C446NLT1G, Q11 NVMFD5C446NLT1G, Q12 NVMFD5C446NLT1G, Q13 FET_P, Q14 FET_N, Q15 FET_P, Q16 NPN, Q2 NVMFD5C446NLT1G, Q3 NVMFD5C446NLT1G, Q4 NVMFD5C446NLT1G, Q5 NVMFD5C446NLT1G, Q6 NVMFD5C446NLT1G, Q7 NVMFD5C446NLT1G, Q8 NVMFD5C446NLT1G, Q9 NVMFD5C446NLT1G, SW1 RST, SW2 SW0, SW3 SW1, SW4 EMG, SW5 MAIN_SW, U1 BD9G101G, U10 NCP5104, U11 NCP5104, U12 NCP5104, U13 NCP5104, U14 NCP5104, U15 NCP5104, U16 NCP5104, U17 NCP5104, U18 V23086-C1001, U19 LOGO, U2 MCP2221A, U20 LOGO, U21 LOGO, U22 AQM0802, U23 74HCT04, U24 74HC02, U25 74HC02, U26 74HC02, U27 LOGO, U3 STM32F446RETx, U4 ROTARY, U5 AZ1086H, U6 NCP5104, U7 NCP5104, U8 NCP5104, U9 NCP5104, Y1 8MHz

Commit message: ラインセンサ寸法線・和基板
Parts:
- added D31: 5V_dcdc, LED_SMD:LED_0603_1608Metric, symbol Device:LED
- added R70: 510, Resistor_SMD:R_0603_1608Metric, symbol Device:R
- JP1: footprint Mizz_lib:GS2 -> Connector_PinHeader_2.54mm:PinHeader_1x02_P2.54mm_Vertical
Connections:
- net +BATT: no longer C48.1, C49.1
- net 5Vc: now also R70.2
- net GND: now also D31.1 (K)
- net MOTOR_BATT: now also C48.1, C49.1
- new net: D31.2 (A), R70.1
Other:
- moved on the sheet: C44, C45, C46, C50, C51, C52, D25, D26, D29, J10, J11, J12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

Commit message: pushできなかったからできるようにして,以前の内容をpush
Connections:
- net ADRESS2: now also U3.57 (PB5); no longer U3.56 (PB4)
- net ADRESS3: now also U3.56 (PB4); no longer U3.57 (PB5)
Changed lines of the file:
@@
 ENC_CH2
 Text Label 3975 5575 0    50   ~ 0
+ADRESS2
+Text Label 3975 5475 0    50   ~ 0
 ADRESS3
-Text Label 3975 5475 0    50   ~ 0
-ADRESS2
 Text Label 3975 5375 0    50   ~ 0
 ADRESS1

Commit message: 信号線の配線終わり
Connections:
- net ADRESS0: now also U3.56 (PB4); no longer U3.54 (PD2)
- net ADRESS1: now also U3.57 (PB5); no longer U3.55 (PB3)
- net ADRESS2: now also U3.55 (PB3); no longer U3.57 (PB5)
- net ADRESS3: now also U3.54 (PD2); no longer U3.56 (PB4)
- net EMG_IO: now also U3.45 (PA12); no longer U3.4 (PC15)
- net Motor0_CW: now also U3.61 (PB8); no longer U3.37 (PC6)
- net Motor0_PWM: now also U3.59 (PB7); no longer U3.41 (PA8)
- net Motor1_CW: now also U3.62 (PB9); no longer U3.38 (PC7)
- net Motor1_PWM: now also U3.58 (PB6); no longer U3.42 (PA9)
- net Motor2_CW: now also U3.40 (PC9); no longer U3.39 (PC8)
- net Motor2_PWM: now also U3.44 (PA11); no longer U3.43 (PA10)
- net Motor3_CW: now also U3.39 (PC8); no longer U3.40 (PC9)
- net Motor3_PWM: now also U3.43 (PA10); no longer U3.44 (PA11)
- net Motor4_CW: now also U3.38 (PC7); no longer U3.61 (PB8)
- net Motor4_PWM: now also U3.41 (PA8); no longer U3.58 (PB6)
- net Motor5_CW: now also U3.37 (PC6); no longer U3.62 (PB9)
- net Motor5_PWM: now also U3.42 (PA9); no longer U3.59 (PB7)
Changed lines of the file:
@@
 	1    0    0    -1
 $EndComp
-Text Label 2575 6475 2    50   ~ 0
+Text Label 3975 4575 0    50   ~ 0
 EMG_IO
 $Comp
@@
 Text Label 2575 5375 2    50   ~ 0
 ADC7
-Text Notes 1275 6475 0    50   ~ 0
+Text Notes 5350 4575 2    50   ~ 0
 EMG is HIGH -> EMG OFF
 $Comp
@@
 Wire Wire Line
 	21650 10925 21725 10925
-Text Label 3975 4175 0    50   ~ 0
-Motor0_PWM
-Text Label 3975 4275 0    50   ~ 0
+Text Label 3975 4375 0    50   ~ 0
+Motor3_PWM
+Text Label 3975 4475 0    50   ~ 0
+Motor2_PWM
+Text Label 3975 5675 0    50   ~ 0
 Motor1_PWM
-Text Label 3975 4375 0    50   ~ 0
-Motor2_PWM
-Text Label 3975 4475 0    50   ~ 0
-Motor3_PWM
-Text Label 3975 5675 0    50   ~ 0
-Motor4_PWM
 Connection ~ 21825 6925
 Wire Wire Line
@@
 Text Label 3975 4075 0    50   ~ 0
 ENC_CH2
-Text Label 3975 5575 0    50   ~ 0
+Text Label 3975 5475 0    50   ~ 0
+ADRESS0
+Text Label 3975 5375 0    50   ~ 0
 ADRESS2
-Text Label 3975 5475 0    50   ~ 0
+Text Label 2575 4775 2    50   ~ 0
 ADRESS3
-Text Label 3975 5375 0    50   ~ 0
-ADRESS1
-Text Label 2575 4775 2    50   ~ 0
-ADRESS0
 $Comp
 L Miz:MCP2221A U2
@@
 Motor5_L_PWM
 Text Label 2575 5575 2    50   ~ 0
-Motor0_CW
+Motor5_CW
 Text Label 3975 5775 0    50   ~ 0
-Motor5_PWM
+Motor0_PWM
 Text Notes 1000 5575 0    50   ~ 0
 Brake is LOW -> Brake
@@
 Connection ~ 7075 7100
 Text Label 2575 5675 2    50   ~ 0
-Motor1_CW
+Motor4_CW
 Text Label 2575 5775 2    50   ~ 0
+Motor3_CW
+Text Label 2575 5875 2    50   ~ 0
 Motor2_CW
-Text Label 2575 5875 2    50   ~ 0
-Motor3_CW
 Text Label 7025 1450 2    50   ~ 0
 Motor0_CW
 Text Label 3975 5875 0    50   ~ 0
-Motor4_CW
+Motor0_CW
 Text Label 3975 5975 0    50   ~ 0
-Motor5_CW
+Motor1_CW
 Text Label 7025 5850 2    50   ~ 0
 Motor4_CW
@@
 Connection ~ 21375 3700
 Connection ~ 21000 3700
+Text Label 3975 5575 0    50   ~ 0
+ADRESS1
+Text Label 3975 4175 0    50   ~ 0
+Motor4_PWM
+Text Label 3975 4275 0    50   ~ 0
+Motor5_PWM
 $EndSCHEMATC
