File: 2020/Robot_Lancer/アロエ定食/Aloe_Set_Meal.kicad_pcb (KiCad board)
At the start: 2 copper layers, 0 parts

Commit message: 小谷ランサー基板
Parts:
- added C1: 22p, Capacitor_SMD:C_0603_1608Metric, F.Cu at (-17.2, 95.2)
- added C10: 0.1u, Capacitor_SMD:C_0603_1608Metric, F.Cu at (-35.0, 124.9)
- added C11: 4.7u, Capacitor_SMD:C_0805_2012Metric, F.Cu at (-43.3, 112.5)
- added C12: 0.1u, Capacitor_SMD:C_0603_1608Metric, F.Cu at (-1.20, 90.8)
- added C13: 10u, Capacitor_SMD:C_0805_2012Metric, F.Cu at (-21.5, 93.4)
- added C14: 0.1u, Capacitor_SMD:C_0603_1608Metric, F.Cu at (-31.1, 112.7)
- added C15: 0.1u, Capacitor_SMD:C_0603_1608Metric, F.Cu at (-13.7, 102.7)
- added C16: 0.1u, Capacitor_SMD:C_0603_1608Metric, F.Cu at (3.39, 85.8)
- added C17: 1u, Capacitor_SMD:C_0603_1608Metric, F.Cu at (-5.21, 93.5)
- added C18: 22u, Capacitor_SMD:C_0603_1608Metric, F.Cu at (-34.6, 122.3)
- added C19: 0.1u, Capacitor_SMD:C_0603_1608Metric, F.Cu at (-20.1, 107.7)
- added C2: 0.1u, Capacitor_SMD:C_0603_1608Metric, F.Cu at (7.73, 74.4)
- added C20: 0.1u, Capacitor_SMD:C_0603_1608Metric, F.Cu at (7.73, 79.4)
- added C21: 0.1u, Capacitor_SMD:C_0603_1608Metric, F.Cu at (-30.6, 117.7)
- added C22: 0.1u, Capacitor_SMD:C_0603_1608Metric, F.Cu at (-1.20, 88.3)
- added C23: 0.1u, Capacitor_SMD:C_0603_1608Metric, F.Cu at (-9.22, 96.0)
- added C24: 0.1u, Capacitor_SMD:C_0603_1608Metric, F.Cu at (-23.1, 110.2)
- added C25: 4.7u, Capacitor_SMD:C_0805_2012Metric, F.Cu at (-12.9, 85.0)
- added C26: 4.7u, Capacitor_SMD:C_0805_2012Metric, F.Cu at (3.80, 69.2)
- added C27: 4.7u, Capacitor_SMD:C_0805_2012Metric, F.Cu at (-84.0, 91.2)
- added C28: 4.7u, Capacitor_SMD:C_0805_2012Metric, F.Cu at (-29.9, 98.9)
- added C29: 4.7u, Capacitor_SMD:C_0805_2012Metric, F.Cu at (-8.51, 78.3)
- added C3: 0.1u, Capacitor_SMD:C_0603_1608Metric, F.Cu at (-16.1, 105.3)
- added C30: 4.7u, Capacitor_SMD:C_0805_2012Metric, F.Cu at (-34.3, 99.1)
- added C31: 0.1u, Capacitor_SMD:C_0603_1608Metric, F.Cu at (-30.6, 115.2)
- added C32: 0.1u, Capacitor_SMD:C_0603_1608Metric, F.Cu at (-27.1, 112.7)
- added C33: 0.1u, Capacitor_SMD:C_0603_1608Metric, F.Cu at (-17.7, 102.7)
- added C34: 0.1u, Capacitor_SMD:C_0603_1608Metric, F.Cu at (-0.62, 85.8)
- added C35: 0.1u, Capacitor_SMD:C_0603_1608Metric, F.Cu at (7.73, 76.9)
- added C36: 0.1u, Capacitor_SMD:C_0603_1608Metric, F.Cu at (-34.6, 119.8)
- added C37: 4.7u, Capacitor_SMD:C_0805_2012Metric, F.Cu at (-56.1, 126.3)
- added C38: 4.7u, Capacitor_SMD:C_0805_2012Metric, F.Cu at (-21.5, 90.4)
- added C39: 4.7u, Capacitor_SMD:C_0805_2012Metric, F.Cu at (-78.8, 84.9)
- added C4: 22p, Capacitor_SMD:C_0603_1608Metric, F.Cu at (-26.6, 117.7)
- added C40: 4.7u, Capacitor_SMD:C_0805_2012Metric, F.Cu at (-46.8, 118.2)
- added C41: 4.7u, Capacitor_SMD:C_0805_2012Metric, F.Cu at (3.88, 66.2)
- added C42: 4.7u, Capacitor_SMD:C_0805_2012Metric, F.Cu at (-31.4, 102.1)
- added C43: 470u, Mizz_lib:CAPAE1300X1400N, F.Cu at (-12.7, 34.8)
- added C44: 0.1u, Capacitor_SMD:C_0603_1608Metric, F.Cu at (-0.62, 83.3)
- added C45: 0.1u, Capacitor_SMD:C_0603_1608Metric, F.Cu at (-5.21, 88.5)
- added C46: 0.1u, Capacitor_SMD:C_0603_1608Metric, F.Cu at (-27.1, 110.2)
- added C47: 470u, Mizz_lib:CAPAE1300X1400N, F.Cu at (-12.7, 50.1)
- added C48: 4.7u, Capacitor_SMD:C_0805_2012Metric, F.Cu at (-36.4, 107.0)
- added C49: 4.7u, Capacitor_SMD:C_0805_2012Metric, F.Cu at (-51.2, 121.6)
- added C5: 4.7u, Capacitor_SMD:C_0603_1608Metric, F.Cu at (2.81, 88.3)
- added C50: 0.1u, Capacitor_SMD:C_0603_1608Metric, F.Cu at (-17.7, 100.2)
- added C51: 0.1u, Capacitor_SMD:C_0603_1608Metric, F.Cu at (-9.22, 91.0)
- added C52: 0.1u, Capacitor_SMD:C_0603_1608Metric, F.Cu at (-43.0, 125.3)
- added C53: 0.1u, Capacitor_SMD:C_0603_1608Metric, F.Cu at (-34.6, 117.3)
- added C54: 0.1u, Capacitor_SMD:C_0603_1608Metric, F.Cu at (-40.9, 144.0)
- added C55: 1u, Capacitor_SMD:C_0603_1608Metric, F.Cu at (-40.9, 146.5)
- added C56: 1u, Capacitor_SMD:C_0603_1608Metric, F.Cu at (-36.9, 144.0)
- added C6: 15000p, Capacitor_SMD:C_0603_1608Metric, F.Cu at (-5.21, 96.0)
- added C7: 2.2u, Capacitor_SMD:C_0603_1608Metric, F.Cu at (-19.1, 110.2)
- added C8: 4.7u, Capacitor_SMD:C_0805_2012Metric, F.Cu at (-17.3, 85.0)
- added C9: 4.7u, Capacitor_SMD:C_0603_1608Metric, F.Cu at (7.73, 81.9)
- added D1: DIODE, Diode_SMD:D_SOD-123, F.Cu at (-39.4, 99.3)
- added D10: DIODE, Diode_SMD:D_SOD-123, F.Cu at (-26.5, 91.4)
- added D11: DIODE, Diode_SMD:D_SOD-123, F.Cu at (-41.4, 106.0)
- added D12: DIODE, Diode_SMD:D_SOD-123, F.Cu at (-61.2, 126.2)
- added D13: DIODE, Diode_SMD:D_SOD-123, F.Cu at (-13.6, 78.5)
- added D14: DIODE, Diode_SMD:D_SOD-123, F.Cu at (-61.2, 122.9)
- added D15: DIODE, Diode_SMD:D_SOD-123, F.Cu at (-46.1, 89.3)
- added D16: DIODE, Diode_SMD:D_SOD-123, F.Cu at (-6.64, 70.2)
- added D17: DIODE, Diode_SMD:D_SOD-123, F.Cu at (-41.4, 102.7)
- added D18: DIODE, Diode_SMD:D_SOD-123, F.Cu at (-100.5, 115.0)
- added D19: DIODE, Diode_SMD:D_SOD-123, F.Cu at (-67.0, 126.2)
- added D2: LED, LED_SMD:LED_0603_1608Metric, F.Cu at (-108.6, 126.4)
- added D20: DIODE, Diode_SMD:D_SOD-123, F.Cu at (-57.6, 115.3)
- added D21: DIODE, Diode_SMD:D_SOD-123, F.Cu at (-57.6, 118.6)
- added D22: BATT, LED_SMD:LED_0603_1608Metric, F.Cu at (-32.7, 71.7)
- added D23: MAIN_BATT, LED_SMD:LED_0603_1608Metric, F.Cu at (-84.7, 126.5)
- added D24: MOTOR_BATT, LED_SMD:LED_0603_1608Metric, F.Cu at (-28.7, 71.7)
- added D25: 5V, LED_SMD:LED_0603_1608Metric, F.Cu at (-80.7, 126.5)
- added D26: 3.3V, LED_SMD:LED_0603_1608Metric, F.Cu at (-46.9, 92.2)
- added D27: DIODE, Diode_SMD:D_SOD-123, F.Cu at (-13.6, 81.8)
- added D28: DIODE, Diode_SMD:D_SOD-123, F.Cu at (-67.0, 122.9)
- added D3: LED, LED_SMD:LED_0603_1608Metric, F.Cu at (-104.5, 126.4)
- added D4: LED, LED_SMD:LED_0603_1608Metric, F.Cu at (-41.8, 66.6)
- added D5: LED0, LED_SMD:LED_0603_1608Metric, F.Cu at (-37.7, 66.6)
- added D6: LED1, LED_SMD:LED_0603_1608Metric, F.Cu at (-100.5, 126.4)
- added D7: DIODE, Diode_SMD:D_SOD-123, F.Cu at (-41.4, 109.4)
- added D8: DIODE, Diode_SMD:D_SOD-123, F.Cu at (-26.5, 94.7)
- added D9: DIODE, Diode_SMD:D_SOD-123, F.Cu at (-51.9, 118.4)
- added J1: SWD, Connector_PinHeader_2.54mm:PinHeader_1x06_P2.54mm_Vertical, F.Cu at (-78.7, 68.4)
- added J10: MOTOR1, Mizz_lib:XT30_F, F.Cu at (-45.5, 68.8)
- added J11: MOTOR3, Mizz_lib:XT30_F, F.Cu at (-57.2, 75.4)
- added J12: MOTOR5, Mizz_lib:XT30_F, F.Cu at (-72.3, 94.3)
- added J13: BATT_IN, Mizz_lib:XT60_M, F.Cu at (189.0, 36.5)
- added J14: 3522-2, SamacSys_Parts:3522-2, F.Cu at (175.0, 44.0)
- added J15: microSD, Connector_Card:microSD_HC_Hirose_DM3AT-SF-PEJM5, F.Cu at (-29.9, 36.5)
- added J16: SERIAL1, Mizz_lib:XA_4P, F.Cu at (-107.3, 121.2)
- added J2: ADC, Connector_PinHeader_2.54mm:PinHeader_1x10_P2.54mm_Vertical, F.Cu at (-73.5, 62.5)
- added J3: ADC_Vdd, Connector_PinHeader_2.54mm:PinHeader_2x10_P2.54mm_Vertical, F.Cu at (-108.3, 92.0)
- added J4: SERIAL0, Connector_USB:USB_Micro-B_Molex_47346-0001, F.Cu at (-80.6, 114.3)
- added J5: ENC, Mizz_lib:XA_4P, F.Cu at (-54.6, 64.2)
- added J6: MOTOR0, Mizz_lib:XT30_F, F.Cu at (-70.4, 81.4)
- added J7: MOTOR2, Mizz_lib:XT30_F, F.Cu at (-57.1, 68.8)
- added J8: MOTOR4, Mizz_lib:XT30_F, F.Cu at (-59.7, 88.0)
- added JP1: SWD_3.3V_JP, Mizz_lib:GS2, F.Cu at (8.08, 62.0)
- added JP2: Relay_JP, Connector_PinHeader_2.54mm:PinHeader_1x02_P2.54mm_Vertical, F.Cu at (-0.65, 62.5)
- added L1: 22uH, Mizz_lib:Inductor_Taiyo-Yuden_NR-60xx, F.Cu at (-23.4, 85.2)
- added LS1: Speaker, Mizz_lib:UGCT7525AN4, F.Cu at (-73.0, 104.7)
- added Q1: NVMFD5C446NLT1G, Mizz_lib:NVMFD5C446NLWFT1G, F.Cu at (175.5, 82.0)
- added Q10: NVMFD5C446NLT1G, Mizz_lib:NVMFD5C446NLWFT1G, F.Cu at (-30.7, 85.5)
- added Q11: NVMFD5C446NLT1G, Mizz_lib:NVMFD5C446NLWFT1G, F.Cu at (-48.8, 112.6)
- added Q12: NVMFD5C446NLT1G, Mizz_lib:NVMFD5C446NLWFT1G, F.Cu at (-12.8, 72.6)
- added Q13: FET_P, Package_TO_SOT_SMD:SOT-23W, F.Cu at (-55.9, 122.6)
- added Q14: FET_N, Package_TO_SOT_SMD:SOT-23W, F.Cu at (-36.1, 103.3)
- added Q15: FET_P, Package_TO_SOT_SMD:SOT-23W, F.Cu at (-7.04, 74.1)
- added Q16: NPN, Package_TO_SOT_SMD:SOT-23W, F.Cu at (4.15, 62.5)
- added Q2: NVMFD5C446NLT1G, Mizz_lib:NVMFD5C446NLWFT1G, F.Cu at (175.5, 88.0)
- added Q3: NVMFD5C446NLT1G, Mizz_lib:NVMFD5C446NLWFT1G, F.Cu at (175.5, 106.8)
- added Q4: NVMFD5C446NLT1G, Mizz_lib:NVMFD5C446NLWFT1G, F.Cu at (175.5, 112.8)
- added Q5: NVMFD5C446NLT1G, Mizz_lib:NVMFD5C446NLWFT1G, F.Cu at (-26.3, 77.2)
- added Q6: NVMFD5C446NLT1G, Mizz_lib:NVMFD5C446NLWFT1G, F.Cu at (-37.2, 85.2)
- added Q7: NVMFD5C446NLT1G, Mizz_lib:NVMFD5C446NLWFT1G, F.Cu at (175.5, 94.5)
- added Q8: NVMFD5C446NLT1G, Mizz_lib:NVMFD5C446NLWFT1G, F.Cu at (175.5, 100.4)
- added Q9: NVMFD5C446NLT1G, Mizz_lib:NVMFD5C446NLWFT1G, F.Cu at (-6.25, 64.3)
- added R1: R, Resistor_SMD:R_0603_1608Metric, F.Cu at (-8.71, 81.0)
- added R10: 330, Resistor_SMD:R_0603_1608Metric, F.Cu at (-76.6, 126.4)
- added R11: 330, Resistor_SMD:R_0603_1608Metric, F.Cu at (-25.7, 100.1)
- added R12: 1k, Resistor_SMD:R_0603_1608Metric, F.Cu at (1.45, 73.3)
- added R13: 1k, Resistor_SMD:R_0603_1608Metric, F.Cu at (-13.5, 87.7)
- added R14: 4.7k, Resistor_SMD:R_0603_1608Metric, F.Cu at (-21.7, 96.1)
- added R15: 4.7k, Resistor_SMD:R_0603_1608Metric, F.Cu at (-47.0, 121.0)
- added R16: 10k, Resistor_SMD:R_0603_1608Metric, F.Cu at (-17.2, 92.7)
- added R17: 10k, Resistor_SMD:R_0603_1608Metric, F.Cu at (-21.7, 101.1)
- added R18: 10k, Resistor_SMD:R_0603_1608Metric, F.Cu at (-27.2, 102.7)
- added R19: 10k, Resistor_SMD:R_0603_1608Metric, F.Cu at (-13.2, 90.2)
- added R2: 10k, Resistor_SMD:R_0603_1608Metric, F.Cu at (-2.56, 73.3)
- added R20: 10k, Resistor_SMD:R_0603_1608Metric, F.Cu at (-35.1, 112.2)
- added R21: 10k, Resistor_SMD:R_0603_1608Metric, F.Cu at (-42.6, 120.3)
- added R22: 10, Resistor_SMD:R_0603_1608Metric, F.Cu at (-8.64, 86.0)
- added R23: 10, Resistor_SMD:R_0603_1608Metric, F.Cu at (-38.6, 117.3)
- added R24: 10, Resistor_SMD:R_0603_1608Metric, F.Cu at (-27.6, 105.2)
- added R25: 10, Resistor_SMD:R_0603_1608Metric, F.Cu at (-0.29, 78.3)
- added R26: 10, Resistor_SMD:R_0603_1608Metric, F.Cu at (-47.4, 126.0)
- added R27: 10, Resistor_SMD:R_0603_1608Metric, F.Cu at (-4.63, 82.6)
- added R28: 10, Resistor_SMD:R_0603_1608Metric, F.Cu at (-0.29, 75.8)
- added R29: 10, Resistor_SMD:R_0603_1608Metric, F.Cu at (-13.2, 92.7)
- added R3: 10k, Resistor_SMD:R_0603_1608Metric, F.Cu at (-4.30, 77.6)
- added R30: 10, Resistor_SMD:R_0603_1608Metric, F.Cu at (-21.7, 98.6)
- added R31: 10, Resistor_SMD:R_0603_1608Metric, F.Cu at (-35.1, 114.8)
- added R32: 10, Resistor_SMD:R_0603_1608Metric, F.Cu at (3.72, 75.8)
- added R33: 10, Resistor_SMD:R_0603_1608Metric, F.Cu at (-17.6, 97.7)
- added R34: 10k, Resistor_SMD:R_0603_1608Metric, F.Cu at (-4.63, 85.2)
- added R35: 10k, Resistor_SMD:R_0603_1608Metric, F.Cu at (-0.29, 80.8)
- added R36: 10k, Resistor_SMD:R_0603_1608Metric, F.Cu at (-28.1, 107.7)
- added R37: 10k, Resistor_SMD:R_0603_1608Metric, F.Cu at (-9.22, 88.5)
- added R38: 10k, Resistor_SMD:R_0603_1608Metric, F.Cu at (-43.0, 122.8)
- added R39: 10k, Resistor_SMD:R_0603_1608Metric, F.Cu at (-31.1, 110.2)
- added R4: R, Resistor_SMD:R_0603_1608Metric, F.Cu at (-43.5, 115.3)
- added R40: 10, Resistor_SMD:R_0603_1608Metric, F.Cu at (-42.6, 117.8)
- added R41: 10, Resistor_SMD:R_0603_1608Metric, F.Cu at (-72.6, 126.4)
- added R42: 10, Resistor_SMD:R_0603_1608Metric, F.Cu at (-17.5, 87.7)
- added R43: 10, Resistor_SMD:R_0603_1608Metric, F.Cu at (-39.1, 112.3)
- added R44: 10, Resistor_SMD:R_0603_1608Metric, F.Cu at (-39.1, 114.8)
- added R45: 10, Resistor_SMD:R_0603_1608Metric, F.Cu at (-4.30, 80.1)
- added R46: 10, Resistor_SMD:R_0603_1608Metric, F.Cu at (-8.64, 83.5)
- added R47: 10, Resistor_SMD:R_0603_1608Metric, F.Cu at (8.01, 68.9)
- added R48: 10, Resistor_SMD:R_0603_1608Metric, F.Cu at (5.46, 71.9)
- added R49: 10, Resistor_SMD:R_0603_1608Metric, F.Cu at (-23.1, 112.7)
- added R5: 330, Resistor_SMD:R_0603_1608Metric, F.Cu at (-51.4, 124.3)
- added R50: 10, Resistor_SMD:R_0603_1608Metric, F.Cu at (-5.21, 91.0)
- added R51: 10, Resistor_SMD:R_0603_1608Metric, F.Cu at (-26.6, 115.2)
- added R52: 10k, Resistor_SMD:R_0603_1608Metric, F.Cu at (3.39, 83.3)
- added R53: 2.2k, Resistor_SMD:R_0603_1608Metric, F.Cu at (-9.62, 98.6)
- added R54: 2.2k, Resistor_SMD:R_0603_1608Metric, F.Cu at (-30.6, 120.2)
- added R55: 2.2k, Resistor_SMD:R_0603_1608Metric, F.Cu at (-23.6, 105.2)
- added R56: 510, Resistor_SMD:R_0603_1608Metric, F.Cu at (-32.1, 107.3)
- added R57: 330, Resistor_SMD:R_0603_1608Metric, F.Cu at (3.72, 78.3)
- added R58: 10k, Resistor_SMD:R_0603_1608Metric, F.Cu at (-13.2, 95.2)
- added R59: 10k, Resistor_SMD:R_0603_1608Metric, F.Cu at (-24.1, 107.7)
- added R6: 330, Resistor_SMD:R_0603_1608Metric, F.Cu at (-36.6, 109.7)
- added R60: 10k, Resistor_SMD:R_0603_1608Metric, F.Cu at (-38.6, 119.8)
- added R61: FILTER, Resistor_SMD:R_0603_1608Metric, F.Cu at (-13.6, 97.7)
- added R62: FILTER, Resistor_SMD:R_0603_1608Metric, F.Cu at (-38.6, 122.3)
- added R63: FILTER, Resistor_SMD:R_0603_1608Metric, F.Cu at (3.72, 80.8)
- added R64: FILTER, Resistor_SMD:R_0603_1608Metric, F.Cu at (-9.22, 93.5)
- added R65: 10k, Resistor_SMD:R_0603_1608Metric, F.Cu at (-39.0, 124.9)
- added R66: 10, Resistor_SMD:R_0603_1608Metric, F.Cu at (-13.7, 100.2)
- added R67: 120, Resistor_SMD:R_0603_1608Metric, F.Cu at (-47.0, 123.5)
- added R68: 10k, Resistor_SMD:R_0603_1608Metric, F.Cu at (-40.9, 149.0)
- added R69: 10k, Resistor_SMD:R_0603_1608Metric, F.Cu at (-36.9, 146.5)
- added R7: 330, Resistor_SMD:R_0603_1608Metric, F.Cu at (-31.6, 104.8)
- added R70: 100k, Resistor_SMD:R_0603_1608Metric, F.Cu at (-36.2, 52.1)
- added R71: 10k, Resistor_SMD:R_0603_1608Metric, F.Cu at (-2.04, 28.5)
- added R8: 10k, Resistor_SMD:R_0603_1608Metric, F.Cu at (-17.2, 90.2)
- added R9: 10k, Resistor_SMD:R_0603_1608Metric, F.Cu at (-25.7, 97.6)
- added SW1: RST, Button_Switch_SMD:SW_SPST_CK_RS282G05A3, F.Cu at (-56.1, 96.3)
- added SW2: SW0, Button_Switch_SMD:SW_SPST_CK_RS282G05A3, F.Cu at (-91.2, 115.9)
- added SW3: SW1, Button_Switch_SMD:SW_SPST_CK_RS282G05A3, F.Cu at (-38.4, 62.8)
- added SW4: EMG, Mizz_lib:2MS1-T1-B4-VS2-Q-E, F.Cu at (-79.7, 96.6)
- added SW5: MAIN_SW, Mizz_lib:2MS1-T1-B4-VS2-Q-E, F.Cu at (-64.5, 77.5)
- added U1: BD9G101G, Package_SO:TSOP-6_1.65x3.05mm_P0.95mm, F.Cu at (-0.69, 69.7)
- added U10: NCP5104, Package_SO:SOIC-8_3.9x4.9mm_P1.27mm, F.Cu at (-82.5, 122.0)
- added U11: NCP5104, Package_SO:SOIC-8_3.9x4.9mm_P1.27mm, F.Cu at (-46.5, 97.0)
- added U12: NCP5104, Package_SO:SOIC-8_3.9x4.9mm_P1.27mm, F.Cu at (164.7, 94.4)
- added U13: NCP5104, Package_SO:SOIC-8_3.9x4.9mm_P1.27mm, F.Cu at (164.7, 100.7)
- added U14: NCP5104, Package_SO:SOIC-8_3.9x4.9mm_P1.27mm, F.Cu at (-20.3, 63.4)
- added U15: NCP5104, Package_SO:SOIC-8_3.9x4.9mm_P1.27mm, F.Cu at (-63.5, 103.3)
- added U16: NCP5104, Package_SO:SOIC-8_3.9x4.9mm_P1.27mm, F.Cu at (-33.8, 77.8)
- added U17: NCP5104, Package_SO:SOIC-8_3.9x4.9mm_P1.27mm, F.Cu at (-44.7, 84.4)
- added U18: V23086-C1001-A403, Mizz_lib:V23086-C1001-A403, F.Cu at (-70.4, 61.0)
- added U19: LOGO, Mizz_lib:Mini_Monster, F.Cu at (-30.0, 14.6)
- added U2: MCP2221A, Package_SO:SOIC-14_3.9x8.7mm_P1.27mm, F.Cu at (-28.7, 65.3)
- added U20: LOGO, Mizz_lib:Sagittarius_Alnasl_silk_40.0x11.4, F.Cu at (-60.6, 27.8)
- added U21: LOGO, Mizz_lib:Goukazal_25.0x18.8_S.Itoh_silk, F.Cu at (-62.2, 42.1)
- added U22: AQM0802, Mizz_lib:AQM0802, F.Cu at (-73.5, 143.5)
- added U3: STM32F446RETx, Package_QFP:LQFP-64_10x10mm_P0.5mm, F.Cu at (-96.2, 106.1)
- added U4: ROTARY, Mizz_lib:rotary_0F, F.Cu at (-83.3, 105.4)
- added U5: AZ1086H, Package_TO_SOT_SMD:SOT-223-3_TabPin2, F.Cu at (-91.7, 122.6)
- added U6: NCP5104, Package_SO:SOIC-8_3.9x4.9mm_P1.27mm, F.Cu at (164.7, 81.9)
- added U7: NCP5104, Package_SO:SOIC-8_3.9x4.9mm_P1.27mm, F.Cu at (164.7, 88.2)
- added U8: NCP5104, Package_SO:SOIC-8_3.9x4.9mm_P1.27mm, F.Cu at (-62.8, 109.7)
- added U9: NCP5104, Package_SO:SOIC-8_3.9x4.9mm_P1.27mm, F.Cu at (-74.1, 122.0)
- added Y1: 8MHz, Mizz_lib:Crystal_SMD_5032_2Pads, F.Cu at (-55.5, 83.9)
Routing:
- net (no net): vias 0 -> 4
Other:
- board outline added: 100 x 100 mm
- board text removed: "Sagittarius Alnasl"

Commit message: 仕様変わりスギィィィgit add -A
Parts:
- removed R70: 100k, Resistor_SMD:R_0603_1608Metric
- removed R71: 10k, Resistor_SMD:R_0603_1608Metric
- added C57: 0.1u, Capacitor_SMD:C_0603_1608Metric, B.Cu at (158.2, 123.2)
- added C58: 0.1u, Capacitor_SMD:C_0603_1608Metric, F.Cu at (80.8, 49.2)
- added C59: 0.1u, Capacitor_SMD:C_0603_1608Metric, F.Cu at (84.8, 49.2)
- added C60: 0.1u, Capacitor_SMD:C_0603_1608Metric, F.Cu at (80.8, 51.7)
- added C61: 0.1u, Capacitor_SMD:C_0603_1608Metric, F.Cu at (88.8, 49.2)
- added D29: DIODE, Diode_SMD:D_SOD-123, B.Cu at (187.8, 46.2)
- added J17: VOLTMETER, Mizz_lib:V_BattMeter, F.Cu at (191.0, 60.0)
- added J18: TO_VOLTMETER, Mizz_lib:XA_2LC, F.Cu at (187.8, 60.5)
- added J9: SERVO, Connector_PinHeader_2.54mm:PinHeader_1x03_P2.54mm_Vertical, F.Cu at (160.2, 121.9)
- added U23: 74HCT04, Package_SO:SOIC-14_3.9x8.7mm_P1.27mm, F.Cu at (134.8, 87.5)
- added U24: 74HC02, Package_SO:SOIC-14_3.9x8.7mm_P1.27mm, F.Cu at (145.9, 65.8)
- added U25: 74HC02, Package_SO:SOIC-14_3.9x8.7mm_P1.27mm, F.Cu at (146.0, 87.5)
- added U26: 74HC02, Package_SO:SOIC-14_3.9x8.7mm_P1.27mm, F.Cu at (146.0, 109.0)
- C44, C45, C46, C50, C51, C52, D21, D27, Q13, R53: moved to B.Cu
- U18: value V23086-C1001-A403 -> V23086-C1001
- U21: footprint Mizz_lib:Goukazal_25.0x18.8_S.Itoh_silk -> Mizz_lib:Goukazal_10.0x7.5_S.Itoh_silk
- moved U21 265.2 mm to (190.8, 121.5), turned to 90 degrees
- moved U20 263.1 mm to (194.2, 93.2), turned to 90 degrees
- moved SW4 258.6 mm to (165.2, 13.5), turned to 90 degrees
- moved U18 250.9 mm to (180.1, 45.5), turned to 180 degrees
- moved J12 246.8 mm to (173.2, 118.2), turned to 90 degrees
- moved J6 244.7 mm to (173.2, 58.8), turned to 90 degrees
- moved U10 239.6 mm to (156.1, 100.9)
- moved D21 239.3 mm to (165.5, 32.2)
- moved Q13 238.4 mm to (166.0, 35.5), turned to 180 degrees
- moved J8 233.7 mm to (173.2, 106.2), turned to 90 degrees
- moved U9 233.2 mm to (156.1, 84.7)
- moved J11 231.2 mm to (173.2, 94.2), turned to 90 degrees
- moved J7 230.7 mm to (173.2, 82.5), turned to 90 degrees
- moved U8 221.0 mm to (156.1, 79.3)
- moved U15 219.8 mm to (156.1, 95.5)
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Connections:
- U3 pad 15: /ADC5 -> /Buzzer_PWM
- U3 pad 20: /ADC6 -> /ADC5
- U3 pad 21: /ADC7 -> /ADC6
- U3 pad 26: /Batter_Voltage_Read -> /ADC7
- U3 pad 37: /Motor0_L_PWM -> /Motor0_CW
- U3 pad 38: /Motor0_R_PWM -> /Motor1_CW
- U3 pad 39: /Motor1_L_PWM -> /Motor2_CW
- U3 pad 40: /Motor1_R_PWM -> /Motor3_CW
- U3 pad 41: /Motor2_L_PWM -> /Motor0_PWM
- U3 pad 42: /Motor2_R_PWM -> /Motor1_PWM
- U3 pad 43: /Motor3_L_PWM -> /Motor2_PWM
- U3 pad 44: /Motor3_R_PWM -> /Motor3_PWM
- U3 pad 50: /Buzzer_PWM -> /SERVO_PWM
- U3 pad 58: /Motor5_L_PWM -> /Motor4_PWM
- U3 pad 59: /Motor5_R_PWM -> /Motor5_PWM
- U3 pad 61: /Motor4_L_PWM -> /Motor4_CW
- U3 pad 62: /Motor4_R_PWM -> /Motor5_CW
Routing:
- net Net-(D29-Pad1): track 0.00 -> 10.1 mm
- net Net-(D27-Pad1): track 0.00 -> 5.40 mm
- net Net-(D27-Pad2): track 0.00 -> 3.49 mm
- net +BATT: track 0.00 -> 2.12 mm
- net /Motor0_R: vias 0 -> 17
- net /Motor0_L: vias 0 -> 18
- added copper zone on B.Cu, net +BATT
- added copper zone on F.Cu, net /MOTOR_BATT
- added copper zone on B.Cu, net /Motor0_L
- added copper zone on F.Cu, net /Motor0_L
- added copper zone on B.Cu, net /Motor0_R
- added copper zone on F.Cu, net /Motor0_R
- added copper zone on F.Cu, net GND
- added copper zone on B.Cu, net Net-(J14-Pad3)
Other:
- board text added: "+"
- board text added: "INPUT:DC5V-15V"

Commit message: つかれた
Parts:
- added D30: DIODE, Diode_SMD:D_SOD-123, B.Cu at (129.1, 41.4)
- added U27: LOGO, Mizz_lib:AloeSetMeal_Mask_50x5.8, F.Cu at (107.5, 31.4)
- C11, C15, C5, C53, C8, D7, L1, Q14, Q15, R1, R12, R13, R4, R50, R51, R65, U1: moved to B.Cu
- C19, C20, C21, C22, C23, C24, C31, C32, C33, C34, C35, C36: footprint Capacitor_SMD:C_0603_1608Metric -> Mizz_lib:1608_WP
- C6: value 15000p -> 0.1u; moved to B.Cu
- R16, R17, R18, R19, R20, R21, R34, R35, R36, R37, R38, R39: footprint Resistor_SMD:R_0603_1608Metric -> Mizz_lib:1608_WP
- U21: footprint Mizz_lib:Goukazal_10.0x7.5_S.Itoh_silk -> Mizz_lib:Goukazal_15.0x11.3_S.Itoh_silk
- moved C27 167.4 mm to (160.4, 78.7), turned to 270 degrees
- moved C39 166.8 mm to (160.4, 89.5), turned to 270 degrees
- moved J5 147.0 mm to (127.5, 123.3)
- moved U19 143.3 mm to (130.4, 86.4)
- moved C37 136.3 mm to (160.4, 68.0), turned to 270 degrees
- moved D2 130.3 mm to (102.5, 79.8), turned to 180 degrees
- moved J16 129.8 mm to (115.0, 123.3), turned to 0 degrees
- moved C40 128.7 mm to (160.4, 94.9), turned to 270 degrees
- moved U4 128.3 mm to (125.2, 69.8), turned to 90 degrees
- moved C42 127.1 mm to (160.4, 116.5), turned to 270 degrees
- moved D3 126.3 mm to (102.5, 78.2), turned to 180 degrees
- moved C30 126.1 mm to (160.4, 105.7), turned to 270 degrees
- moved Q14 121.7 mm to (162.2, 24.8), turned to 270 degrees
- moved C41 119.3 mm to (160.4, 111.1), turned to 270 degrees
- moved R51 118.9 mm to (161.6, 119.0)
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Connections:
- U2 pad 1: Net-(U2-Pad1) -> +3V3
- U3 pad 24: /ADC8 -> /ADC7
- U3 pad 25: /ADC9 -> /ADC8
- U3 pad 26: /ADC7 -> /ADC9
Routing:
- net /Batt: track 0.00 -> 78.0 mm, vias 0 -> 2
- net +3V3: track 0.00 -> 58.0 mm
- net GND: track 0.00 -> 57.9 mm, vias 0 -> 4
- net /ADC9: track 0.00 -> 50.3 mm
- net /ADC8: track 0.00 -> 48.3 mm
- net /ADC7: track 0.00 -> 46.3 mm
- net /ADC6: track 0.00 -> 42.9 mm
- net /ADC5: track 0.00 -> 40.9 mm
- net /ADC4: track 0.00 -> 32.0 mm
- net /ADC3: track 0.00 -> 31.2 mm
- net /ADC2: track 0.00 -> 30.0 mm
- net /ADC0: track 0.00 -> 29.3 mm
- net /ADC1: track 0.00 -> 28.8 mm
- net Net-(U23-Pad6): track 0.00 -> 20.9 mm, vias 0 -> 2
- net +5V: track 0.00 -> 20.3 mm
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- added copper zone on B.Cu, net /Motor1_L
- added copper zone on B.Cu, net /Motor1_R
- added copper zone on B.Cu, net /Motor2_L
- added copper zone on B.Cu, net /Motor2_R
- added copper zone on B.Cu, net /Motor3_L
- added copper zone on B.Cu, net /Motor3_R
- added copper zone on B.Cu, net /Motor4_L
- added copper zone on B.Cu, net /Motor4_R
- added copper zone on B.Cu, net /Motor5_L
- added copper zone on B.Cu, net /Motor5_R
- added copper zone on B.Cu, net GND
Other:
- board text added: "0"
- board text added: "9"
- board text added: "Designed by A.Mizuta(@wrf_lab) in 2020/01/17."
- board text added: "INPUT:DC5V-30V"
- board text added: "Main+Power+MD*6 Non-isolation ver."
- board text added: "Painted by @SKiE1108"
- board text added: "Robot-GrandPrix."
- board text removed: "INPUT:DC5V-15V"

Commit message: ラインセンサ寸法線・和基板
Parts:
- added D31: 5V_dcdc, LED_SMD:LED_0603_1608Metric, F.Cu at (108.8, 36.8)
- added R70: 510, Resistor_SMD:R_0603_1608Metric, F.Cu at (112.8, 36.8)
- C13, C18, C54, D1, R52, R68, R69, U5: moved to B.Cu
- JP1: footprint Mizz_lib:GS2 -> Connector_PinHeader_2.54mm:PinHeader_1x02_P2.54mm_Vertical
- moved D22 147.9 mm to (194.7, 43.5), turned to 270 degrees
- moved C49 132.4 mm to (159.2, 47.0), turned to 270 degrees
- moved U5 123.3 mm to (109.7, 49.5), turned to 270 degrees
- moved D23 121.4 mm to (108.8, 34.2)
- moved C48 117.4 mm to (161.1, 47.0), turned to 270 degrees
- moved D25 115.8 mm to (108.8, 39.4)
- moved R68 86.9 mm to (116.5, 60.8), turned to 270 degrees
- moved C54 81.0 mm to (112.7, 61.4), turned to 180 degrees
- moved R69 80.9 mm to (115.0, 60.8), turned to 270 degrees
- moved D1 79.8 mm to (119.8, 67.0), turned to 270 degrees
- moved R52 78.0 mm to (162.1, 35.9), turned to 270 degrees
- moved R62 76.1 mm to (117.3, 87.2)
- moved D26 75.1 mm to (108.8, 41.9)
- moved R54 73.5 mm to (112.7, 34.2)
- moved R56 67.4 mm to (112.8, 39.4)
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Connections:
- C48 pad 1: +BATT -> /MOTOR_BATT
- C49 pad 1: +BATT -> /MOTOR_BATT
Routing:
- net Net-(D27-Pad2): track 23.1 -> 68.7 mm, vias 0 -> 2
- net +3V3: track 58.0 -> 87.7 mm, vias 0 -> 1
- net /Batt: track 78.0 -> 97.2 mm, vias 2 -> 3
- net GND: track 57.9 -> 72.2 mm
- net +5V: track 20.3 -> 31.1 mm, vias 0 -> 1
- net Net-(Q13-Pad1): track 0.00 -> 9.84 mm
- net 5Vc: track 4.86 -> 13.4 mm, vias 0 -> 1
- net Net-(C6-Pad1): track 2.00 -> 8.39 mm
- net Net-(J1-Pad2): track 0.00 -> 5.02 mm
- net Net-(D27-Pad1): track 5.40 -> 9.89 mm
- net Net-(J15-Pad3): track 0.00 -> 3.77 mm
- net Net-(J15-Pad2): track 0.00 -> 3.62 mm
- net Net-(J15-Pad5): track 0.00 -> 3.46 mm
- net Net-(J15-Pad7): track 0.00 -> 3.15 mm
- net Net-(D1-Pad2): track 0.00 -> 2.73 mm
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Other:
- board text added: "-"
- board text removed: "+"

Commit message: 配置終わり
Parts:
- C10, C16, C17, C2, C55, C56, C9, D10, D11, D12, D13, D14, D15, D16, D17, D18, D19, D20, D28, D8, D9, Q16, R10, R11, R2, R22, R23, R24, R25, R26, R27, R28, R29, R3, R30, R31, R32, R33, R40, R41, R42, R43, R44, R45, R46, R47, R48, R49, R58, R66, R67, R8, R9: moved to B.Cu
- moved D18 177.5 mm to (155.8, 93.7), turned to 180 degrees
- moved SW2 160.7 mm to (141.3, 121.5), turned to 90 degrees
- moved R41 155.2 mm to (162.6, 64.8), turned to 270 degrees
- moved SW3 147.7 mm to (145.2, 121.5), turned to 90 degrees
- moved D19 145.4 mm to (155.8, 109.8), turned to 180 degrees
- moved D20 140.8 mm to (155.8, 115.2), turned to 180 degrees
- moved D14 139.3 mm to (155.8, 104.5), turned to 180 degrees
- moved D6 137.9 mm to (117.0, 97.0), turned to 90 degrees
- moved LS1 137.9 mm to (135.4, 109.5)
- moved D12 136.4 mm to (155.8, 82.8), turned to 180 degrees
- moved D28 128.1 mm to (135.5, 115.6), turned to 180 degrees
- moved D9 127.9 mm to (155.8, 55.9), turned to 180 degrees
- moved R26 127.8 mm to (161.2, 76.8), turned to 270 degrees
- moved D15 123.7 mm to (155.8, 66.7), turned to 180 degrees
- moved R40 123.1 mm to (161.2, 64.8), turned to 270 degrees
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Routing:
- net GND: track 72.2 -> 67.9 mm
Other:
- board text added: "1"
- board text added: "SW"

Commit message: 疲れた
Routing:
- net /Batt: track 97.2 -> 129.0 mm, vias 3 -> 15
- net Net-(Q7-Pad2): track 0.00 -> 4.15 mm, vias 0 -> 1
- net Net-(Q2-Pad2): track 0.00 -> 4.15 mm, vias 0 -> 1
- net Net-(Q9-Pad2): track 0.00 -> 4.15 mm, vias 0 -> 1
- net Net-(Q10-Pad2): track 0.00 -> 4.13 mm, vias 0 -> 1
- net Net-(Q4-Pad2): track 0.00 -> 4.13 mm, vias 0 -> 1
- net Net-(Q8-Pad2): track 0.00 -> 4.11 mm, vias 0 -> 1
- net Net-(Q3-Pad2): track 0.00 -> 4.11 mm, vias 0 -> 1
- net Net-(Q1-Pad2): track 0.00 -> 4.11 mm, vias 0 -> 1
- net Net-(R48-Pad2): track 0.00 -> 3.00 mm, vias 0 -> 1
- net Net-(R49-Pad2): track 0.00 -> 2.54 mm, vias 0 -> 1
- net Net-(C37-Pad1): track 0.00 -> 2.33 mm, vias 0 -> 1
- net Net-(C26-Pad1): track 0.00 -> 2.33 mm, vias 0 -> 1
- net Net-(C41-Pad2): track 0.00 -> 2.32 mm
- net Net-(C28-Pad2): track 0.00 -> 2.32 mm
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
Commit message: ねむい
Parts:
- moved D28 5.61 mm to (135.8, 110.0), turned to 270 degrees
- moved C53 4.40 mm to (120.8, 125.5)
- moved LS1 0.95 mm to (136.3, 109.5)
Routing:
- net +3V3: track 87.7 -> 201.8 mm, vias 1 -> 8
- net +5V: track 31.1 -> 128.9 mm, vias 1 -> 3
- net /I2C2_SCL: track 1.78 -> 44.7 mm, vias 0 -> 2
- net /USART2_RX: track 0.00 -> 40.5 mm, vias 0 -> 1
- net /USART2_TX: track 0.00 -> 38.6 mm, vias 0 -> 1
- net /ENC_CH1: track 1.75 -> 32.6 mm, vias 0 -> 2
- net /Buzzer_PWM: track 0.00 -> 28.8 mm, vias 0 -> 1
- net /ENC_CH2: track 1.75 -> 30.4 mm, vias 0 -> 2
- net /I2C2_SDA: track 1.78 -> 28.5 mm
- net Net-(D2-Pad1): track 0.00 -> 9.21 mm
- net Net-(D3-Pad1): track 0.00 -> 9.04 mm
- net Net-(R23-Pad2): track 0.00 -> 8.88 mm, vias 0 -> 1
- net /OSC_IN: track 0.00 -> 8.73 mm
- net /OSC_OUT: track 0.00 -> 8.36 mm
- net Net-(R25-Pad2): track 0.00 -> 8.29 mm, vias 0 -> 1
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