File: 2020/Robot_Lancer/アロエ定食/Aloe_Set_Meal.kicad_pcb (KiCad board)
At the start: 2 copper layers, 100 x 100 mm, 233 parts, among them J1 SWD, J10 MOTOR1, J11 MOTOR3, J12 MOTOR5, J13 BATT_IN, J14 3522-2, J15 microSD, J16 SERIAL1, J17 VOLTMETER, J18 TO_VOLTMETER, J2 ADC, J3 ADC_Vdd, J4 SERIAL0, J5 ENC, J6 MOTOR0, J7 MOTOR2, J8 MOTOR4, J9 SERVO, Q1 NVMFD5C446NLT1G, Q10 NVMFD5C446NLT1G, Q11 NVMFD5C446NLT1G, Q12 NVMFD5C446NLT1G, Q13 FET_P, Q14 FET_N, Q15 FET_P, Q16 NPN, Q2 NVMFD5C446NLT1G, Q3 NVMFD5C446NLT1G, Q4 NVMFD5C446NLT1G, Q5 NVMFD5C446NLT1G, Q6 NVMFD5C446NLT1G, Q7 NVMFD5C446NLT1G, Q8 NVMFD5C446NLT1G, Q9 NVMFD5C446NLT1G, SW1 RST, SW2 SW0, SW3 SW1, SW4 EMG, SW5 MAIN_SW, U1 BD9G101G, U10 NCP5104, U11 NCP5104, U12 NCP5104, U13 NCP5104, U14 NCP5104, U15 NCP5104, U16 NCP5104, U17 NCP5104, U18 V23086-C1001, U19 LOGO, U2 MCP2221A, U20 LOGO, U21 LOGO, U22 AQM0802, U23 74HCT04, U24 74HC02, U25 74HC02, U26 74HC02, U27 LOGO, U3 STM32F446RETx, U4 ROTARY, U5 AZ1086H, U6 NCP5104, U7 NCP5104, U8 NCP5104, U9 NCP5104, Y1 8MHz

Commit message: pushできなかったからできるようにして,以前の内容をpush
Parts:
- moved C3 2.78 mm to (112.5, 77.4), turned to 270 degrees
- moved R8 0.46 mm to (127.5, 84.0)
Connections:
- U3 pad 56: /ADRESS2 -> /ADRESS3
- U3 pad 57: /ADRESS3 -> /ADRESS2
Routing:
- net /Batt: track 129.0 -> 193.3 mm
- net +3V3: track 201.8 -> 260.8 mm, vias 8 -> 14
- net /USART3_TX: track 0.00 -> 32.6 mm, vias 0 -> 2
- net /USART3_RX: track 0.00 -> 31.7 mm, vias 0 -> 2
- net /ADRESS2: track 0.00 -> 24.9 mm, vias 0 -> 2
- net /ADRESS3: track 0.00 -> 18.9 mm, vias 0 -> 2
- net /LED0: track 0.00 -> 12.3 mm, vias 0 -> 1
- net /LED1: track 0.00 -> 10.7 mm, vias 0 -> 1
- net /Motor0_R_PWM: track 2.46 -> 10.1 mm, vias 1 -> 2
- net Net-(D8-Pad2): track 0.00 -> 2.18 mm, vias 0 -> 1
- net Net-(R37-Pad1): track 0.00 -> 2.05 mm
- net Net-(R36-Pad1): track 0.00 -> 2.05 mm
- net Net-(R34-Pad1): track 0.00 -> 2.05 mm
- net Net-(R21-Pad1): track 0.00 -> 2.05 mm
- net Net-(R18-Pad1): track 0.00 -> 2.05 mm
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
Commit message: 信号線の配線終わり
Parts:
- moved J9 81.6 mm to (131.8, 45.5)
- moved C57 81.1 mm to (130.0, 47.2)
- moved D24 12.3 mm to (165.8, 120.8), turned to 0 degrees
- moved R55 4.76 mm to (170.2, 120.8), turned to 0 degrees
- moved C58 0.75 mm to (146.9, 87.5)
- moved C59 0.75 mm to (146.9, 60.4)
- moved C60 0.75 mm to (146.9, 74.0)
- moved C61 0.75 mm to (146.9, 103.7)
- moved U23 0.75 mm to (145.2, 92.8)
- moved U24 0.75 mm to (145.2, 65.8)
- moved U25 0.75 mm to (145.2, 79.2)
- moved U26 0.75 mm to (145.2, 109.0)
Connections:
- U3 pad 37: /Motor0_CW -> /Motor5_CW
- U3 pad 38: /Motor1_CW -> /Motor4_CW
- U3 pad 39: /Motor2_CW -> /Motor3_CW
- U3 pad 4: /EMG_IO -> Net-(U3-Pad4)
- U3 pad 40: /Motor3_CW -> /Motor2_CW
- U3 pad 41: /Motor0_PWM -> /Motor4_PWM
- U3 pad 42: /Motor1_PWM -> /Motor5_PWM
- U3 pad 43: /Motor2_PWM -> /Motor3_PWM
- U3 pad 44: /Motor3_PWM -> /Motor2_PWM
- U3 pad 45: Net-(U3-Pad45) -> /EMG_IO
- U3 pad 54: /ADRESS0 -> /ADRESS3
- U3 pad 55: /ADRESS1 -> /ADRESS2
- U3 pad 56: /ADRESS3 -> /ADRESS0
- U3 pad 57: /ADRESS2 -> /ADRESS1
- U3 pad 58: /Motor4_PWM -> /Motor1_PWM
- U3 pad 59: /Motor5_PWM -> /Motor0_PWM
- U3 pad 61: /Motor4_CW -> /Motor0_CW
- U3 pad 62: /Motor5_CW -> /Motor1_CW
Routing:
- net GND: track 68.2 -> 135.1 mm, vias 13 -> 90
- net /Motor1_CW: track 0.00 -> 56.8 mm, vias 0 -> 2
- net +3V3: track 260.8 -> 315.5 mm, vias 14 -> 19
- net /Motor0_CW: track 0.00 -> 52.6 mm, vias 0 -> 2
- net /Motor1_PWM: track 0.00 -> 49.0 mm, vias 0 -> 6
- net /Motor0_PWM: track 0.00 -> 48.4 mm, vias 0 -> 3
- net /Motor5_PWM: track 0.00 -> 46.9 mm, vias 0 -> 3
- net /EMG_IO: track 1.76 -> 46.7 mm, vias 0 -> 1
- net /Motor4_PWM: track 0.00 -> 40.6 mm, vias 0 -> 3
- net /Motor5_CW: track 0.00 -> 38.9 mm
- net /Motor4_CW: track 0.00 -> 36.0 mm
- net /SW1: track 2.11 -> 36.9 mm
- net /Motor3_PWM: track 0.00 -> 33.0 mm, vias 0 -> 4
- net /SERVO_PWM: track 0.00 -> 32.3 mm, vias 0 -> 2
- net /SW0: track 2.11 -> 33.0 mm
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- added copper zone on F.Cu, net /Motor1_L
- added copper zone on F.Cu, net /Motor1_R
- added copper zone on F.Cu, net /Motor2_L
- added copper zone on F.Cu, net /Motor2_R
- added copper zone on F.Cu, net /Motor3_L
- added copper zone on F.Cu, net /Motor3_R
- added copper zone on F.Cu, net /Motor4_L
- added copper zone on F.Cu, net /Motor4_R
- added copper zone on F.Cu, net /Motor5_L
- added copper zone on F.Cu, net /Motor5_R

Commit message: 和完成
Routing:
- net /Motor4_CW: track 36.0 -> 35.3 mm
- net /Motor5_CW: track 38.9 -> 38.3 mm
- net /Motor3_CW: track 16.9 -> 17.4 mm
- net GND: vias 90 -> 155
