File: 2020/Robot_Lancer/新型ラインセンサ_3V3_out/LineSensor/rancer_sensor.kicad_pcb (KiCad board)
At the start: 2 copper layers, 170 x 44 mm, 32 parts, among them P1 XH_08, U1 S7136, U2 TPR-105F, U3 TPR-105F, U4 S7136, U5 S7136

Commit message: ああああああああああああああああああ
Connections:
- P1 pad 1: +5V -> GND
- P1 pad 2: GND -> +5V
