File: 2020/Robot_Lancer/新型ラインセンサ_3V3_out/LineSensor/rancer_sensor.sch (KiCad schematic (older format))
At the start: 35 parts, among them P1 XH_08, U1 S7136, U2 TPR-105F, U3 TPR-105F, U4 S7136, U5 S7136

Commit message: ああああああああああああああああああ
Connections:
- wire segments 62 -> 63
Changed lines of the file:
@@
 L power:+5V #PWR03
 U 1 1 5C5036D6
-P 1750 3175
-F 0 "#PWR03" H 1750 3025 50  0001 C CNN
-F 1 "+5V" H 1750 3315 50  0000 C CNN
-F 2 "" H 1750 3175 50  0000 C CNN
-F 3 "" H 1750 3175 50  0000 C CNN
-	1    1750 3175
+P 1850 3275
+F 0 "#PWR03" H 1850 3125 50  0001 C CNN
+F 1 "+5V" H 1850 3415 50  0000 C CNN
+F 2 "" H 1850 3275 50  0000 C CNN
+F 3 "" H 1850 3275 50  0000 C CNN
+	1    1850 3275
 	1    0    0    -1
 $EndComp
@@
 L power:GND #PWR04
 U 1 1 5C5036EA
-P 2075 3375
-F 0 "#PWR04" H 2075 3125 50  0001 C CNN
-F 1 "GND" H 2075 3225 50  0000 C CNN
-F 2 "" H 2075 3375 50  0000 C CNN
-F 3 "" H 2075 3375 50  0000 C CNN
-	1    2075 3375
+P 2075 3175
+F 0 "#PWR04" H 2075 2925 50  0001 C CNN
+F 1 "GND" H 2075 3025 50  0000 C CNN
+F 2 "" H 2075 3175 50  0000 C CNN
+F 3 "" H 2075 3175 50  0000 C CNN
+	1    2075 3175
 	1    0    0    -1
 $EndComp
@@
 	-1   0    0    -1
 $EndComp
-Text Label 1750 3575 0    60   ~ 0
+Text Label 1750 3475 0    60   ~ 0
 AN_1
-Text Label 1750 3875 0    60   ~ 0
+Text Label 1750 3775 0    60   ~ 0
 AN_2
-$Comp
-L power:PWR_FLAG #FLG01
-U 1 1 5C506650
-P 1750 4325
-F 0 "#FLG01" H 1750 4420 50  0001 C CNN
-F 1 "PWR_FLAG" H 1750 4505 50  0000 C CNN
-F 2 "" H 1750 4325 50  0000 C CNN
-F 3 "" H 1750 4325 50  0000 C CNN
-	1    1750 4325
-	0    -1   -1   0
-$EndComp
-$Comp
-L power:PWR_FLAG #FLG02
-U 1 1 5C506692
-P 1750 4925
-F 0 "#FLG02" H 1750 5020 50  0001 C CNN
-F 1 "PWR_FLAG" H 1750 5105 50  0000 C CNN
-F 2 "" H 1750 4925 50  0000 C CNN
-F 3 "" H 1750 4925 50  0000 C CNN
-	1    1750 4925
-	0    -1   -1   0
-$EndComp
 $Comp
 L Device:C C1
@@
 Wire Wire Line
 	9250 3925 9250 4650
-Text Label 1750 3475 0    60   ~ 0
+Text Label 1750 3375 0    60   ~ 0
 DB_L
-Text Label 1750 3775 0    60   ~ 0
+Text Label 1750 3675 0    60   ~ 0
 DB_R
-Text Label 1750 3675 0    60   ~ 0
+Text Label 1750 3575 0    60   ~ 0
 DB_CENTER
 $Comp
@@
 Connection ~ 8150 2975
 Connection ~ 8150 3675
-Connection ~ 1750 4325
-Connection ~ 1750 4925
-Wire Wire Line
-	2075 3375 1750 3375
+Wire Wire Line
+	2075 3175 1750 3175
 $Comp
 L Device:R R15
@@
 	1    0    0    -1
 $EndComp
+Wire Wire Line
+	1850 3275 1750 3275
 $EndSCHEMATC
