File: 2020/Robot_Rancer/新型ラインセンサ_3V3_out/LineSensor/rancer_sensor.kicad_pcb (KiCad board)
At the start: 2 copper layers, 170 x 44 mm, 32 parts, among them P1 XH_08, U1 S7136, U2 TPR-105F, U3 TPR-105F, U4 S7136, U5 S7136

Commit message: ラインセンサmendoi
Parts:
- added RV1: 5k, Mizz_lib:VR, F.Cu at (111.0, 117.5)
- added RV2: 5k, Mizz_lib:VR, F.Cu at (234.8, 117.5)
- added RV3: 5k, Mizz_lib:VR, F.Cu at (222.2, 52.6)
- moved R5 1.67 mm to (235.6, 112.0)
Routing:
- net GND: track 100.2 -> 86.3 mm, vias 8 -> 2
- net +5V: track 249.5 -> 257.8 mm
