File: 2020/Robot_Rancer/新型ラインセンサ_3V3_out/LineSensor/rancer_sensor.sch (KiCad schematic (older format))
At the start: 35 parts, among them P1 XH_08, U1 S7136, U2 TPR-105F, U3 TPR-105F, U4 S7136, U5 S7136

Commit message: ラインセンサmendoi
Parts:
- RV1, RV2, RV3: footprint _local_TMD:myVR -> Mizz_lib:VR
Changed lines of the file:
@@
 F 0 "RV1" H 3405 3079 50  0000 R CNN
 F 1 "5k" H 3405 3170 50  0000 R CNN
-F 2 "_local_TMD:myVR" H 3475 3125 50  0001 C CNN
+F 2 "Mizz_lib:VR" H 3475 3125 50  0001 C CNN
 F 3 "~" H 3475 3125 50  0001 C CNN
 	1    3475 3125
@@
 F 0 "RV2" H 6430 3104 50  0000 R CNN
 F 1 "5k" H 6430 3195 50  0000 R CNN
-F 2 "_local_TMD:myVR" H 6500 3150 50  0001 C CNN
+F 2 "Mizz_lib:VR" H 6500 3150 50  0001 C CNN
 F 3 "~" H 6500 3150 50  0001 C CNN
 	1    6500 3150
@@
 F 0 "RV3" H 9830 3079 50  0000 R CNN
 F 1 "5k" H 9830 3170 50  0000 R CNN
-F 2 "_local_TMD:myVR" H 9900 3125 50  0001 C CNN
+F 2 "Mizz_lib:VR" H 9900 3125 50  0001 C CNN
 F 3 "~" H 9900 3125 50  0001 C CNN
 	1    9900 3125
@@
 Text Notes 2875 5075 0    50   ~ 0
 DIGITAL_LEFT
-Wire Notes Line
-	5425 2750 5425 5075
 Wire Notes Line
 	5425 5075 7075 5075
@@
 Wire Wire Line
 	1850 3275 1750 3275
+Wire Notes Line
+	5425 2750 5425 5075
 $EndSCHEMATC
