File: 2020/Robot_Rancer/Aqualius_Sadalsuud/Main.kicad_pcb (KiCad board)
At the start: 2 copper layers, 100 x 100 mm, 344 parts, among them J1 microSD, J10 I/O_Vdd, J11 ENC1, J12 ENC0, J13 ENC3, J14 ENC2, J15 5Vin, J16 EMERGENCY, J17 MOTOR0, J18 MOTOR1, J19 MOTOR2, J2 ADC, J20 MOTOR3, J21 MOTOR4, J22 MOTOR5, J23 BATT_IN, J24 BATT_IN, J25 FUSE, J27 Advanced_SBDBT, J28 PICkit3, J3 SWD, J4 CAN, J5 ADC_Vdd, J6 SERIAL0, J7 CAN, J8 VALVE, J9 SERIAL2, Q1 NPN, Q10 NVMFD5C446NLT1G, Q11 FET_N, Q12 NVMFD5C446NLT1G, Q13 NVMFD5C446NLT1G, Q14 NVMFD5C446NLT1G, Q15 NVMFD5C446NLT1G, Q16 NVMFD5C446NLT1G, Q17 NVMFD5C446NLT1G, Q2 FET_P, Q3 FET_P, Q4 FET_P, Q5 NVMFD5C446NLT1G, Q6 NVMFD5C446NLT1G, Q7 NVMFD5C446NLT1G, Q8 NVMFD5C446NLT1G, Q9 NVMFD5C446NLT1G, SW1 RESET, SW10 TOGGLESW1, SW11 TOGGLESW2, SW12 TOGGLESW3, SW2 TOGGLESW0, SW3 SW0, SW4 SW1, SW5 Control-Power_SW, SW6 SW2, SW7 SW3, SW8 EMERGENCY_SW, SW9 MAIN_SW, U1 MAX3051, U10 BD9G101G, U11 CCG30-24-12, U12 NCP5104, U13 NCP5104, U14 NCP5104, U15 NCP5104, U16 NCP5104, U17 NCP5104, U18 V23086-C1001, U19 NCP5104, U2 BD9G101G, U20 NCP5104, U21 NCP5104, U22 NCP5104, U23 NCP5104, U24 NCP5104, U25 LOGO, U26 7805, U27 TBD62083A, U28 LOGO, U29 LOGO, U3 MCP2221A, U4 AQM0802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

Commit message: 基板のシルク表記にミスがあったので直した
Parts:
- J9: value SERIAL2 -> SERIAL1
Connections:
- net /PA0_TIM5_CH2 renamed /PA1_TIM5_CH2

Commit message: モータ電源用のリレーのN.O.とN.C.間違えた
Connections:
- U18 pad 3: Net-(U18-Pad3) -> MOTOR_Batt
- U18 pad 5: MOTOR_Batt -> Net-(U18-Pad5)

Commit message: リレー,前のままであってた...
Connections:
- U18 pad 3: MOTOR_Batt -> Net-(U18-Pad3)
- U18 pad 5: Net-(U18-Pad5) -> MOTOR_Batt
Changed lines of the file:
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@@
   )
   (setup
-    (last_trace_width 0.5)
+    (last_trace_width 0.25)
     (user_trace_width 0.2)
     (user_trace_width 0.3)
@@
   (net 336 /PA8_BLUE)
   (net 337 /PA1_TIM5_CH2)
-  (net 338 "Net-(U18-Pad5)")
+  (net 338 "Net-(U18-Pad3)")
   (net_class Default "これはデフォルトのネット クラスです。"
     (clearance 0.2)
@@
     (add_net "Net-(SW9-Pad3)")
     (add_net "Net-(U11-Pad5)")
-    (add_net "Net-(U18-Pad5)")
+    (add_net "Net-(U18-Pad3)")
     (add_net "Net-(U3-Pad10)")
     (add_net "Net-(U3-Pad8)")
@@
     (fp_line (start 0 0) (end 12 0) (layer F.SilkS) (width 0.15))
     (pad 3 thru_hole circle (at 9.78 1.38 270) (size 2.5 2.5) (drill 1.5) (layers *.Cu *.Mask F.SilkS)
-      (net 25 MOTOR_Batt))
+      (net 338 "Net-(U18-Pad3)"))
     (pad 4 thru_hole circle (at 1.78 1.38 270) (size 2.5 2.5) (drill 1.5) (layers *.Cu *.Mask F.SilkS)
       (net 76 POWER_Batt))
     (pad 5 thru_hole circle (at 9.78 4.38 270) (size 2.5 2.5) (drill 1.5) (layers *.Cu *.Mask F.SilkS)
-      (net 338 "Net-(U18-Pad5)"))
+      (net 25 MOTOR_Batt))
     (pad 2 thru_hole circle (at 10.28 11.58 270) (size 1.5 1.5) (drill 0.9) (layers *.Cu *.Mask F.SilkS)
       (net 78 "Net-(D56-Pad2)"))
