File: 2020/Robot_Rancer/Aqualius_Sadalsuud/Main.sch (KiCad schematic (older format))
At the start: 344 parts, among them J1 microSD, J10 I/O_Vdd, J11 ENC1, J12 ENC0, J13 ENC3, J14 ENC2, J15 5Vin, J16 EMERGENCY, J17 MOTOR0, J18 MOTOR1, J19 MOTOR2, J2 ADC, J20 MOTOR3, J21 MOTOR4, J22 MOTOR5, J23 BATT_IN, J24 BATT_IN, J25 FUSE, J27 Advanced_SBDBT, J28 PICkit3, J3 SWD, J4 CAN, J5 ADC_Vdd, J6 SERIAL0, J7 CAN, J8 VALVE, J9 SERIAL2, Q1 NPN, Q10 NVMFD5C446NLT1G, Q11 FET_N, Q12 NVMFD5C446NLT1G, Q13 NVMFD5C446NLT1G, Q14 NVMFD5C446NLT1G, Q15 NVMFD5C446NLT1G, Q16 NVMFD5C446NLT1G, Q17 NVMFD5C446NLT1G, Q2 FET_P, Q3 FET_P, Q4 FET_P, Q5 NVMFD5C446NLT1G, Q6 NVMFD5C446NLT1G, Q7 NVMFD5C446NLT1G, Q8 NVMFD5C446NLT1G, Q9 NVMFD5C446NLT1G, SW1 RESET, SW10 TOGGLESW1, SW11 TOGGLESW2, SW12 TOGGLESW3, SW2 TOGGLESW0, SW3 SW0, SW4 SW1, SW5 Control-Power_SW, SW6 SW2, SW7 SW3, SW8 EMERGENCY_SW, SW9 MAIN_SW, U1 MAX3051, U10 BD9G101G, U11 CCG30-24-12, U12 NCP5104, U13 NCP5104, U14 NCP5104, U15 NCP5104, U16 NCP5104, U17 NCP5104, U18 V23086-C1001, U19 NCP5104, U2 BD9G101G, U20 NCP5104, U21 NCP5104, U22 NCP5104, U23 NCP5104, U24 NCP5104, U25 LOGO, U26 7805, U27 TBD62083A, U28 LOGO, U29 LOGO, U3 MCP2221A, U4 AQM0802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

Commit message: 基板のシルク表記にミスがあったので直した
Parts:
- J9: value SERIAL2 -> SERIAL1
Connections:
- net PA0_TIM5_CH2 renamed PA1_TIM5_CH2
Changed lines of the file:
@@
 P 3925 11625
 F 0 "J9" H 3982 12092 50  0000 C CNN
-F 1 "SERIAL2" H 3982 12001 50  0000 C CNN
+F 1 "SERIAL1" H 3982 12001 50  0000 C CNN
 F 2 "Connector_USB:USB_Micro-B_Molex_47346-0001" H 4075 11575 50  0001 C CNN
 F 3 "~" H 4075 11575 50  0001 C CNN
@@
 PA0_TIM5_CH1
 Text Label 2100 4975 2    50   ~ 0
-PA0_TIM5_CH2
+PA1_TIM5_CH2
 Text Label 5750 14900 0    50   ~ 0
 PA0_TIM5_CH1
 Text Label 5750 14800 0    50   ~ 0
-PA0_TIM5_CH2
+PA1_TIM5_CH2
 Wire Wire Line
 	5750 14800 5700 14800

Commit message: モータ電源用のリレーのN.O.とN.C.間違えた
Connections:
- net MOTOR_Batt: now also U18.3 (N.C); no longer U18.5 (N.O)
Other:
- moved on the sheet: C44, C45, C46, C47, C48, C49, C53, C54, C55, C56, C57, C58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

Commit message: リレー,前のままであってた...
Connections:
- net MOTOR_Batt: now also U18.5 (N.O); no longer U18.3 (N.C)
Changed lines of the file:
@@
 	1    0    0    -1
 $EndComp
-Text GLabel 18375 2050 2    50   Input ~ 0
+Text GLabel 18375 2150 2    50   Input ~ 0
 MOTOR_Batt
 Wire Wire Line
@@
 Wire Wire Line
 	18050 3075 18025 3075
-NoConn ~ 18375 2150
+NoConn ~ 18375 2050
 Text GLabel 18425 1425 2    50   Input ~ 0
 Batt
