File: 2020/Robot_Rancer/Sagittarius_Alnasl/Aloe_Set_Meal.kicad_pcb (KiCad board)
At the start: 2 copper layers, 100 x 100 mm, 235 parts, among them J1 SWD, J10 MOTOR1, J11 MOTOR3, J12 MOTOR5, J13 BATT_IN, J14 3522-2, J15 microSD, J16 SERIAL1, J17 VOLTMETER, J18 TO_VOLTMETER, J2 ADC, J3 ADC_Vdd, J4 SERIAL0, J5 ENC, J6 MOTOR0, J7 MOTOR2, J8 MOTOR4, J9 SERVO, Q1 NVMFD5C446NLT1G, Q10 NVMFD5C446NLT1G, Q11 NVMFD5C446NLT1G, Q12 NVMFD5C446NLT1G, Q13 FET_P, Q14 FET_N, Q15 FET_P, Q16 NPN, Q2 NVMFD5C446NLT1G, Q3 NVMFD5C446NLT1G, Q4 NVMFD5C446NLT1G, Q5 NVMFD5C446NLT1G, Q6 NVMFD5C446NLT1G, Q7 NVMFD5C446NLT1G, Q8 NVMFD5C446NLT1G, Q9 NVMFD5C446NLT1G, SW1 RST, SW2 SW0, SW3 SW1, SW4 EMG, SW5 MAIN_SW, U1 BD9G101G, U10 NCP5104, U11 NCP5104, U12 NCP5104, U13 NCP5104, U14 NCP5104, U15 NCP5104, U16 NCP5104, U17 NCP5104, U18 V23086-C1001, U19 LOGO, U2 MCP2221A, U20 LOGO, U21 LOGO, U22 AQM0802, U23 74HCT04, U24 74HC02, U25 74HC02, U26 74HC02, U27 LOGO, U28 FULLCOLOR, U29 LOGO, U3 STM32F446RETx, U30 LOGO, U4 ROTARY, U5 AZ1086H, U6 NCP5104, U7 NCP5104, U8 NCP5104, U9 NCP5104, Y1 8MHz

Commit message: リレー逆転
Connections:
- U18 pad 3: Net-(U18-Pad3) -> /MOTOR_BATT
- U18 pad 5: /MOTOR_BATT -> Net-(U18-Pad5)

Commit message: リレー,前のままであってた...
Connections:
- U18 pad 3: /MOTOR_BATT -> Net-(U18-Pad3)
- U18 pad 5: Net-(U18-Pad5) -> /MOTOR_BATT
Changed lines of the file:
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@@
   (net 232 /LED_Green)
   (net 233 /LED_Red)
-  (net 234 "Net-(U18-Pad5)")
+  (net 234 "Net-(U18-Pad3)")
   (net_class Default "これはデフォルトのネット クラスです。"
     (clearance 0.2)
@@
     (add_net "Net-(SW4-Pad1)")
     (add_net "Net-(SW5-Pad1)")
-    (add_net "Net-(U18-Pad5)")
+    (add_net "Net-(U18-Pad3)")
     (add_net "Net-(U2-Pad10)")
     (add_net "Net-(U2-Pad8)")
@@
     (fp_line (start 0 0) (end 12 0) (layer F.SilkS) (width 0.15))
     (pad 3 thru_hole circle (at 9.78 1.38 180) (size 2.5 2.5) (drill 1.5) (layers *.Cu *.Mask F.SilkS)
-      (net 91 /MOTOR_BATT))
+      (net 234 "Net-(U18-Pad3)"))
     (pad 4 thru_hole circle (at 1.78 1.38 180) (size 2.5 2.5) (drill 1.5) (layers *.Cu *.Mask F.SilkS)
       (net 204 "Net-(J14-Pad3)"))
     (pad 5 thru_hole circle (at 9.78 4.38 180) (size 2.5 2.5) (drill 1.5) (layers *.Cu *.Mask F.SilkS)
-      (net 234 "Net-(U18-Pad5)"))
+      (net 91 /MOTOR_BATT))
     (pad 2 thru_hole circle (at 10.28 11.58 180) (size 1.5 1.5) (drill 0.9) (layers *.Cu *.Mask F.SilkS)
       (net 65 "Net-(D27-Pad1)"))

Commit message: 抵抗値入れ忘れていたから入れた
Parts:
- R1: value R -> 680
- R4: value R -> 3.9k
Changed lines of the file:
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@@
       (effects (font (size 1 1) (thickness 0.15)) (justify mirror))
     )
-    (fp_text value R (at -2 0 90) (layer B.SilkS)
+    (fp_text value 680 (at -2 0 90) (layer B.SilkS)
       (effects (font (size 1 1) (thickness 0.15)) (justify mirror))
     )
@@
       (effects (font (size 1 1) (thickness 0.15)) (justify mirror))
     )
-    (fp_text value R (at -2 0 90) (layer B.SilkS)
+    (fp_text value 3.9k (at -2 0 90) (layer B.SilkS)
       (effects (font (size 0.8 0.8) (thickness 0.15)) (justify mirror))
     )

Commit message: Pch FET,ミスっていた---git add -A!
Parts:
- moved Q15 1.03 mm to (116.0, 41.7), turned to 180 degrees
- moved R65 0.30 mm to (116.2, 44.0)
- turned Q13 to 0 degrees
Connections:
- Q13 pad 2: Net-(D27-Pad1) -> /Batt
- Q13 pad 3: /Batt -> Net-(D27-Pad1)
- Q15 pad 2: +5V -> 5Vc
- Q15 pad 3: 5Vc -> +5V
Routing:
- net Net-(Q13-Pad1): track 9.84 -> 6.44 mm
- net 5Vc: track 13.4 -> 15.6 mm
- net /Batt: track 192.5 -> 190.9 mm
- net +5V: track 128.9 -> 128.2 mm

Commit message: 抵抗値入れた
Parts:
- Q13, Q15: footprint Package_TO_SOT_SMD:SOT-23W -> Package_TO_SOT_SMD:SOT-23
- moved Q15 50.5 mm to (166.2, 35.6), turned to 0 degrees
- moved Q13 50.4 mm to (116.0, 41.6), turned to 180 degrees
Connections:
- Q13 pad 2: /Batt -> 5Vc
- Q13 pad 3: Net-(D27-Pad1) -> +5V
- Q15 pad 2: 5Vc -> /Batt
- Q15 pad 3: +5V -> Net-(D27-Pad1)
- R52 pad 2: Net-(Q13-Pad1) -> Net-(Q15-Pad1)
- R65 pad 2: Net-(Q15-Pad1) -> Net-(Q13-Pad1)
- SW4 pad 2: Net-(Q13-Pad1) -> Net-(Q15-Pad1)
- SW5 pad 2: Net-(Q15-Pad1) -> Net-(Q13-Pad1)
Routing:
- net Net-(Q13-Pad1): track 6.44 -> 17.2 mm
- net Net-(Q15-Pad1): track 17.2 -> 6.96 mm
- net Net-(D27-Pad1): track 10.3 -> 8.74 mm
- net /Batt: track 190.9 -> 192.1 mm

Commit message: 和ランサー基板に機体のロゴを追加した
Parts:
- added U31: LOGO, Mizz_lib:kodani_miconCar_30x19_silk, F.Cu at (187.5, 86.8)
- moved U20 2.93 mm to (194.5, 93.0)
- moved U29 1.60 mm to (188.8, 101.8)
Other:
- board text added: "Designed by @wrf_lab in 2020/01/21."
- board text removed: "Designed by A.Mizuta(@wrf_lab) in 2020/01/21."
