File: Aqualius_Sadalsuud_for_KITRP/Main.kicad_pcb (KiCad board)
At the start: 2 copper layers, 100 x 100 mm, 341 parts, among them J1 microSD, J10 I/O_Vdd, J11 ENC1, J12 ENC0, J13 ENC3, J14 ENC2, J15 5Vin, J16 EMG, J17 MOTOR0, J18 MOTOR1, J19 MOTOR2, J2 ADC, J20 MOTOR3, J21 MOTOR4, J22 MOTOR5, J23 BATT_IN, J24 BATT_IN, J25 FUSE, J27 Advanced_SBDBT, J28 PICkit3, J3 SWD, J4 CAN, J5 ADC_Vdd, J6 SERIAL0, J7 CAN, J8 VALVE, J9 SERIAL2, Q1 NPN, Q10 NVMFD5C446NLT1G, Q11 FET_N, Q12 NVMFD5C446NLT1G, Q13 NVMFD5C446NLT1G, Q14 NVMFD5C446NLT1G, Q15 NVMFD5C446NLT1G, Q16 NVMFD5C446NLT1G, Q17 NVMFD5C446NLT1G, Q18 FET_P, Q2 FET_P, Q3 FET_P, Q4 FET_P, Q5 NVMFD5C446NLT1G, Q6 NVMFD5C446NLT1G, Q7 NVMFD5C446NLT1G, Q8 NVMFD5C446NLT1G, Q9 NVMFD5C446NLT1G, SW1 RESET, SW10 TOGGLESW1, SW11 TOGGLESW2, SW12 TOGGLESW3, SW2 TOGGLESW0, SW3 SW0, SW4 SW1, SW5 Control-Power_SW, SW6 SW2, SW7 SW3, SW8 EMG_SW, SW9 MAIN_SW, U1 MAX3051, U10 BD9G101G, U11 CCG30-24-12, U12 NCP5104, U13 NCP5104, U14 NCP5104, U15 NCP5104, U16 NCP5104, U17 NCP5104, U18 V23086-C1001, U19 NCP5104, U2 BD9G101G, U20 NCP5104, U21 NCP5104, U22 NCP5104, U23 NCP5104, U24 NCP5104, U25 LOGO, U26 7805, U27 TBD62083A, U28 LOGO, U29 LOGO, U30 LM7812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

Commit message: Aqualius for KIT-RP Edition... complite
Parts:
- ISO1, ISO2: footprint Package_SO:SOIC-16W_5.3x10.2mm_P1.27mm -> Package_SO:SOIC-16_3.9x9.9mm_P1.27mm
- R11: value 120 -> 10
- moved C19 1.15 mm to (62.7, 132.7)
- moved J9 1.10 mm to (56.9, 134.9)
Routing:
- net +5P: track 49.3 -> 51.4 mm
- net /motor1_R_signal: track 19.9 -> 21.7 mm
- net /motor0_L_signal: track 24.5 -> 26.4 mm
- net /motor2_R_signal: track 20.0 -> 21.7 mm
- net /motor1_L_signal: track 20.6 -> 22.3 mm
- net /motor4_R_signal: track 50.7 -> 52.4 mm
- net /motor2_L_signal: track 19.9 -> 21.5 mm
- net /motor0_R_signal: track 25.4 -> 27.0 mm
- net /motor3_L_signal: track 32.0 -> 33.6 mm
- net +3V3: track 376.6 -> 378.2 mm
- net /motor5_R_signal: track 56.5 -> 58.0 mm
- net /motor4_L_signal: track 48.2 -> 49.6 mm
- net /motor3_R_signal: track 34.2 -> 35.5 mm
- net /MOTOR5R_PWM: track 23.4 -> 24.5 mm
- net /MOTOR5L_PWM: track 18.3 -> 19.4 mm
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Other:
- board text added: "7"

Commit message: for KIT-RP
Connections:
- net /~RST renamed /~{RST}
Other:
- net class Default removed
