File: Aqualius_Sadalsuud_for_KITRP/Main.kicad_sch (KiCad schematic)
At the start: 341 parts, among them J1 microSD, J10 I/O_Vdd, J11 ENC1, J12 ENC0, J13 ENC3, J14 ENC2, J15 5Vin, J16 EMG, J17 MOTOR0, J18 MOTOR1, J19 MOTOR2, J2 ADC, J20 MOTOR3, J21 MOTOR4, J22 MOTOR5, J23 BATT_IN, J24 BATT_IN, J25 FUSE, J27 Advanced_SBDBT, J28 PICkit3, J3 SWD, J4 CAN, J5 ADC_Vdd, J6 SERIAL0, J7 CAN, J8 VALVE, J9 SERIAL2, Q1 NPN, Q10 NVMFD5C446NLT1G, Q11 FET_N, Q12 NVMFD5C446NLT1G, Q13 NVMFD5C446NLT1G, Q14 NVMFD5C446NLT1G, Q15 NVMFD5C446NLT1G, Q16 NVMFD5C446NLT1G, Q17 NVMFD5C446NLT1G, Q18 FET_P, Q2 FET_P, Q3 FET_P, Q4 FET_P, Q5 NVMFD5C446NLT1G, Q6 NVMFD5C446NLT1G, Q7 NVMFD5C446NLT1G, Q8 NVMFD5C446NLT1G, Q9 NVMFD5C446NLT1G, SW1 RESET, SW10 TOGGLESW1, SW11 TOGGLESW2, SW12 TOGGLESW3, SW2 TOGGLESW0, SW3 SW0, SW4 SW1, SW5 Control-Power_SW, SW6 SW2, SW7 SW3, SW8 EMG_SW, SW9 MAIN_SW, U1 MAX3051, U10 BD9G101G, U11 CCG30-24-12, U12 NCP5104, U13 NCP5104, U14 NCP5104, U15 NCP5104, U16 NCP5104, U17 NCP5104, U18 V23086-C1001, U19 NCP5104, U2 BD9G101G, U20 NCP5104, U21 NCP5104, U22 NCP5104, U23 NCP5104, U24 NCP5104, U25 LOGO, U26 7805, U27 TBD62083A, U28 LOGO, U29 LOGO, U30 LM7812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

Commit message: fix:motor-vdd 12V
Connections:
- net FB_OUT: now also C41.1, R58.1; no longer C41.2, R58.2
- net at R57.1, U10.3 (FB): now also C41.2, R58.2; no longer C41.1, R58.1
Other:
- moved on the sheet: C41, R57, R58
Changed lines of the file:
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@@
   (junction (at 431.8 268.605) (diameter 0) (color 0 0 0 0)
   )
-  (junction (at 342.9 103.505) (diameter 0) (color 0 0 0 0)
-  )
   (junction (at 120.015 36.195) (diameter 0) (color 0 0 0 0)
   )
@@
   (junction (at 481.33 92.075) (diameter 0) (color 0 0 0 0)
   )
+  (junction (at 326.39 103.505) (diameter 0) (color 0 0 0 0)
+  )
   (junction (at 447.675 20.955) (diameter 0) (color 0 0 0 0)
   )
@@
   (junction (at 238.76 59.69) (diameter 0) (color 0 0 0 0)
   )
-  (junction (at 334.645 103.505) (diameter 0) (color 0 0 0 0)
-  )
   (junction (at 180.34 386.08) (diameter 0) (color 0 0 0 0)
   )
@@
   (junction (at 459.74 304.8) (diameter 0) (color 0 0 0 0)
   )
-  (junction (at 342.9 111.125) (diameter 0) (color 0 0 0 0)
-  )
   (junction (at 563.88 258.445) (diameter 0) (color 0 0 0 0)
   )
@@
   (junction (at 118.11 388.62) (diameter 0) (color 0 0 0 0)
   )
+  (junction (at 334.645 95.885) (diameter 0) (color 0 0 0 0)
+  )
   (junction (at 57.15 370.84) (diameter 0) (color 0 0 0 0)
   )
@@
   (junction (at 149.86 31.115) (diameter 0) (color 0 0 0 0)
   )
+  (junction (at 334.645 103.505) (diameter 0) (color 0 0 0 0)
+  )
   (junction (at 414.655 350.52) (diameter 0) (color 0 0 0 0)
   )
@@
     (stroke (width 0) (type default) (color 0 0 0 0))
   )
-  (wire (pts (xy 334.645 103.505) (xy 327.66 103.505))
-    (stroke (width 0) (type default) (color 0 0 0 0))
-  )
   (wire (pts (xy 251.46 297.815) (xy 253.365 297.815))
     (stroke (width 0) (type default) (color 0 0 0 0))
@@
     (stroke (width 0) (type default) (color 0 0 0 0))
   )
+  (wire (pts (xy 326.39 95.885) (xy 334.645 95.885))
+    (stroke (width 0) (type default) (color 0 0 0 0))
+  )
   (wire (pts (xy 424.815 189.23) (xy 430.53 189.23))
     (stroke (width 0) (type default) (color 0 0 0 0))
@@
     (stroke (width 0) (type default) (color 0 0 0 0))
   )
-  (wire (pts (xy 343.535 111.125) (xy 342.9 111.125))
+  (wire (pts (xy 335.28 95.885) (xy 334.645 95.885))
     (stroke (width 0) (type default) (color 0 0 0 0))
   )
@@
     (stroke (width 0) (type default) (color 0 0 0 0))
   )
-  (wire (pts (xy 342.9 111.125) (xy 334.645 111.125))
+  (wire (pts (xy 334.645 103.505) (xy 326.39 103.505))
     (stroke (width 0) (type default) (color 0 0 0 0))
   )
@@
     (effects (font (size 1.27 1.27)) (justify right bottom))
   )
-  (label "FB_OUT" (at 343.535 111.125 0)
+  (label "FB_OUT" (at 335.28 95.885 0)
     (effects (font (size 1.27 1.27)) (justify left bottom))
   )
@@
     (pin "6")
   )
-  (symbol (lib_id "Device:R") (at 334.645 107.315 0) (unit 1)
+  (symbol (lib_id "Device:R") (at 326.39 99.695 0) (unit 1)
     (in_bom yes) (on_board yes)
-    (property "Reference" "R58" (id 0) (at 336.423 106.1466 0)
+    (property "Reference" "R58" (id 0) (at 328.168 98.5266 0)
       (effects (font (size 1.27 1.27)) (justify left))
     )
-    (property "Value" "7.5k" (id 1) (at 336.423 108.458 0)
+    (property "Value" "7.5k" (id 1) (at 328.168 100.838 0)
       (effects (font (size 1.27 1.27)) (justify left))
     )
-    (property "Footprint" "Resistor_SMD:R_0603_1608Metric" (id 2) (at 332.867 107.315 90)
+    (property "Footprint" "Resistor_SMD:R_0603_1608Metric" (id 2) (at 324.612 99.695 90)
       (effects (font (size 1.27 1.27)) hide)
     )
-    (property "Datasheet" "~" (id 3) (at 334.645 107.315 0)
+    (property "Datasheet" "~" (id 3) (at 326.39 99.695 0)
       (effects (font (size 1.27 1.27)) hide)
     )
@@
     (pin "2")
   )
-  (symbol (lib_id "Device:C") (at 342.9 107.315 0) (unit 1)
+  (symbol (lib_id "Device:C") (at 334.645 99.695 0) (unit 1)
     (in_bom yes) (on_board yes)
-    (property "Reference" "C41" (id 0) (at 345.821 106.1466 0)
+    (property "Reference" "C41" (id 0) (at 337.566 98.5266 0)
       (effects (font (size 1.27 1.27)) (justify left))
     )
-    (property "Value" "0.1u" (id 1) (at 345.821 108.458 0)
+    (property "Value" "0.1u" (id 1) (at 337.566 100.838 0)
       (effects (font (size 1.27 1.27)) (justify left))
     )
-    (property "Footprint" "Capacitor_SMD:C_0603_1608Metric" (id 2) (at 343.8652 111.125 0)
+    (property "Footprint" "Capacitor_SMD:C_0603_1608Metric" (id 2) (at 335.6102 103.505 0)
       (effects (font (size 1.27 1.27)) hide)
     )
-    (property "Datasheet" "~" (id 3) (at 342.9 107.315 0)
+    (property "Datasheet" "~" (id 3) (at 334.645 99.695 0)
       (effects (font (size 1.27 1.27)) hide)
     )
@@
     (pin "2")
   )
-  (symbol (lib_id "Device:R") (at 327.66 107.315 0) (unit 1)
+  (symbol (lib_id "Device:R") (at 326.39 107.315 0) (unit 1)
     (in_bom yes) (on_board yes)
-    (property "Reference" "R57" (id 0) (at 329.438 106.1466 0)
+    (property "Reference" "R57" (id 0) (at 328.168 106.1466 0)
       (effects (font (size 1.27 1.27)) (justify left))
     )
-    (property "Value" "510" (id 1) (at 329.438 108.458 0)
+    (property "Value" "510" (id 1) (at 328.168 108.458 0)
       (effects (font (size 1.27 1.27)) (justify left))
     )
-    (property "Footprint" "Resistor_SMD:R_0603_1608Metric" (id 2) (at 325.882 107.315 90)
+    (property "Footprint" "Resistor_SMD:R_0603_1608Metric" (id 2) (at 324.612 107.315 90)
       (effects (font (size 1.27 1.27)) hide)
     )
-    (property "Datasheet" "~" (id 3) (at 327.66 107.315 0)
+    (property "Datasheet" "~" (id 3) (at 326.39 107.315 0)
       (effects (font (size 1.27 1.27)) hide)
     )
@@
     (pin "2")
   )
-  (symbol (lib_id "power:GNDPWR") (at 327.66 111.125 0) (unit 1)
+  (symbol (lib_id "power:GNDPWR") (at 326.39 111.125 0) (unit 1)
     (in_bom yes) (on_board yes)
-    (property "Reference" "#PWR0161" (id 0) (at 327.66 116.205 0)
+    (property "Reference" "#PWR0161" (id 0) (at 326.39 116.205 0)
       (effects (font (size 1.27 1.27)) hide)
     )
-    (property "Value" "GNDPWR" (id 1) (at 327.7616 115.0366 0))
-    (property "Footprint" "" (id 2) (at 327.66 112.395 0)
+    (property "Value" "GNDPWR" (id 1) (at 326.4916 115.0366 0))
+    (property "Footprint" "" (id 2) (at 326.39 112.395 0)
       (effects (font (size 1.27 1.27)) hide)
     )
-    (property "Datasheet" "" (id 3) (at 327.66 112.395 0)
+    (property "Datasheet" "" (id 3) (at 326.39 112.395 0)
       (effects (font (size 1.27 1.27)) hide)
     )

Commit message: RC22 R2
Parts:
- R9: value 680 -> (none)
Changed lines of the file:
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@@
   (junction (at 512.445 45.085) (diameter 0) (color 0 0 0 0)
   )
+  (junction (at 302.895 24.13) (diameter 0) (color 0 0 0 0)
+  )
   (junction (at 142.24 278.13) (diameter 0) (color 0 0 0 0)
   )
@@
     (stroke (width 0) (type default) (color 0 0 0 0))
   )
+  (wire (pts (xy 301.625 24.13) (xy 302.895 24.13))
+    (stroke (width 0) (type default) (color 0 0 0 0))
+  )
   (wire (pts (xy 208.915 363.22) (xy 208.28 363.22))
     (stroke (width 0) (type default) (color 0 0 0 0))
@@
     (stroke (width 0) (type default) (color 0 0 0 0))
   )
+  (wire (pts (xy 306.705 21.59) (xy 306.705 26.67))
+    (stroke (width 0) (type default) (color 0 0 0 0))
+  )
   (wire (pts (xy 44.45 365.76) (xy 44.45 368.3))
     (stroke (width 0) (type default) (color 0 0 0 0))
@@
     )
   )
-  (global_label "External_5V" (shape input) (at 302.895 24.13 180) (fields_autoplaced)
+  (global_label "External_5V" (shape input) (at 301.625 24.13 180) (fields_autoplaced)
     (effects (font (size 1.27 1.27)) (justify right))
-    (property "Intersheet References" "${INTERSHEET_REFS}" (id 0) (at 0 0 0)
+    (property "Intersheet References" "${INTERSHEET_REFS}" (id 0) (at -1.27 0 0)
       (effects (font (size 1.27 1.27)) hide)
     )
@@
       (effects (font (size 1.27 1.27)) (justify left))
     )
-    (property "Value" "680" (id 1) (at 85.598 33.528 0)
+    (property "Value" "" (id 1) (at 85.598 33.528 0)
       (effects (font (size 1.27 1.27)) (justify left))
     )
@@
     (pin "2")
   )
-  (symbol (lib_id "power:GND") (at 306.705 21.59 0) (unit 1)
+  (symbol (lib_id "power:GND") (at 306.705 26.67 0) (unit 1)
     (in_bom yes) (on_board yes)
-    (property "Reference" "#PWR0127" (id 0) (at 306.705 27.94 0)
+    (property "Reference" "#PWR0127" (id 0) (at 306.705 33.02 0)
       (effects (font (size 1.27 1.27)) hide)
     )
-    (property "Value" "GND" (id 1) (at 306.832 25.9842 0))
-    (property "Footprint" "" (id 2) (at 306.705 21.59 0)
+    (property "Value" "GND" (id 1) (at 306.832 31.0642 0))
+    (property "Footprint" "" (id 2) (at 306.705 26.67 0)
       (effects (font (size 1.27 1.27)) hide)
     )
-    (property "Datasheet" "" (id 3) (at 306.705 21.59 0)
+    (property "Datasheet" "" (id 3) (at 306.705 26.67 0)
       (effects (font (size 1.27 1.27)) hide)
     )
@@
     )
     (path "/00000000-0000-0000-0000-00005e3f36cc"
-      (reference "R9") (unit 1) (value "680") (footprint "Resistor_SMD:R_0603_1608Metric")
+      (reference "R9") (unit 1) (value "600") (footprint "Resistor_SMD:R_0603_1608Metric")
     )
     (path "/00000000-0000-0000-0000-00005e0337d1"
